File: KiCad/Commodore 7/Commodore 7.kicad_sch (KiCad schematic)
At the start: 2 parts, among them J1 M20-6112045, U2 Barometer

Commit message: added stuff to 6 7 ha ha ha ha ha
Parts:
- added U1: IIM-42652 Main Accelerometer, Package_LGA:Bosch_LGA-14_3x2.5mm_P0.5mm, symbol Sensor_Motion:IIM-42652
- added U3: IIM-42652 - Main Accelerometer 2, Package_LGA:Bosch_LGA-14_3x2.5mm_P0.5mm, symbol Sensor_Motion:IIM-42652
- added U4: BMI270 - Secondary Accelerometer, BMI270 (1):XDCR_BMI270, symbol BMI270:BMI270
Connections:
- new net: U3.6 (GND), U3.7 (GND)
- new net: U1.6 (GND), U1.7 (GND)

Commit message: hiiiiiiiii!!!!!!!!
Parts:
- added U5: MMC5983MA, MMC5983MA:PQFN50P300X300X100-16N, symbol MMC5983MA:MMC5983MA
- added U6: TMP1075D, Package_SO:SO-8_3.9x4.9mm_P1.27mm, symbol Sensor_Temperature:TMP1075D
- added U7: TCA9543APWR, TCA9543APWR (1):SOP65P640X120-14N, symbol TCA9543APWR:TCA9543APWR
Connections:
- net at U4.7 (GND): now also J1.2, U2.3 (GND), U4.8 (VDD), U5.9 (GND)
- net at U2.1 (VDD): now also J1.4, U5.2 (VDD)
- net at U3.1 (AP_SDO/AP_AD0): now also J1.1, U1.1 (AP_SDO/AP_AD0), U1.6 (GND), U1.7 (GND), U3.6 (GND), U3.7 (GND), U6.4 (GND), U7.1 (AO), U7.2 (A1), U7.7 (GND)
- net at U3.13 (AP_SCL/AP_SCLK): now also U7.10 (8C1)
- net at U3.14 (AP_SDA/AP_SDIO/AP_SDI): now also U7.9 (SD1)
- net at U3.4 (INT1/INT): now also U7.8 (INT1)
- net at U3.8 (VDD): now also J1.3, U1.8 (VDD), U6.8 (V+), U7.14 (VCC)
- net at U1.13 (AP_SCL/AP_SCLK): now also U7.6 (SCO)
- net at U1.14 (AP_SDA/AP_SDIO/AP_SDI): now also U7.5 (SDO)
- net at U1.4 (INT1/INT): now also U7.11 (INT)
- net at J1.19: now also U7.13 (SDA)
- net at J1.21: now also U7.12 (SCL)
Other:
- moved on the sheet: U2, U3, U4

Commit message: heeeloooooooooooo
Parts:
- removed J1: M20-6112045, KiCad:RHDR40W69P254_2X20_5146X500X1105P, symbol M20-6112045:M20-6112045
- added C1, C3: 2.2uf, CC0805KK7R7BB225:CAP_CC0805_YAG, symbol 2025-10-06_19-14-39:CC0805KKX7R7BB225
- added C2, C4: .1uf, CC0603KRXQRQBB104:CC0603N_YAG, symbol 2025-10-06_19-12-57:CC0603KRX7R7BB104
- added C5, C6: 10nF, C0603C103K4RECTU:CAPC17595_87N_KEM, symbol 2025-10-06_19-30-10:C0603C103K4RECTU
- added J2: Conn_02x20_Odd_Even_MountingPin, symbol Connector_Generic_MountingPin:Conn_02x20_Odd_Even_MountingPin
Connections:
- net at U1.8 (VDD), U3.8 (VDD), U6.8 (V+)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: now also U1.5 (VDDIO), U3.5 (VDDIO), C1.1, C2.1, C3.1, C4.1, C5.1, C6.1
- new net: C1.2, C2.2, C5.2
- new net 3.3v: J2.5 (Pin_5), J2.6 (Pin_6)
- new net 5v: J2.7 (Pin_7), J2.8 (Pin_8)
- new net GNDA: J2.3 (Pin_3), J2.4 (Pin_4)
- new net GNDD: J2.1 (Pin_1), J2.2 (Pin_2)

Commit message: oops i delieted everything
Parts:
- added C7: 10uF, CAPC17595_87N_KEM, symbol 2025-10-06_19-30-10:C0603C103K4RECTU
Connections:
- net 3.3v: now also C1.1, C2.1, C3.1, C4.1, C5.1, C6.1, U1.12 (AP_CS), U1.5 (VDDIO), U1.8 (VDD), U3.12 (AP_CS), U3.14 (AP_SDA/AP_SDIO/AP_SDI), U3.5 (VDDIO), U3.8 (VDD), U5.13 (VDDIO), U5.2 (VDD), U6.8 (V+), U7.14 (VCC), U7.9 (SD1)
- net GNDA: now also C1.2, C2.2, C3.2, C4.2, C5.2, C6.2
- net GNDD: now also U1.1 (AP_SDO/AP_AD0), U1.6 (GND), U1.7 (GND), U3.1 (AP_SDO/AP_AD0), U3.6 (GND), U3.7 (GND), U5.11 (GND__1), U5.9 (GND), U7.1 (AO), U7.2 (A1), U7.7 (GND), C7.2
- net at U5.10 (CAP): now also C7.1
- net at U2.1 (VDD): no longer U5.2 (VDD)
- net SDA-IIM: now reaches J2.11 (Pin_11)
- net SDA-IIM: now also U7.13 (SDA)
- net SCL-IIM: now reaches J2.9 (Pin_9)
- net SCL-IIM: now also U7.12 (SCL)
- net SCL-IIM2: now reaches U3.13 (AP_SCL/AP_SCLK), U7.10 (8C1)
- net at U3.4 (INT1/INT): no longer U7.8 (INT1)
- net SCL-IIM1: now reaches U1.13 (AP_SCL/AP_SCLK), U7.6 (SCO)
- net SDA-IIM1: now reaches U1.14 (AP_SDA/AP_SDIO/AP_SDI), U7.5 (SDO)
- net at U1.4 (INT1/INT): no longer U7.11 (INT)
- now unconnected: U2.3 (GND), U4.7 (GND), U4.8 (VDD), U6.4 (GND)
Other:
- moved on the sheet: C1, C2, C3, C4, C5, C6

Commit message: uhhhhh
Parts:
- removed C7: 10uF, CAPC17595_87N_KEM, symbol 2025-10-06_19-30-10:C0603C103K4RECTU
- added C7: 10uF, CC0805KK7R7BB225:CAP_CC0805_YAG, symbol 2025-10-06_20-59-07:CC0805MKX7R7BB106
- added C8: 1uF, YAG_CC0603_YAG, symbol 2025-10-06_21-03-45:CC0603KRX7R7BB105
- added R1, R2: 2.7K, RES0805_CRG_TYCO_TYC, symbol 2025-10-06_20-52-39:CRG0805F2K7
Connections:
- net 3.3v: now also U5.4 (~{SPI_CS}), C8.1, R1.2, R2.2
- net GNDA: now also C8.2
- net GNDD: now also C7.2
- net at U5.1 (SCL/SPI_SCK): now also R1.1
- net at U5.10 (CAP): now also C7.1
- net at U5.16 (SDA/SPI_SDI): now also R2.1
- net INT-IIM2: now reaches U3.4 (INT1/INT)
- net INT-IIM2: now also U7.8 (INT1)
- net INT-IIM1: now reaches U1.4 (INT1/INT)
- net INT-IIM1: now also U7.4 (INTO)

Commit message: connecting 6 or 7 wires ha ha ha ha ha ha ha
Parts:
- removed U6: TMP1075D, Package_SO:SO-8_3.9x4.9mm_P1.27mm, symbol Sensor_Temperature:TMP1075D
- added C9: 10nF, C0603C103K4RECTU:CAPC17595_87N_KEM, symbol 2025-10-06_19-30-10:C0603C103K4RECTU
- added R10, R11, R13, R3, R4, R5, R6, R7, R8, R9: 2.7K, CRG0805F2K7:RES0805_CRG_TYCO_TYC, symbol 2025-10-06_20-52-39:CRG0805F2K7
- added R12: 5K, CRCW08055K00FKTA:RESC2012X50N, symbol CRCW08055K00FKTA:CRCW08055K00FKTA
- added R14, R15: 5k, CRCW08055K00FKTA:RESC2012X50N, symbol CRCW08055K00FKTA:CRCW08055K00FKTA
- added U6: TMP112AIDRLR, TMP112AIDRLR:SOT50P160X60-6N, symbol TMP112AIDRLR:TMP112AIDRLR
- C8: footprint YAG_CC0603_YAG -> CC0603KRX7R7BB105:YAG_CC0603_YAG
- R1, R2: footprint RES0805_CRG_TYCO_TYC -> CRG0805F2K7:RES0805_CRG_TYCO_TYC
Connections:
- net SCL-IIM is gone; now on net I2C-SCL-MAIN: J2.9 (Pin_9), U7.12 (SCL)
- net 3.3v: now also R10.1, R11.2, R13.2, R14.2, R15.2, R3.2, R4.2, R5.2, R6.2, R7.2, R8.2, R9.2; no longer U3.14 (AP_SDA/AP_SDIO/AP_SDI), U7.9 (SD1)
- net GNDA: now also C9.2, U6.3 (ALERT)
- net GNDD: now also U1.9 (INT2/FSYNC/CLKIN), U3.9 (INT2/FSYNC/CLKIN), U6.2 (GND), U6.4 (ADD0)
- net INT-IIM1: now also R7.1
- net INT-IIM2: now also R11.1
- net SCL-IIM1: now also R8.1
- net SCL-IIM2: now also R10.2
- net SDA-IIM1: now also R13.1
- net I2C-SCL-MAIN: now reaches J2.13 (Pin_13)
- net I2C-SCL-MAIN: now also U7.11 (INT), R14.1, R3.1, R5.1, U6.1 (SCL)
- net IIM-MAIN-RESET: now reaches J2.15 (Pin_15)
- net I2C-MAIN-RESET: now reaches U7.3 (RESET)
- net I2C-MAIN-RESET: now also R4.1
- net SDA-IIM renamed I2C-SDA-MAIN
- net I2C-SDA-MAIN: now also R15.1, U6.6 (SDA); no longer U7.13 (SDA)
- new net: C9.1, R12.1, U6.5 (V+)
- new net 3.3V: R12.2
- new net IIM-SDA-MAIN: R6.1, U7.13 (SDA)
- new net SDA-IIM2: R9.1, U3.14 (AP_SDA/AP_SDIO/AP_SDI), U7.9 (SD1)

Commit message: doing sensors ha ha
Parts:
- added C10, C11: .1uF, CC0603KRXQRQBB104:CC0603N_YAG, symbol 2025-10-06_19-12-57:CC0603KRX7R7BB104
- added R16, R17, R18: 2.7K, CRG0805F2K7:RES0805_CRG_TYCO_TYC, symbol 2025-10-06_20-52-39:CRG0805F2K7
Connections:
- net 3.3v: now also U4.12 (CSB), U4.5 (VDDIO), U4.8 (VDD), C10.2, C11.1, R16.1, R17.1, R18.1
- net GNDA: no longer U6.3 (ALERT)
- net GNDD: now also U4.10 (OSCB), U4.11 (OSDO), U4.6 (GNDIO), U4.7 (GND), U6.3 (ALERT), C10.1, C11.2
- net I2C-SCL-MAIN: now also U4.13 (SCX), R17.2
- net I2C-SDA-MAIN: now also U4.14 (SDX), R16.2
- net at U4.1 (SDO): now also R18.2
- net INT1-BMI: now reaches U4.4 (INT1)
- net INT1-BMI: now also J2.10 (Pin_10)
- net INT2-BMI: now reaches U4.9 (INT2)
- net INT2-BMI: now also J2.12 (Pin_12)
Other:
- moved on the sheet: C7, U4

Commit message: SENSORS WIRED RAHHHHHHHHHHHHHHHHH
Parts:
- removed C1, C3: 2.2uf, CC0805KK7R7BB225:CAP_CC0805_YAG, symbol 2025-10-06_19-14-39:CC0805KKX7R7BB225
- removed C10, C11: .1uF, CC0603KRXQRQBB104:CC0603N_YAG, symbol 2025-10-06_19-12-57:CC0603KRX7R7BB104
- removed C2, C4: .1uf, CC0603KRXQRQBB104:CC0603N_YAG, symbol 2025-10-06_19-12-57:CC0603KRX7R7BB104
- removed C5, C6, C9: 10nF, C0603C103K4RECTU:CAPC17595_87N_KEM, symbol 2025-10-06_19-30-10:C0603C103K4RECTU
- removed C7: 10uF, CC0805KK7R7BB225:CAP_CC0805_YAG, symbol 2025-10-06_20-59-07:CC0805MKX7R7BB106
- removed C8: 1uF, CC0603KRX7R7BB105:YAG_CC0603_YAG, symbol 2025-10-06_21-03-45:CC0603KRX7R7BB105
- removed R1, R10, R11, R13, R16, R17, R18, R2, R3, R4, R5, R6, R7, R8, R9: 2.7K, CRG0805F2K7:RES0805_CRG_TYCO_TYC, symbol 2025-10-06_20-52-39:CRG0805F2K7
- removed R12: 5K, CRCW08055K00FKTA:RESC2012X50N, symbol CRCW08055K00FKTA:CRCW08055K00FKTA
- removed R14, R15: 5k, CRCW08055K00FKTA:RESC2012X50N, symbol CRCW08055K00FKTA:CRCW08055K00FKTA
- removed U1: IIM-42652 Main Accelerometer, Package_LGA:Bosch_LGA-14_3x2.5mm_P0.5mm, symbol Sensor_Motion:IIM-42652
- removed U2: Barometer, MS560702BA03_50 (1):SON125P300X500X100-8N, symbol MS560702BA03-50:MS560702BA03-50
- removed U3: IIM-42652 - Main Accelerometer 2, Package_LGA:Bosch_LGA-14_3x2.5mm_P0.5mm, symbol Sensor_Motion:IIM-42652
- removed U4: BMI270 - Secondary Accelerometer, BMI270 (1):XDCR_BMI270, symbol BMI270:BMI270
- removed U5: MMC5983MA, MMC5983MA:PQFN50P300X300X100-16N, symbol MMC5983MA:MMC5983MA
- removed U6: TMP112AIDRLR, TMP112AIDRLR:SOT50P160X60-6N, symbol TMP112AIDRLR:TMP112AIDRLR
- removed U7: TCA9543APWR, TCA9543APWR (1):SOP65P640X120-14N, symbol TCA9543APWR:TCA9543APWR
Connections:
- net I2C-SCL-MAIN: no longer J2.13 (Pin_13)
- net INT-MMC: now reaches J2.14 (Pin_14)
- new net IIM-MAIN-INT: J2.13 (Pin_13)
Other:
- added sheet BMI270 (BMI270.kicad_sch)
- added sheet IIM-42652 (MAIN CONNECTION.kicad_sch)
- added sheet MMC5983 (MMC5983.kicad_sch)
- added sheet MS560702 (MS560702.kicad_sch)
- added sheet TMP112 (TMP112.kicad_sch)
