File: KiCad/Commodore 7/MAIN CONNECTION.kicad_sch (KiCad schematic)
At the start: 19 parts, among them U10 TCA9543APWR, U8 IIM-42652 - Main Acceleromete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, U9 IIM-42652 Main Accelerometer

Commit message: helloooo
Parts:
- removed R22, R24, R25, R26: 2.7k, CRG0805F2K7:RES0805_CRG_TYCO_TYC, symbol 2025-10-06_20-52-39:CRG0805F2K7
- added R1, R2, R3, R4: 4.7k, RC0402FR:YAG_R0402_YAG, symbol RC0402FR:RC0402FR-074K7L
Connections:
- net 3.3v: now also R1.2, R2.2, R3.2, R4.2
- net I2C-MAIN-RESET: now also R3.1
- net I2C-SCL-MAIN: now also R2.1
- net IIM-MAIN-INT: now also R4.1
- net IIM-SDA-MAIN: now also R1.1

Commit message: pcb started igggggggg
Connections:
- net 3.3v: now also R23.2; no longer R23.1
- net SDA-IIM2: now also R23.1; no longer R23.2
Other:
- moved on the sheet: R23
Changed lines of the file:
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@@
 	)
 	(junction
+		(at 52.07 149.86)
+		(diameter 0)
+		(color 0 0 0 0)
+	)
+	(junction
 		(at 90.17 66.04)
 		(diameter 0)
@@
 	)
 	(junction
-		(at 52.07 149.86)
-		(diameter 0)
-		(color 0 0 0 0)
-	)
-	(junction
 		(at 116.84 82.55)
 		(diameter 0)
@@
 	(wire
 		(pts
+			(xy 52.07 149.86) (xy 72.39 149.86)
+		)
+		(stroke
+			(width 0)
+			(type default)
+		)
+	)
+	(wire
+		(pts
 			(xy 93.98 125.73) (xy 99.06 125.73)
 		)
@@
 	(wire
 		(pts
-			(xy 52.07 149.86) (xy 72.39 149.86)
-		)
-		(stroke
-			(width 0)
-			(type default)
-		)
-	)
-	(wire
-		(pts
 			(xy 95.25 138.43) (xy 95.25 139.7)
 		)
@@
 	(wire
 		(pts
-			(xy 43.18 149.86) (xy 52.07 149.86)
+			(xy 207.01 77.47) (xy 185.42 77.47)
 		)
 		(stroke
@@
 	(wire
 		(pts
-			(xy 207.01 77.47) (xy 185.42 77.47)
+			(xy 69.85 77.47) (xy 53.34 77.47)
 		)
 		(stroke
@@
 	(wire
 		(pts
-			(xy 69.85 77.47) (xy 53.34 77.47)
+			(xy 43.18 149.86) (xy 52.07 149.86)
 		)
 		(stroke
@@
 	(wire
 		(pts
+			(xy 59.69 109.22) (xy 59.69 147.32)
+		)
+		(stroke
+			(width 0)
+			(type default)
+		)
+	)
+	(wire
+		(pts
 			(xy 207.01 54.61) (xy 207.01 46.99)
 		)
@@
 	(wire
 		(pts
+			(xy 52.07 138.43) (xy 52.07 149.86)
+		)
+		(stroke
+			(width 0)
+			(type default)
+		)
+	)
+	(wire
+		(pts
 			(xy 185.42 105.41) (xy 209.55 105.41)
 		)
@@
 	(wire
 		(pts
-			(xy 59.69 147.32) (xy 59.69 109.22)
-		)
-		(stroke
-			(width 0)
-			(type default)
-		)
-	)
-	(wire
-		(pts
 			(xy 93.98 59.69) (xy 95.25 59.69)
 		)
@@
 	(wire
 		(pts
-			(xy 52.07 138.43) (xy 52.07 149.86)
-		)
-		(stroke
-			(width 0)
-			(type default)
-		)
-	)
-	(wire
-		(pts
 			(xy 191.77 46.99) (xy 198.12 46.99)
 		)
@@
 	(symbol
 		(lib_id "2025-10-06_20-52-39:CRG0805F2K7")
-		(at 52.07 138.43 180)
+		(at 39.37 138.43 0)
 		(unit 1)
 		(exclude_from_sim no)
@@
 		(dnp no)
 		(property "Reference" "R23"
-			(at 48.006 140.97 0)
+			(at 43.434 135.89 0)
 			(effects
 				(font
@@
 		)
 		(property "Value" "2.7K"
-			(at 42.672 141.224 0)
+			(at 48.768 135.636 0)
 			(effects
 				(font
@@
 		)
 		(property "Footprint" "CRG0805F2K7:RES0805_CRG_TYCO_TYC"
-			(at 52.07 138.43 0)
+			(at 39.37 138.43 0)
 			(effects
 				(font
@@
 		)
 		(property "Datasheet" "https://www.te.com/commerce/DocumentDelivery/DDEController?Action=srchrtrv&DocNm=1773204&DocType=Data+Sheet&DocLang=English&PartCntxt=1623181-1&DocFormat=pdf"
-			(at 52.07 138.43 0)
+			(at 39.37 138.43 0)
 			(effects
 				(font
@@
 		)
 		(property "Description" ""
-			(at 52.07 138.43 0)
+			(at 39.37 138.43 0)
 			(effects
 				(font

Commit message: uhhhh didnt do as much as i shoulve mb gang
Connections:
- net I2C-SCL-MAIN renamed I2C-SLC-MAIN
Changed lines of the file:
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@@
-		)
-	)
-	(global_label "I2C-SCL-MAIN"
-		(shape input)
-		(at 201.93 114.3 180)
-		(fields_autoplaced yes)
-		(effects
-			(font
-				(size 1.27 1.27)
-			)
-			(justify right)
-		)
-		(property "Intersheetrefs" "${INTERSHEET_REFS}"
-			(at 184.7328 114.3 0)
-			(effects
-				(font
-					(size 1.27 1.27)
-				)
-				(justify right)
-				(hide yes)
-			)
 		)
 	)
@@
 			(effects
 				(font
+					(size 1.27 1.27)
+				)
+				(justify right)
+				(hide yes)
+			)
+		)
+	)
+	(global_label "I2C-SLC-MAIN"
+		(shape input)
+		(at 201.93 114.3 180)
+		(fields_autoplaced yes)
+		(effects
+			(font
+				(size 1.27 1.27)
+			)
+			(justify right)
+		)
+		(property "Intersheetrefs" "${INTERSHEET_REFS}"
+			(at 184.7328 114.3 0)
+			(effects
+				(font

Commit message: uhhhh its not working agian
Connections:
- net IIM-SDA-MAIN renamed I2C-SDA-MAIN
Changed lines of the file:
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@@
 		)
 	)
-	(global_label "IIM-SDA-MAIN"
+	(global_label "I2C-SDA-MAIN"
 		(shape input)
 		(at 201.93 129.54 180)
@@
 		)
 		(property "Intersheetrefs" "${INTERSHEET_REFS}"
-			(at 185.0956 129.54 0)
+			(at 184.6723 129.54 0)
 			(effects
 				(font

Commit message: uhhhhhh theres a lot of vias oh well
Connections:
- net GNDA is gone; now on net GNDD: C12.2, C13.2, C14.2, C15.2, C16.2, C17.2
- net I2C-SLC-MAIN renamed I2C-SCL-MAIN
