File: KiCad/Commodore 7/Commodore 7.kicad_pcb (KiCad board)
At the start: 2 copper layers, 41 parts, among them IC1 BGU7004,115, J1 M20-6112045, U1 TMP112AIDRLR-Temperature, U10 TCA9543APWR, U2 NEO-M9N-00B, U3 BMI270 - Secondary Accelerome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, U4 MMC5983MA-Magnetomer, U5 MS560702BA03-50 - Barometer, U6 TCA9509DGKR, U7 SN65HVD74DR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

Commit message: fix j2 header
Parts:
- U2: moved to B.Cu
- moved C3 141.6 mm to (180.9, 119.6), turned to 90 degrees
- moved R6 141.2 mm to (172.0, 125.2), turned to 180 degrees
- moved U3 134.2 mm to (172.2, 119.4), turned to 90 degrees
- moved C2 132.6 mm to (174.5, 116.4), turned to -45 degrees
- moved C13 111.8 mm to (140.3, 125.3), turned to -90 degrees
- moved C15 109.0 mm to (138.1, 125.0), turned to -90 degrees
- moved C16 103.0 mm to (136.0, 70.2), turned to 90 degrees
- moved U9 102.1 mm to (135.5, 78.3), turned to 180 degrees
- moved R23 100.8 mm to (130.5, 114.7), turned to 180 degrees
- moved U8 100.5 mm to (135.5, 120.3), turned to 0 degrees
- moved R27 100.0 mm to (135.6, 84.6), turned to -90 degrees
- moved R1 98.9 mm to (132.1, 106.4), turned to -90 degrees
- moved R19 97.3 mm to (130.5, 112.2), turned to 180 degrees
- moved C14 97.0 mm to (134.1, 70.2), turned to 90 degrees
- moved R2 96.8 mm to (130.6, 106.4), turned to -90 degrees
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Connections:
- C2 pad 1: GNDD -> 3.3v
- C2 pad 2: 3.3v -> GNDD
- R2 pad 1: 3.3v -> I2C-SLC-MAIN
- R23 pad 1: 3.3v -> SDA-IIM2
- R23 pad 2: SDA-IIM2 -> 3.3v
- U10 pad 12: 3.3v -> I2C-SLC-MAIN
Routing:
- net 3.3v: track 8.60 -> 77.5 mm, vias 0 -> 5
- net SCL-IIM2: track 7.41 -> 27.9 mm, vias 0 -> 2
- net SDA-IIM2: track 7.35 -> 26.7 mm, vias 0 -> 2
- net Net-(U11-RF_OUT): track 0.00 -> 18.3 mm, vias 0 -> 1
- net INT-IIM2: track 10.9 -> 27.0 mm, vias 0 -> 2
- net GNDD: track 0.00 -> 12.2 mm
- net Net-(E1-Pad1): track 0.00 -> 9.23 mm, vias 0 -> 1
- net Net-(U1-V+): track 0.00 -> 8.31 mm
- net Net-(IC1-VCC): track 0.00 -> 7.98 mm
- net IIM-SDA-MAIN: track 0.00 -> 5.20 mm
- net I2C-SLC-MAIN: track 0.00 -> 4.85 mm
- net Net-(U3-SDO): track 0.00 -> 4.74 mm
- net IIM-MAIN-INT: track 0.00 -> 4.50 mm
- net Net-(U4-CAP): track 0.00 -> 2.93 mm
- net Net-(IC1-RF_OUT): track 0.00 -> 2.75 mm
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
Commit message: oops
Parts:
- removed J1: M20-6112045, KiCad:RHDR40W69P254_2X20_5146X500X1105P
- added J2: Conn_02x20_Odd_Even_MountingPin, Connector_PinHeader_1.00mm:PinHeader_2x20_P1.00mm_Vertical, F.Cu at (149.9, 81.4)

Commit message: update
Connections:
- J2 pad 31: IIM-MAIN-RESET -> I2C-MAIN-RESET

Commit message: uhhhh its not working agian
Parts:
- moved C3 24.8 mm to (171.0, 96.9)
- moved C5 24.8 mm to (159.9, 90.2)
- moved R6 24.8 mm to (162.1, 102.5)
- moved U3 24.8 mm to (162.2, 96.7)
- moved U4 24.8 mm to (161.4, 85.6)
- moved C2 24.8 mm to (164.6, 93.7)
- moved C4 24.8 mm to (161.7, 80.5)
Routing:
- net IIM-MAIN-INT: track 4.50 -> 33.3 mm, vias 0 -> 1
- net I2C-MAIN-RESET: track 9.33 -> 31.1 mm
- net INT1-BMI: track 0.00 -> 20.0 mm, vias 0 -> 1
- net INT-MMC: track 0.00 -> 17.0 mm
- net INT2-BMI: track 0.00 -> 15.4 mm

Commit message: oh wow
Connections:
- J2 pad 3: 3.3v -> I2C-SDA-MAIN
- J2 pad 4: 3.3v -> I2C-SCL-MAIN
- R1 pad 1: IIM-SDA-MAIN -> I2C-SDA-MAIN
- U1 pad 1: 3.3v -> I2C-SCL-MAIN
- U1 pad 6: 3.3v -> I2C-SDA-MAIN
- U10 pad 13: IIM-SDA-MAIN -> I2C-SDA-MAIN
- U3 pad 13: 3.3v -> I2C-SCL-MAIN
- U3 pad 14: 3.3v -> I2C-SDA-MAIN
- U4 pad 1: 3.3v -> I2C-SCL-MAIN
- U4 pad 16: 3.3v -> I2C-SDA-MAIN
- U5 pad 7: 3.3v -> I2C-SDA-MAIN
- U5 pad 8: 3.3v -> I2C-SCL-MAIN
Routing:
- net IIM-SDA-MAIN: track 5.20 -> 0.00 mm
- net I2C-SDA-MAIN: track 0.00 -> 5.20 mm
Changed lines of the file:
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@@
 	(net 22 "I2C-MAIN-RESET")
 	(net 23 "INT-IIM2")
-	(net 24 "IIM-SDA-MAIN")
+	(net 24 "I2C-SDA-MAIN")
 	(net 25 "SDA-IIM2")
 	(net 26 "IIM-MAIN-INT")
@@
 	(net 86 "unconnected-(U7-Y-Pad5)")
 	(net 87 "I2C-SLC-MAIN")
+	(net 88 "I2C-SCL-MAIN")
 	(footprint "RC0402FR:YAG_R0402_YAG"
 		(layer "F.Cu")
@@
 			(size 0.5588 0.5588)
 			(layers "F.Cu" "F.Mask" "F.Paste")
-			(net 24 "IIM-SDA-MAIN")
+			(net 24 "I2C-SDA-MAIN")
 			(pintype "unspecified")
 		)
@@
 			(size 0.25 0.475)
 			(layers "F.Cu" "F.Mask" "F.Paste")
-			(net 21 "3.3v")
+			(net 88 "I2C-SCL-MAIN")
 			(pinfunction "SCX")
 			(pintype "input")
@@
 			(size 0.25 0.475)
 			(layers "F.Cu" "F.Mask" "F.Paste")
-			(net 21 "3.3v")
+			(net 24 "I2C-SDA-MAIN")
 			(pinfunction "SDX")
 			(pintype "bidirectional")
@@
 			(size 0.45 0.3)
 			(layers "F.Cu" "F.Mask" "F.Paste")
-			(net 21 "3.3v")
+			(net 88 "I2C-SCL-MAIN")
 			(pinfunction "SCL/SPI_SCK")
 			(pintype "input")
@@
 			(size 0.3 0.45)
 			(layers "F.Cu" "F.Mask" "F.Paste")
-			(net 21 "3.3v")
+			(net 24 "I2C-SDA-MAIN")
 			(pinfunction "SDA/SPI_SDI")
 			(pintype "bidirectional")
@@
 			(layers "*.Cu" "*.Mask")
 			(remove_unused_layers no)
-			(net 21 "3.3v")
+			(net 24 "I2C-SDA-MAIN")
 			(pinfunction "Pin_3")
 			(pintype "passive")
@@
 			(layers "*.Cu" "*.Mask")
 			(remove_unused_layers no)
-			(net 21 "3.3v")
+			(net 88 "I2C-SCL-MAIN")
 			(pinfunction "Pin_4")
 			(pintype "passive")
@@
 			(layers "F.Cu" "F.Mask" "F.Paste")
 			(roundrect_rratio 0.08)
-			(net 21 "3.3v")
+			(net 24 "I2C-SDA-MAIN")
 			(pinfunction "SDI/SDA")
 			(pintype "bidirectional")
@@
 			(layers "F.Cu" "F.Mask" "F.Paste")
 			(roundrect_rratio 0.08)
-			(net 21 "3.3v")
+			(net 88 "I2C-SCL-MAIN")
 			(pinfunction "SCLK")
 			(pintype "input")
@@
 			(layers "F.Cu" "F.Mask" "F.Paste")
 			(roundrect_rratio 0.125)
-			(net 24 "IIM-SDA-MAIN")
+			(net 24 "I2C-SDA-MAIN")
 			(pinfunction "SDA")
 			(pintype "bidirectional")
@@
 			(size 0.66 0.31)
 			(layers "F.Cu" "F.Mask" "F.Paste")
-			(net 21 "3.3v")
+			(net 88 "I2C-SCL-MAIN")
 			(pinfunction "SCL")
 			(pintype "input")
@@
 			(size 0.66 0.31)
 			(layers "F.Cu" "F.Mask" "F.Paste")
-			(net 21 "3.3v")
+			(net 24 "I2C-SDA-MAIN")
 			(pinfunction "SDA")
 			(pintype "bidirectional")

Commit message: uhhhhhh theres a lot of vias oh well
Parts:
- added R10: 4.7k, RC0402FR:YAG_R0402_YAG, F.Cu at (159.7, 99.1)
- added R11: 4.7k, RC0402FR:YAG_R0402_YAG, F.Cu at (157.4, 89.0)
- added R12: 4.7k, RC0402FR:YAG_R0402_YAG, F.Cu at (158.7, 90.3)
- added R9: 4.7k, RC0402FR:YAG_R0402_YAG, F.Cu at (159.6, 93.1)
- moved C1 67.9 mm to (159.4, 72.6), turned to 0 degrees
- moved R5 62.2 mm to (154.8, 70.7), turned to 90 degrees
- moved U1 52.8 mm to (150.4, 72.7), turned to 0 degrees
- moved U5 44.4 mm to (145.2, 66.7)
- moved C5 4.35 mm to (164.3, 90.4), turned to -45 degrees
- moved C4 2.28 mm to (163.8, 81.5), turned to -45 degrees
Connections:
- C1 pad 2: GNDA -> GNDD
- C12 pad 2: GNDA -> GNDD
- C13 pad 2: GNDA -> GNDD
- C14 pad 2: GNDA -> GNDD
- C15 pad 2: GNDA -> GNDD
- C16 pad 2: GNDA -> GNDD
- C17 pad 2: GNDA -> GNDD
- C5 pad 2: GNDA -> GNDD
- R2 pad 1: I2C-SLC-MAIN -> I2C-SCL-MAIN
- U10 pad 12: I2C-SLC-MAIN -> I2C-SCL-MAIN
Routing:
- net I2C-SDA-MAIN: track 5.20 -> 142.0 mm, vias 0 -> 4
- net I2C-SCL-MAIN: track 0.00 -> 121.1 mm, vias 0 -> 5
- net 3.3v: track 77.7 -> 72.4 mm
- net I2C-SLC-MAIN: track 4.85 -> 0.00 mm
- net I2C-MAIN-RESET: track 31.1 -> 32.9 mm, vias 0 -> 1
- net IIM-MAIN-INT: track 33.3 -> 34.6 mm, vias 1 -> 3
- net Net-(U4-CAP): track 2.93 -> 4.04 mm
- net Net-(U1-V+): track 8.31 -> 8.82 mm

Commit message: uhhh idk i got the same color wires over each other for fun ig
Parts:
- moved U2 127.0 mm to (160.0, 135.1), turned to -110 degrees
- moved U11 106.0 mm to (155.9, 120.4), turned to -155 degrees
- moved L1 101.9 mm to (162.3, 119.8), turned to 160 degrees
- moved IC1 101.8 mm to (159.1, 118.8), turned to 25 degrees
- moved E1 97.5 mm to (173.9, 119.2), turned to -110 degrees
- moved C6 96.4 mm to (158.8, 115.2), turned to 25 degrees
- moved R8 95.9 mm to (155.6, 113.6), turned to -155 degrees
- moved R7 92.6 mm to (158.0, 112.5), turned to -155 degrees
- moved C12 8.07 mm to (140.0, 68.8)
- moved C13 8.07 mm to (148.2, 123.8)
- moved C14 8.07 mm to (142.0, 68.7)
- moved C15 8.07 mm to (146.1, 123.5)
- moved C17 8.07 mm to (142.9, 123.5)
- moved R19 8.07 mm to (138.4, 110.7)
- moved R20 8.07 mm to (138.7, 83.2)
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Connections:
- J2 pad 17: A -> Y
- J2 pad 18: B -> Z
- J2 pad 21: X -> B
- J2 pad 22: Y -> A
Routing:
- net 3.3v: track 72.4 -> 227.9 mm, vias 5 -> 17
- net I2C-SCL-MAIN: track 121.1 -> 77.8 mm
- net I2C-SDA-MAIN: track 142.0 -> 103.4 mm, vias 4 -> 3
- net I2C-MAIN-RESET: track 32.9 -> 19.1 mm, vias 1 -> 3
- net IIM-MAIN-INT: track 34.6 -> 22.0 mm, vias 3 -> 1
- net INT1-BMI: track 20.0 -> 17.4 mm
- net INT2-BMI: track 14.9 -> 14.0 mm
Other:
- copper layers 2 -> 4

Commit message: uhhhhhhhh idk
Parts:
- removed R10, R11, R12, R9: 4.7k, RC0402FR:YAG_R0402_YAG
- removed R5: 5K, CRCW08055K00FKTA:RESC2012X50N
- moved L1 13.2 mm to (157.2, 107.7), turned to 170 degrees
- moved E1 11.3 mm to (166.2, 110.9), turned to -100 degrees
- moved IC1 11.0 mm to (153.9, 109.1), turned to 35 degrees
- moved U11 11.0 mm to (151.2, 110.5), turned to -145 degrees
- moved C6 10.3 mm to (152.8, 106.8), turned to 35 degrees
- moved U2 9.32 mm to (158.4, 125.9), turned to -100 degrees
- moved R7 9.24 mm to (152.6, 105.0), turned to -145 degrees
- moved R8 8.92 mm to (150.5, 106.3), turned to -145 degrees
- moved C1 2.22 mm to (157.3, 74.5)
- moved R6 2.20 mm to (163.4, 100.7)
Connections:
- J2 pad 38: unconnected-(J2-Pin_38-Pad38) -> TXD
- J2 pad 40: unconnected-(J2-Pin_40-Pad40) -> RDX
- U2 pad 20: unconnected-(U2-TXD/SPI_MISO-Pad20) -> TXD
- U2 pad 21: unconnected-(U2-RXD/SPI_MOSI-Pad21) -> RDX
Routing:
- net TXD: track 0.00 -> 39.3 mm, vias 0 -> 1
- net RDX: track 0.00 -> 35.4 mm, vias 0 -> 1
- net 3.3v: track 227.9 -> 217.5 mm, vias 17 -> 14
- net Net-(U11-RF_OUT): track 18.1 -> 22.4 mm
- net Net-(U1-V+): track 8.82 -> 5.42 mm
- net I2C-SCL-MAIN: track 77.8 -> 80.8 mm
- net I2C-SDA-MAIN: track 103.4 -> 101.6 mm
- net Net-(U3-SDO): track 4.74 -> 3.28 mm
- net Net-(IC1-VCC): track 7.50 -> 6.34 mm
- net Net-(E1-Pad1): track 9.23 -> 8.51 mm
- net INT1-BMI: track 17.4 -> 18.0 mm
- net Net-(IC1-RF_IN): track 2.24 -> 2.78 mm
