File: KiCad/Commodore 7/I2C Buffer.kicad_sch (KiCad schematic)
At the start: 2 parts

Commit message: beep beep beep placed
Parts:
- gave numbers to parts that had none: 1
- renumbered 10K to 10K1
Changed lines of the file:
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@@
 		(on_board yes)
 		(dnp no)
-		(property "Reference" "U?"
+		(property "Reference" "U6"
 			(at 137.414 85.598 0)
 			(effects
@@
 			(project ""
 				(path "/42cf917d-ec14-4557-b98d-6a3f3b8cf25c/87bcbd75-d39f-4349-beeb-9080787b8c18"
-					(reference "U?")
+					(reference "U6")
 					(unit 1)
 				)
@@
 		(on_board yes)
 		(dnp no)
-		(property "Reference" "10K"
+		(property "Reference" "10K1"
 			(at 162.814 107.696 90)
 			(effects
@@
 			(project ""
 				(path "/42cf917d-ec14-4557-b98d-6a3f3b8cf25c/87bcbd75-d39f-4349-beeb-9080787b8c18"
-					(reference "10K")
+					(reference "10K1")
 					(unit 1)
 				)

Commit message: TRANSWHATEVER
Other:
- note added: "Connect at diffrent points"
Changed lines of the file:
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@@
 	(generator_version "9.0")
 	(paper "A4")
+	(text "Connect at diffrent points\n"
+		(exclude_from_sim no)
+		(at 137.922 109.728 0)
+		(effects
+			(font
+				(size 1.27 1.27)
+			)
+		)
+	)
 	(wire
 		(pts

Commit message: uhhhhhhhh idk
Parts:
- U6: footprint DGK8 -> TCA9509DGKR:DGK8
Changed lines of the file:
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@@
 			)
 		)
-		(property "Footprint" "DGK8"
+		(property "Footprint" "TCA9509DGKR:DGK8"
 			(at 120.65 95.25 0)
 			(effects

Commit message: i sitll got mroe to do ssry yall
Parts:
- removed 10K1: R, symbol Device:R
- added R9: RC0402FR-0710KL, RC0402FR:YAG_R0402_YAG, symbol RC0402FR-0710KL:RC0402FR-0710KL
Connections:
- net at U6.5 (EN): now also R9.1
- net +3.3V renamed 3.3v
- net 3.3v: now also R9.2
- net I2C_SCL renamed I2C-SCL-MAIN
- net I2C_SDA renamed I2C-SDA-MAIN
