File: KiCad/Commodore 7/BMI270.kicad_sch (KiCad schematic)
At the start: 6 parts, among them U3 BMI270 - Secondary Accelerome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

Commit message: deleteeeeeeeeee
Parts:
- removed R7, R8: 2.7K, CRG0805F2K7:RES0805_CRG_TYCO_TYC, symbol 2025-10-06_20-52-39:CRG0805F2K7
Connections:
- net I2C-SCL-MAIN is gone; now on net 3.3v: U3.13 (SCX)
- net I2C-SDA-MAIN is gone; now on net 3.3v: U3.14 (SDX)
Changed lines of the file:
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@@
 	(wire
 		(pts
-			(xy 104.14 64.77) (xy 90.17 64.77)
+			(xy 90.17 64.77) (xy 152.4 64.77)
 		)
 		(stroke
@@
 	(wire
 		(pts
-			(xy 116.84 64.77) (xy 152.4 64.77)
-		)
-		(stroke
-			(width 0)
-			(type default)
-		)
-	)
-	(wire
-		(pts
 			(xy 154.94 120.65) (xy 154.94 118.11)
 		)
@@
 	(wire
 		(pts
-			(xy 115.57 69.85) (xy 95.25 69.85)
+			(xy 95.25 69.85) (xy 147.32 69.85)
 		)
 		(stroke
@@
 		(pts
 			(xy 152.4 85.09) (xy 156.21 85.09)
-		)
-		(stroke
-			(width 0)
-			(type default)
-		)
-	)
-	(wire
-		(pts
-			(xy 128.27 69.85) (xy 147.32 69.85)
 		)
 		(stroke
@@
 	)
 	(symbol
-		(lib_id "2025-10-06_20-52-39:CRG0805F2K7")
-		(at 104.14 64.77 0)
-		(unit 1)
-		(exclude_from_sim no)
-		(in_bom yes)
-		(on_board yes)
-		(dnp no)
-		(fields_autoplaced yes)
-		(property "Reference" "R7"
-			(at 110.49 58.42 0)
-			(effects
-				(font
-					(size 1.524 1.524)
-				)
-			)
-		)
-		(property "Value" "2.7K"
-			(at 110.49 60.96 0)
-			(effects
-				(font
-					(size 1.524 1.524)
-				)
-			)
-		)
-		(property "Footprint" "CRG0805F2K7:RES0805_CRG_TYCO_TYC"
-			(at 104.14 64.77 0)
-			(effects
-				(font
-					(size 1.27 1.27)
-					(italic yes)
-				)
-				(hide yes)
-			)
-		)
-		(property "Datasheet" "https://www.te.com/commerce/DocumentDelivery/DDEController?Action=srchrtrv&DocNm=1773204&DocType=Data+Sheet&DocLang=English&PartCntxt=1623181-1&DocFormat=pdf"
-			(at 104.14 64.77 0)
-			(effects
-				(font
-					(size 1.27 1.27)
-					(italic yes)
-				)
-				(hide yes)
-			)
-		)
-		(property "Description" ""
-			(at 104.14 64.77 0)
-			(effects
-				(font
-					(size 1.27 1.27)
-				)
-				(hide yes)
-			)
-		)
-		(pin "1"
-		)
-		(pin "2"
-		)
-		(instances
-			(project "Commodore 7"
-				(path "/42cf917d-ec14-4557-b98d-6a3f3b8cf25c/5957d6f3-67b6-46f3-b569-ac79090e2ab1"
-					(reference "R7")
-					(unit 1)
-				)
-			)
-		)
-	)
-	(symbol
 		(lib_id "power:GNDD")
 		(at 111.76 92.71 180)
@@
 					(unit 1)
 				)
-			)
-		)
-	)
-	(symbol
-		(lib_id "2025-10-06_20-52-39:CRG0805F2K7")
-		(at 115.57 69.85 0)
-		(unit 1)
-		(exclude_from_sim no)
-		(in_bom yes)
-		(on_board yes)
-		(dnp no)
-		(property "Reference" "R8"
-			(at 122.174 74.168 0)
-			(effects
-				(font
-					(size 1.524 1.524)
-				)
-			)
-		)
-		(property "Value" "2.7K"
-			(at 121.666 72.136 0)
-			(effects
-				(font
-					(size 1.524 1.524)
-				)
-			)
-		)
-		(property "Footprint" "CRG0805F2K7:RES0805_CRG_TYCO_TYC"
-			(at 115.57 69.85 0)
-			(effects
-				(font
-					(size 1.27 1.27)
-					(italic yes)
-				)
-				(hide yes)
-			)
-		)
-		(property "Datasheet" "https://www.te.com/commerce/DocumentDelivery/DDEController?Action=srchrtrv&DocNm=1773204&DocType=Data+Sheet&DocLang=English&PartCntxt=1623181-1&DocFormat=pdf"
-			(at 115.57 69.85 0)
-			(effects
-				(font
-					(size 1.27 1.27)
-					(italic yes)
-				)
-				(hide yes)
-			)
-		)
-		(property "Description" ""
-			(at 115.57 69.85 0)
-			(effects
-				(font
-					(size 1.27 1.27)
-				)
-				(hide yes)
-			)
-		)
-		(pin "1"
-		)
-		(pin "2"
-		)
-		(instances
-			(project "Commodore 7"
-				(path "/42cf917d-ec14-4557-b98d-6a3f3b8cf25c/5957d6f3-67b6-46f3-b569-ac79090e2ab1"
-					(reference "R8")
-					(unit 1)
-				)

Commit message: uhhhh didnt do as much as i shoulve mb gang
Connections:
- net 3.3v: now also C2.1; no longer C2.2
- net GNDD: now also C2.2; no longer C2.1
Other:
- moved on the sheet: C2
Changed lines of the file:
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@@
+	(wire
+		(pts
+			(xy 162.56 118.11) (xy 162.56 97.79)
+		)
+		(stroke
+			(width 0)
+			(type default)
+		)
+	)
 	(wire
 		(pts
@@
 		(pts
 			(xy 147.32 85.09) (xy 152.4 85.09)
-		)
-		(stroke
-			(width 0)
-			(type default)
-		)
-	)
-	(wire
-		(pts
-			(xy 162.56 97.79) (xy 162.56 118.11)
 		)
 		(stroke
@@
 	(symbol
 		(lib_id "2025-10-06_19-12-57:CC0603KRX7R7BB104")
-		(at 162.56 97.79 90)
+		(at 162.56 90.17 270)
 		(unit 1)
 		(exclude_from_sim no)
@@
 		(dnp no)
 		(property "Reference" "C2"
-			(at 163.576 91.186 90)
+			(at 161.544 96.774 90)
 			(effects
 				(font
@@
 		)
 		(property "Value" ".1uF"
-			(at 164.338 95.758 90)
+			(at 160.782 92.202 90)
 			(effects
 				(font
@@
 		)
 		(property "Footprint" "CC0603KRXQRQBB104:CC0603N_YAG"
-			(at 162.56 97.79 0)
+			(at 162.56 90.17 0)
 			(effects
 				(font
@@
 		)
 		(property "Datasheet" "CC0603KRX7R7BB104"
-			(at 162.56 97.79 0)
+			(at 162.56 90.17 0)
 			(effects
 				(font
@@
 		)
 		(property "Description" ""
-			(at 162.56 97.79 0)
-			(effects
-				(font
+			(at 162.56 90.17 0)
+			(effects
+				(font

Commit message: oh wow
Connections:
- net 3.3v: no longer U3.13 (SCX), U3.14 (SDX)
- new net I2C-SCL-MAIN: U3.13 (SCX)
- new net I2C-SDA-MAIN: U3.14 (SDX)
Changed lines of the file:
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@@
-	)
-	(junction
-		(at 90.17 100.33)
-		(diameter 0)
-		(color 0 0 0 0)
 	)
 	(junction
@@
 		(color 0 0 0 0)
 	)
-	(junction
-		(at 95.25 102.87)
-		(diameter 0)
-		(color 0 0 0 0)
-	)
 	(wire
 		(pts
@@
 	(wire
 		(pts
-			(xy 95.25 102.87) (xy 111.76 102.87)
+			(xy 86.36 102.87) (xy 111.76 102.87)
 		)
 		(stroke
@@
 	(wire
 		(pts
-			(xy 86.36 102.87) (xy 95.25 102.87)
-		)
-		(stroke
-			(width 0)
-			(type default)
-		)
-	)
-	(wire
-		(pts
 			(xy 90.17 64.77) (xy 152.4 64.77)
 		)
@@
 	(wire
 		(pts
-			(xy 86.36 100.33) (xy 90.17 100.33)
-		)
-		(stroke
-			(width 0)
-			(type default)
-		)
-	)
-	(wire
-		(pts
 			(xy 161.29 120.65) (xy 154.94 120.65)
 		)
@@
 	(wire
 		(pts
-			(xy 90.17 64.77) (xy 90.17 100.33)
-		)
-		(stroke
-			(width 0)
-			(type default)
-		)
-	)
-	(wire
-		(pts
 			(xy 147.32 69.85) (xy 147.32 85.09)
 		)
@@
 	(wire
 		(pts
-			(xy 90.17 100.33) (xy 111.76 100.33)
+			(xy 86.36 100.33) (xy 111.76 100.33)
 		)
 		(stroke
@@
 		)
 		(stroke
-			(width 0)
-			(type default)
-		)
-	)
-	(wire
-		(pts
-			(xy 95.25 69.85) (xy 95.25 102.87)
-		)
-		(stroke

Commit message: uhhhhhh theres a lot of vias oh well
Parts:
- added R10, R9: 4.7k, YAG_R0402_YAG, symbol RC0402FR:RC0402FR-074K7L
Connections:
- net 3.3v: now also R10.1, R9.1
- net I2C-SCL-MAIN: now also R9.2
- net I2C-SDA-MAIN: now also R10.2
Changed lines of the file:
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@@
+	)
+	(junction
+		(at 90.17 100.33)
+		(diameter 0)
+		(color 0 0 0 0)
 	)
 	(junction
@@
 	)
 	(junction
+		(at 95.25 102.87)
+		(diameter 0)
+		(color 0 0 0 0)
+	)
+	(junction
 		(at 156.21 85.09)
 		(diameter 0)
@@
 	(wire
 		(pts
-			(xy 86.36 102.87) (xy 111.76 102.87)
+			(xy 86.36 102.87) (xy 95.25 102.87)
 		)
 		(stroke
@@
 	(wire
 		(pts
+			(xy 90.17 100.33) (xy 111.76 100.33)
+		)
+		(stroke
+			(width 0)
+			(type default)
+		)
+	)
+	(wire
+		(pts
+			(xy 95.25 82.55) (xy 95.25 102.87)
+		)
+		(stroke
+			(width 0)
+			(type default)
+		)
+	)
+	(wire
+		(pts
+			(xy 95.25 102.87) (xy 111.76 102.87)
+		)
+		(stroke
+			(width 0)
+			(type default)
+		)
+	)
+	(wire
+		(pts
 			(xy 142.24 87.63) (xy 146.05 87.63)
 		)
@@
 	(wire
 		(pts
+			(xy 90.17 77.47) (xy 90.17 100.33)
+		)
+		(stroke
+			(width 0)
+			(type default)
+		)
+	)
+	(wire
+		(pts
 			(xy 175.26 104.14) (xy 175.26 127)
 		)
@@
 	(wire
 		(pts
-			(xy 86.36 100.33) (xy 111.76 100.33)
+			(xy 86.36 100.33) (xy 90.17 100.33)
 		)
 		(stroke
@@
 				(justify right)
 				(hide yes)
+			)
+		)
+	)
+	(symbol
+		(lib_id "RC0402FR:RC0402FR-074K7L")
+		(at 90.17 64.77 270)
+		(unit 1)
+		(exclude_from_sim no)
+		(in_bom yes)
+		(on_board yes)
+		(dnp no)
+		(property "Reference" "R9"
+			(at 84.836 68.072 90)
+			(effects
+				(font
+					(size 1.524 1.524)
+				)
+				(justify left)
+			)
+		)
+		(property "Value" "4.7k"
+			(at 83.82 71.12 90)
+			(effects
+				(font
+					(size 1.524 1.524)
+				)
+				(justify left)
+			)
+		)
+		(property "Footprint" "YAG_R0402_YAG"
+			(at 90.17 64.77 0)
+			(effects
+				(font
+					(size 1.27 1.27)
+					(italic yes)
+				)
+				(hide yes)
+			)
+		)
+		(property "Datasheet" "RC0402FR-074K7L"
+			(at 90.17 64.77 0)
+			(effects
+				(font
+					(size 1.27 1.27)
+					(italic yes)
+				)
+				(hide yes)
+			)
+		)
+		(property "Description" ""
+			(at 90.17 64.77 0)
+			(effects
+				(font
+					(size 1.27 1.27)
+				)
+				(hide yes)
+			)
+		)
+		(pin "2"
+		)
+		(pin "1"
+		)
+		(instances
+			(project ""
+				(path "/42cf917d-ec14-4557-b98d-6a3f3b8cf25c/5957d6f3-67b6-46f3-b569-ac79090e2ab1"
+					(reference "R9")
+					(unit 1)
+				)
 			)
 		)
@@
 					(unit 1)
 				)
+			)
+		)
+	)
+	(symbol
+		(lib_id "RC0402FR:RC0402FR-074K7L")
+		(at 95.25 69.85 270)
+		(unit 1)
+		(exclude_from_sim no)
+		(in_bom yes)
+		(on_board yes)
+		(dnp no)
+		(property "Reference" "R10"
+			(at 97.79 71.882 90)
+			(effects
+				(font
+					(size 1.524 1.524)
+				)
+				(justify left)
+			)
+		)
+		(property "Value" "4.7k"
+			(at 97.79 74.676 90)
+			(effects
+				(font
+					(size 1.524 1.524)
+				)
+				(justify left)
+			)
+		)
+		(property "Footprint" "YAG_R0402_YAG"
+			(at 95.25 69.85 0)
+			(effects
+				(font
+					(size 1.27 1.27)
+					(italic yes)
+				)
+				(hide yes)
+			)
+		)
+		(property "Datasheet" "RC0402FR-074K7L"
+			(at 95.25 69.85 0)
+			(effects
+				(font
+					(size 1.27 1.27)
+					(italic yes)
+				)
+				(hide yes)
+			)
+		)
+		(property "Description" ""
+			(at 95.25 69.85 0)
+			(effects
+				(font
+					(size 1.27 1.27)
+				)
+				(hide yes)
+			)
+		)
+		(pin "2"
+		)
+		(pin "1"
+		)
+		(instances
+			(project ""
+				(path "/42cf917d-ec14-4557-b98d-6a3f3b8cf25c/5957d6f3-67b6-46f3-b569-ac79090e2ab1"
+					(reference "R10")
+					(unit 1)
+				)

Commit message: uhhhhhhhh idk
Parts:
- removed R10, R9: 4.7k, YAG_R0402_YAG, symbol RC0402FR:RC0402FR-074K7L

Commit message: holy
Parts:
- added R8: 2.7K, Resistor_SMD:R_1206_3216Metric, symbol 2025-10-06_20-52-39:CRG0805F2K7
Connections:
- net 3.3v: now also R8.1; no longer U3.12 (CSB)
- new net: R8.2, U3.12 (CSB)
Changed lines of the file:
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@@
+	(wire
+		(pts
+			(xy 119.38 76.2) (xy 144.78 76.2)
+		)
+		(stroke
+			(width 0)
+			(type default)
+		)
+	)
 	(wire
 		(pts
@@
 	(wire
 		(pts
-			(xy 101.6 76.2) (xy 144.78 76.2)
+			(xy 101.6 76.2) (xy 106.68 76.2)
 		)
 		(stroke
@@
 					(unit 1)
 				)
+			)
+		)
+	)
+	(symbol
+		(lib_id "2025-10-06_20-52-39:CRG0805F2K7")
+		(at 106.68 76.2 0)
+		(unit 1)
+		(exclude_from_sim no)
+		(in_bom yes)
+		(on_board yes)
+		(dnp no)
+		(fields_autoplaced yes)
+		(property "Reference" "R8"
+			(at 113.03 69.85 0)
+			(effects
+				(font
+					(size 1.524 1.524)
+				)
+			)
+		)
+		(property "Value" "2.7K"
+			(at 113.03 72.39 0)
+			(effects
+				(font
+					(size 1.524 1.524)
+				)
+			)
+		)
+		(property "Footprint" "Resistor_SMD:R_1206_3216Metric"
+			(at 106.68 76.2 0)
+			(effects
+				(font
+					(size 1.27 1.27)
+					(italic yes)
+				)
+				(hide yes)
+			)
+		)
+		(property "Datasheet" "https://www.te.com/commerce/DocumentDelivery/DDEController?Action=srchrtrv&DocNm=1773204&DocType=Data+Sheet&DocLang=English&PartCntxt=1623181-1&DocFormat=pdf"
+			(at 106.68 76.2 0)
+			(effects
+				(font
+					(size 1.27 1.27)
+					(italic yes)
+				)
+				(hide yes)
+			)
+		)
+		(property "Description" ""
+			(at 106.68 76.2 0)
+			(effects
+				(font
+					(size 1.27 1.27)
+				)
+				(hide yes)
+			)
+		)
+		(pin "1"
+		)
+		(pin "2"
+		)
+		(instances
+			(project "Commodore 7"
+				(path "/42cf917d-ec14-4557-b98d-6a3f3b8cf25c/5957d6f3-67b6-46f3-b569-ac79090e2ab1"
+					(reference "R8")
+					(unit 1)
+				)
