File: KiCad/Commodore 7/Transceiver.kicad_sch (KiCad schematic)
At the start: 1 part

Commit message: hi!!!!!
Parts:
- gave numbers to parts that had none: 1
Changed lines of the file:
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@@
 		(on_board yes)
 		(dnp no)
-		(property "Reference" "U?"
+		(property "Reference" "U7"
 			(at 60.96 34.29 0)
 			(effects
@@
 			(project ""
 				(path "/42cf917d-ec14-4557-b98d-6a3f3b8cf25c/94b03863-4f6c-4232-bb6c-dbc8fe3a9ec0"
-					(reference "U?")
+					(reference "U7")
 					(unit 1)
 				)

Commit message: uhhhhhhhh idk
Parts:
- U7: footprint D8_TEX -> 2N65HVD74DR:D8_TEX
Changed lines of the file:
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@@
 			)
 		)
-		(property "Footprint" "D8_TEX"
+		(property "Footprint" "2N65HVD74DR:D8_TEX"
 			(at 40.64 44.45 0)
 			(effects

Commit message: i sitll got mroe to do ssry yall
Parts:
- added R10, R5: RMCF1206JT68K0, Resistor_SMD:R_1206_3216Metric, symbol RMCF1206JT68K0:RMCF1206JT68K0
Connections:
- net R: now reaches U7.2 (R)
- net T: now reaches U7.3 (D)
- net A: now reaches U7.5 (Y)
- net A: now also R10.1
- net B: now reaches U7.6 (Z)
- net B: now also R10.2
- net Z: now reaches U7.7 (B)
- net Z: now also R5.1
- net Y: now reaches U7.8 (A)
- net Y: now also R5.2
- net +3.3V renamed 3.3v
Other:
- moved on the sheet: U7

Commit message: uhhhhhh i think its almost done now?
Parts:
- removed R10, R5: RMCF1206JT68K0, Resistor_SMD:R_1206_3216Metric, symbol RMCF1206JT68K0:RMCF1206JT68K0
- added R5, R7: RC1206FR-0724RL, Resistor_SMD:R_1206_3216Metric, symbol RC1206FR-0724RL:RC1206FR-0724RL
Connections:
- net A renamed a+
- net a+: now also R7.1
- net B renamed a-
- net a-: now also R7.2
- net Y renamed y+
- net y+: now also R5.1
- net Z renamed y-
- net y-: now also R5.2
Changed lines of the file:
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@@
 	(wire
 		(pts
-			(xy 102.87 43.18) (xy 110.49 43.18)
+			(xy 102.87 43.18) (xy 116.84 43.18)
+		)
+		(stroke
+			(width 0)
+			(type default)
+		)
+	)
+	(wire
+		(pts
+			(xy 99.06 54.61) (xy 109.22 54.61)
 		)
 		(stroke
@@
 	(wire
 		(pts
-			(xy 83.82 30.48) (xy 110.49 30.48)
+			(xy 116.84 48.26) (xy 121.92 48.26)
+		)
+		(stroke
+			(width 0)
+			(type default)
+		)
+	)
+	(wire
+		(pts
+			(xy 83.82 30.48) (xy 121.92 30.48)
+		)
+		(stroke
+			(width 0)
+			(type default)
+		)
+	)
+	(wire
+		(pts
+			(xy 116.84 43.18) (xy 116.84 48.26)
 		)
 		(stroke
@@
 	(wire
 		(pts
+			(xy 121.92 30.48) (xy 121.92 27.94)
+		)
+		(stroke
+			(width 0)
+			(type default)
+		)
+	)
+	(wire
+		(pts
 			(xy 43.18 52.07) (xy 40.64 52.07)
 		)
@@
 	(wire
 		(pts
+			(xy 99.06 77.47) (xy 109.22 77.47)
+		)
+		(stroke
+			(width 0)
+			(type default)
+		)
+	)
+	(wire
+		(pts
+			(xy 99.06 67.31) (xy 99.06 77.47)
+		)
+		(stroke
+			(width 0)
+			(type default)
+		)
+	)
+	(wire
+		(pts
+			(xy 109.22 54.61) (xy 109.22 57.15)
+		)
+		(stroke
+			(width 0)
+			(type default)
+		)
+	)
+	(wire
+		(pts
 			(xy 83.82 49.53) (xy 99.06 49.53)
 		)
@@
 		)
 	)
-	(global_label "Z"
+	(global_label "y-"
 		(shape input)
 		(at 102.87 45.72 0)
@@
 		)
 		(property "Intersheetrefs" "${INTERSHEET_REFS}"
-			(at 107.0647 45.72 0)
+			(at 108.3952 45.72 0)
 			(effects
 				(font
@@
 		)
 	)
-	(global_label "B"
+	(global_label "a-"
 		(shape input)
 		(at 99.06 52.07 0)
@@
 		)
 		(property "Intersheetrefs" "${INTERSHEET_REFS}"
-			(at 103.3152 52.07 0)
+			(at 104.7666 52.07 0)
 			(effects
 				(font
@@
 		)
 	)
-	(global_label "Y"
+	(global_label "y+"
 		(shape input)
 		(at 88.9 30.48 90)
@@
 		)
 		(property "Intersheetrefs" "${INTERSHEET_REFS}"
-			(at 88.9 26.4062 90)
+			(at 88.9 24.9548 90)
 			(effects
 				(font
@@
 		)
 	)
-	(global_label "A"
+	(global_label "a+"
 		(shape input)
 		(at 90.17 67.31 270)
@@
 		)
 		(property "Intersheetrefs" "${INTERSHEET_REFS}"
-			(at 90.17 71.3838 90)
-			(effects
-				(font
-					(size 1.27 1.27)
-				)
-				(justify right)
-				(hide yes)
-			)
-		)
-	)
-	(symbol
-		(lib_id "RMCF1206JT68K0:RMCF1206JT68K0")
-		(at 99.06 67.31 90)
-		(unit 1)
-		(exclude_from_sim no)
-		(in_bom yes)
-		(on_board yes)
-		(dnp no)
-		(fields_autoplaced yes)
-		(property "Reference" "R10"
-			(at 101.6 59.6899 90)
-			(effects
-				(font
-					(size 1.524 1.524)
-				)
-				(justify right)
-			)
-		)
-		(property "Value" "RMCF1206JT68K0"
-			(at 101.6 62.2299 90)
-			(effects
-				(font
-					(size 1.524 1.524)
-				)
-				(justify right)
-			)
-		)
-		(property "Footprint" "Resistor_SMD:R_1206_3216Metric"
-			(at 99.06 67.31 0)
-			(effects
-				(font
-					(size 1.27 1.27)
-					(italic yes)
-				)
-				(hide yes)
-			)
-		)
-		(property "Datasheet" "RMCF1206JT68K0"
-			(at 99.06 67.31 0)
-			(effects
-				(font
-					(size 1.27 1.27)
-					(italic yes)
-				)
-				(hide yes)
-			)
-		)
-		(property "Description" ""
-			(at 99.06 67.31 0)
-			(effects
-				(font
-					(size 1.27 1.27)
-				)
-				(hide yes)
-			)
-		)
-		(pin "2"
-		)
-		(pin "1"
-		)
-		(instances
-			(project "Commodore 7"
-				(path "/42cf917d-ec14-4557-b98d-6a3f3b8cf25c/94b03863-4f6c-4232-bb6c-dbc8fe3a9ec0"
-					(reference "R10")
-					(unit 1)
-				)
-			)
-		)
-	)
-	(symbol
-		(lib_id "RMCF1206JT68K0:RMCF1206JT68K0")
-		(at 110.49 43.18 90)
-		(unit 1)
-		(exclude_from_sim no)
-		(in_bom yes)
-		(on_board yes)
-		(dnp no)
-		(fields_autoplaced yes)
-		(property "Reference" "R5"
-			(at 113.03 35.5599 90)
-			(effects
-				(font
-					(size 1.524 1.524)
-				)
-				(justify right)
-			)
-		)
-		(property "Value" "RMCF1206JT68K0"
-			(at 113.03 38.0999 90)
-			(effects
-				(font
-					(size 1.524 1.524)
-				)
-				(justify right)
-			)
-		)
-		(property "Footprint" "Resistor_SMD:R_1206_3216Metric"
-			(at 110.49 43.18 0)
-			(effects
-				(font
-					(size 1.27 1.27)
-					(italic yes)
-				)
-				(hide yes)
-			)
-		)
-		(property "Datasheet" "RMCF1206JT68K0"
-			(at 110.49 43.18 0)
-			(effects
-				(font
-					(size 1.27 1.27)
-					(italic yes)
-				)
-				(hide yes)
-			)
-		)
-		(property "Description" ""
-			(at 110.49 43.18 0)
-			(effects
-				(font
-					(size 1.27 1.27)
-				)
-				(hide yes)
-			)
-		)
-		(pin "2"
-		)
-		(pin "1"
-		)
-		(instances
-			(project ""
-				(path "/42cf917d-ec14-4557-b98d-6a3f3b8cf25c/94b03863-4f6c-4232-bb6c-dbc8fe3a9ec0"
-					(reference "R5")
-					(unit 1)
-				)
+			(at 90.17 73.0166 90)
+			(effects
+				(font
+					(size 1.27 1.27)
+				)
+				(justify right)
+				(hide yes)
 			)
 		)
@@
 	)
 	(symbol
+		(lib_id "RC1206FR-0724RL:RC1206FR-0724RL")
+		(at 121.92 38.1 270)
+		(unit 1)
+		(exclude_from_sim no)
+		(in_bom yes)
+		(on_board yes)
+		(dnp no)
+		(fields_autoplaced yes)
+		(property "Reference" "R5"
+			(at 125.73 36.8299 90)
+			(effects
+				(font
+					(size 1.27 1.27)
+				)
+				(justify left)
+			)
+		)
+		(property "Value" "RC1206FR-0724RL"
+			(at 125.73 39.3699 90)
+			(effects
+				(font
+					(size 1.27 1.27)
+				)
+				(justify left)
+			)
+		)
+		(property "Footprint" "Resistor_SMD:R_1206_3216Metric"
+			(at 121.92 38.1 0)
+			(effects
+				(font
+					(size 1.27 1.27)
+				)
+				(justify bottom)
+				(hide yes)
+			)
+		)
+		(property "Datasheet" ""
+			(at 121.92 38.1 0)
+			(effects
+				(font
+					(size 1.27 1.27)
+				)
+				(hide yes)
+			)
+		)
+		(property "Description" ""
+			(at 121.92 38.1 0)
+			(effects
+				(font
+					(size 1.27 1.27)
+				)
+				(hide yes)
+			)
+		)
+		(pin "1"
+		)
+		(pin "2"
+		)
+		(instances
+			(project ""
+				(path "/42cf917d-ec14-4557-b98d-6a3f3b8cf25c/94b03863-4f6c-4232-bb6c-dbc8fe3a9ec0"
+					(reference "R5")
+					(unit 1)
+				)
+			)
+		)
+	)
+	(symbol
 		(lib_id "power:GNDD")
 		(at 40.64 52.07 270)
@@
 					(unit 1)
 				)
+			)
+		)
+	)
+	(symbol
+		(lib_id "RC1206FR-0724RL:RC1206FR-0724RL")
+		(at 109.22 67.31 90)
+		(unit 1)
+		(exclude_from_sim no)
+		(in_bom yes)
+		(on_board yes)
+		(dnp no)
+		(fields_autoplaced yes)
+		(property "Reference" "R7"
+			(at 113.03 66.0399 90)
+			(effects
+				(font
+					(size 1.27 1.27)
+				)
+				(justify right)
+			)
+		)
+		(property "Value" "RC1206FR-0724RL"
+			(at 113.03 68.5799 90)
+			(effects
+				(font
+					(size 1.27 1.27)
+				)
+				(justify right)
+			)
+		)
+		(property "Footprint" "Resistor_SMD:R_1206_3216Metric"
+			(at 109.22 67.31 0)
+			(effects
+				(font
+					(size 1.27 1.27)
+				)
+				(justify bottom)
+				(hide yes)
+			)
+		)
+		(property "Datasheet" ""
+			(at 109.22 67.31 0)
+			(effects
+				(font
+					(size 1.27 1.27)
+				)
+				(hide yes)
+			)
+		)
+		(property "Description" ""
+			(at 109.22 67.31 0)
+			(effects
+				(font
+					(size 1.27 1.27)
+				)
+				(hide yes)
+			)
+		)
+		(pin "1"
+		)
+		(pin "2"
+		)
+		(instances
+			(project ""
+				(path "/42cf917d-ec14-4557-b98d-6a3f3b8cf25c/94b03863-4f6c-4232-bb6c-dbc8fe3a9ec0"
+					(reference "R7")
+					(unit 1)
+				)

Commit message: holy
Connections:
- net a+: now also R5.1, U7.8 (A); no longer R7.1, U7.5 (Y)
- net a-: now also R5.2, U7.7 (B); no longer R7.2, U7.6 (Z)
- net y+: now also R7.1, U7.5 (Y); no longer R5.1, U7.8 (A)
- net y-: now also R7.2, U7.6 (Z); no longer R5.2, U7.7 (B)
Other:
- moved on the sheet: R5, R7
Changed lines of the file:
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@@
 	(wire
 		(pts
-			(xy 102.87 43.18) (xy 116.84 43.18)
-		)
-		(stroke
-			(width 0)
-			(type default)
-		)
-	)
-	(wire
-		(pts
-			(xy 99.06 54.61) (xy 109.22 54.61)
-		)
-		(stroke
-			(width 0)
-			(type default)
-		)
-	)
-	(wire
-		(pts
-			(xy 102.87 43.18) (xy 102.87 46.99)
-		)
-		(stroke
-			(width 0)
-			(type default)
-		)
-	)
-	(wire
-		(pts
-			(xy 116.84 48.26) (xy 121.92 48.26)
-		)
-		(stroke
-			(width 0)
-			(type default)
-		)
-	)
-	(wire
-		(pts
-			(xy 83.82 30.48) (xy 121.92 30.48)
-		)
-		(stroke
-			(width 0)
-			(type default)
-		)
-	)
-	(wire
-		(pts
-			(xy 116.84 43.18) (xy 116.84 48.26)
-		)
-		(stroke
-			(width 0)
-			(type default)
-		)
-	)
-	(wire
-		(pts
-			(xy 83.82 44.45) (xy 83.82 30.48)
-		)
-		(stroke
-			(width 0)
-			(type default)
-		)
-	)
-	(wire
-		(pts
-			(xy 99.06 49.53) (xy 99.06 54.61)
-		)
-		(stroke
-			(width 0)
-			(type default)
-		)
-	)
-	(wire
-		(pts
-			(xy 121.92 30.48) (xy 121.92 27.94)
+			(xy 85.09 44.45) (xy 83.82 44.45)
+		)
+		(stroke
+			(width 0)
+			(type default)
+		)
+	)
+	(wire
+		(pts
+			(xy 93.98 46.99) (xy 83.82 46.99)
+		)
+		(stroke
+			(width 0)
+			(type default)
+		)
+	)
+	(wire
+		(pts
+			(xy 85.09 25.4) (xy 93.98 25.4)
+		)
+		(stroke
+			(width 0)
+			(type default)
+		)
+	)
+	(wire
+		(pts
+			(xy 85.09 25.4) (xy 85.09 44.45)
 		)
 		(stroke
@@
 	(wire
 		(pts
-			(xy 83.82 52.07) (xy 83.82 67.31)
-		)
-		(stroke
-			(width 0)
-			(type default)
-		)
-	)
-	(wire
-		(pts
-			(xy 83.82 67.31) (xy 99.06 67.31)
-		)
-		(stroke
-			(width 0)
-			(type default)
-		)
-	)
-	(wire
-		(pts
-			(xy 102.87 46.99) (xy 83.82 46.99)
-		)
-		(stroke
-			(width 0)
-			(type default)
-		)
-	)
-	(wire
-		(pts
-			(xy 99.06 77.47) (xy 109.22 77.47)
-		)
-		(stroke
-			(width 0)
-			(type default)
-		)
-	)
-	(wire
-		(pts
-			(xy 99.06 67.31) (xy 99.06 77.47)
-		)
-		(stroke
-			(width 0)
-			(type default)
-		)
-	)
-	(wire
-		(pts
-			(xy 109.22 54.61) (xy 109.22 57.15)
-		)
-		(stroke
-			(width 0)
-			(type default)
-		)
-	)
-	(wire
-		(pts
-			(xy 83.82 49.53) (xy 99.06 49.53)
+			(xy 85.09 69.85) (xy 93.98 69.85)
+		)
+		(stroke
+			(width 0)
+			(type default)
+		)
+	)
+	(wire
+		(pts
+			(xy 85.09 52.07) (xy 83.82 52.07)
+		)
+		(stroke
+			(width 0)
+			(type default)
+		)
+	)
+	(wire
+		(pts
+			(xy 85.09 52.07) (xy 85.09 69.85)
+		)
+		(stroke
+			(width 0)
+			(type default)
+		)
+	)
+	(wire
+		(pts
+			(xy 93.98 49.53) (xy 83.82 49.53)
+		)
+		(stroke
+			(width 0)
+			(type default)
+		)
+	)
+	(wire
+		(pts
+			(xy 93.98 45.72) (xy 93.98 46.99)
 		)
 		(stroke
@@
 		)
 	)
+	(global_label "a-"
+		(shape input)
+		(at 93.98 45.72 0)
+		(fields_autoplaced yes)
+		(effects
+			(font
+				(size 1.27 1.27)
+			)
+			(justify left)
+		)
+		(property "Intersheetrefs" "${INTERSHEET_REFS}"
+			(at 99.6866 45.72 0)
+			(effects
+				(font
+					(size 1.27 1.27)
+				)
+				(justify left)
+				(hide yes)
+			)
+		)
+	)
 	(global_label "y-"
 		(shape input)
-		(at 102.87 45.72 0)
+		(at 93.98 49.53 0)
 		(fields_autoplaced yes)
 		(effects
@@
 		)
 		(property "Intersheetrefs" "${INTERSHEET_REFS}"
-			(at 108.3952 45.72 0)
+			(at 99.5052 49.53 0)
 			(effects
 				(font
@@
 		)
 	)
-	(global_label "a-"
-		(shape input)
-		(at 99.06 52.07 0)
+	(global_label "y+"
+		(shape input)
+		(at 85.09 69.85 270)
+		(fields_autoplaced yes)
+		(effects
+			(font
+				(size 1.27 1.27)
+			)
+			(justify right)
+		)
+		(property "Intersheetrefs" "${INTERSHEET_REFS}"
+			(at 85.09 75.3752 90)
+			(effects
+				(font
+					(size 1.27 1.27)
+				)
+				(justify right)
+				(hide yes)
+			)
+		)
+	)
+	(global_label "a+"
+		(shape input)
+		(at 85.09 25.4 90)
 		(fields_autoplaced yes)
 		(effects
@@
 		)
 		(property "Intersheetrefs" "${INTERSHEET_REFS}"
-			(at 104.7666 52.07 0)
+			(at 85.09 19.6934 90)
 			(effects
 				(font
@@
 		)
 	)
-	(global_label "y+"
-		(shape input)
-		(at 88.9 30.48 90)
-		(fields_autoplaced yes)
-		(effects
-			(font
-				(size 1.27 1.27)
-			)
-			(justify left)
-		)
-		(property "Intersheetrefs" "${INTERSHEET_REFS}"
-			(at 88.9 24.9548 90)
-			(effects
-				(font
-					(size 1.27 1.27)
-				)
-				(justify left)
-				(hide yes)
-			)
-		)
-	)
 	(global_label "3.3v"
 		(shape input)
@@
 		(property "Intersheetrefs" "${INTERSHEET_REFS}"
 			(at 33.6634 44.45 0)
-			(effects
-				(font
-					(size 1.27 1.27)
-				)
-				(justify right)
-				(hide yes)
-			)
-		)
-	)
-	(global_label "a+"
-		(shape input)
-		(at 90.17 67.31 270)
-		(fields_autoplaced yes)
-		(effects
-			(font
-				(size 1.27 1.27)
-			)
-			(justify right)
-		)
-		(property "Intersheetrefs" "${INTERSHEET_REFS}"
-			(at 90.17 73.0166 90)
 			(effects
 				(font
@@
 	(symbol
 		(lib_id "RC1206FR-0724RL:RC1206FR-0724RL")
-		(at 121.92 38.1 270)
+		(at 93.98 35.56 270)
 		(unit 1)
 		(exclude_from_sim no)
@@
 		(fields_autoplaced yes)
 		(property "Reference" "R5"
-			(at 125.73 36.8299 90)
+			(at 97.79 34.2899 90)
 			(effects
 				(font
@@
 		)
 		(property "Value" "RC1206FR-0724RL"
-			(at 125.73 39.3699 90)
+			(at 97.79 36.8299 90)
 			(effects
 				(font
@@
 		)
 		(property "Footprint" "Resistor_SMD:R_1206_3216Metric"
-			(at 121.92 38.1 0)
+			(at 93.98 35.56 0)
 			(effects
 				(font
@@
 		)
 		(property "Datasheet" ""
-			(at 121.92 38.1 0)
+			(at 93.98 35.56 0)
 			(effects
 				(font
@@
 		)
 		(property "Description" ""
-			(at 121.92 38.1 0)
+			(at 93.98 35.56 0)
 			(effects
 				(font
@@
 	(symbol
 		(lib_id "RC1206FR-0724RL:RC1206FR-0724RL")
-		(at 109.22 67.31 90)
+		(at 93.98 59.69 90)
 		(unit 1)
 		(exclude_from_sim no)
@@
 		(fields_autoplaced yes)
 		(property "Reference" "R7"
-			(at 113.03 66.0399 90)
+			(at 97.79 58.4199 90)
 			(effects
 				(font
@@
 		)
 		(property "Value" "RC1206FR-0724RL"
-			(at 113.03 68.5799 90)
+			(at 97.79 60.9599 90)
 			(effects
 				(font
@@
 		)
 		(property "Footprint" "Resistor_SMD:R_1206_3216Metric"
-			(at 109.22 67.31 0)
+			(at 93.98 59.69 0)
 			(effects
 				(font
@@
 		)
 		(property "Datasheet" ""
-			(at 109.22 67.31 0)
+			(at 93.98 59.69 0)
 			(effects
 				(font
@@
 		)
 		(property "Description" ""
-			(at 109.22 67.31 0)
-			(effects
-				(font
+			(at 93.98 59.69 0)
+			(effects
+				(font
