File: KiCad/EGSE2/bustingballscrazystylenolube/IO.kicad_sch (KiCad schematic)
At the start: 1 part, among them J1 USB_C_Receptacle_USB2.0_16P

Commit message: here comes the
Parts:
- added J2: USB_C_Receptacle_USB2.0_16P, symbol Connector:USB_C_Receptacle_USB2.0_16P
- added J3: DA15_Socket_MountingHoles, Connector_Dsub:DSUB-15-HD_Socket_Horizontal_P2.29x2.54mm_EdgePinOffset8.35mm_Housed_MountingHolesOffset10.89mm, symbol Connector:DA15_Socket_MountingHoles
Connections:
- net D+: now also J2.A6 (D+), J2.B6 (D+); no longer J1.A6 (D+), J1.B6 (D+)
- net D-: now also J2.A7 (D-), J2.B7 (D-); no longer J1.A7 (D-), J1.B7 (D-)
- net GND: now also J2.A1 (GND), J2.A12 (GND), J2.B1 (GND), J2.B12 (GND), J2.S1 (SHIELD), J3.11 (P111), J3.12 (P12), J3.3, J3.4
- new net RXD: J3.15 (P15)
- new net TXD: J3.8
- new net VBATT: J3.1, J3.10 (P10), J3.2, J3.9 (P9)
- new net VBUS_comm: J2.A4 (VBUS), J2.A9 (VBUS), J2.B4 (VBUS), J2.B9 (VBUS)

Commit message: wo
Parts:
- J1, J2: footprint (none) -> Connector_USB:USB_C_Receptacle_GCT_USB4105-xx-A_16P_TopMnt_Horizontal
Changed lines of the file:
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@@
 			)
 		)
-		(property "Footprint" ""
+		(property "Footprint" "Connector_USB:USB_C_Receptacle_GCT_USB4105-xx-A_16P_TopMnt_Horizontal"
 			(at 52.07 55.88 0)
 			(effects
@@
 			)
 		)
-		(property "Footprint" ""
+		(property "Footprint" "Connector_USB:USB_C_Receptacle_GCT_USB4105-xx-A_16P_TopMnt_Horizontal"
 			(at 52.07 114.3 0)
 			(effects

Commit message: slumpt
Parts:
- added J4: Conn_02x08_Top_Bottom, Connector_PinHeader_2.54mm:PinHeader_2x08_P2.54mm_Vertical, symbol Connector_Generic:Conn_02x08_Top_Bottom
Connections:
- net GND: now also J3.13 (P13), J3.8, J3.9 (P9), J4.1 (Pin_1), J4.3 (Pin_3), J4.5 (Pin_5), J4.7 (Pin_7); no longer J3.3, J3.4
- net RXD: now also J3.5, J4.11 (Pin_11), J4.12 (Pin_12); no longer J3.15 (P15)
- net TXD: now also J3.4, J4.10 (Pin_10), J4.9 (Pin_9); no longer J3.8
- net VBATT: now also J3.3, J3.6, J3.7, J4.2 (Pin_2), J4.4 (Pin_4), J4.6 (Pin_6), J4.8 (Pin_8); no longer J3.10 (P10), J3.9 (P9)
