File: KiCad/EGSE2/bustingballscrazystylenolube/bustingballscrazystylenolube.kicad_sch (KiCad schematic)
At the start: 0 parts

Commit message: here comes the
Other:
- added sheet BttChg (BttChg.kicad_sch)
- added sheet CP2102 (CP2102.kicad_sch)
- sheet IO ports: added CC1, CC2, D+, D-, GND, RXD, TXD, VBATT, VBUS, VBUS_comm; removed none
- sheet USBHELL ports: added CC1, CC2, GND, I2Ct_SCL, I2Ct_SDA, PPHV, VBUS; removed none

Commit message: wo
Changed lines of the file:
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@@
 	(paper "A4")
+	(junction
+		(at 93.98 154.94)
+		(diameter 0)
+		(color 0 0 0 0)
+	)
 	(junction
 		(at 93.98 106.68)
@@
 	(wire
 		(pts
+			(xy 93.98 154.94) (xy 93.98 162.56)
+		)
+		(stroke
+			(width 0)
+			(type default)
+		)
+	)
+	(wire
+		(pts
 			(xy 129.54 137.16) (xy 129.54 147.32)
 		)
@@
 		)
 	)
+	(symbol
+		(lib_id "power:GND")
+		(at 93.98 162.56 0)
+		(unit 1)
+		(exclude_from_sim no)
+		(in_bom yes)
+		(on_board yes)
+		(dnp no)
+		(fields_autoplaced yes)
+		(property "Reference" "#PWR01"
+			(at 93.98 168.91 0)
+			(effects
+				(font
+					(size 1.27 1.27)
+				)
+				(hide yes)
+			)
+		)
+		(property "Value" "GND"
+			(at 93.98 167.64 0)
+			(effects
+				(font
+					(size 1.27 1.27)
+				)
+			)
+		)
+		(property "Footprint" ""
+			(at 93.98 162.56 0)
+			(effects
+				(font
+					(size 1.27 1.27)
+				)
+				(hide yes)
+			)
+		)
+		(property "Datasheet" ""
+			(at 93.98 162.56 0)
+			(effects
+				(font
+					(size 1.27 1.27)
+				)
+				(hide yes)
+			)
+		)
+		(property "Description" "Power symbol creates a global label with name \"GND\" , ground"
+			(at 93.98 162.56 0)
+			(effects
+				(font
+					(size 1.27 1.27)
+				)
+				(hide yes)
+			)
+		)
+		(pin "1"
+		)
+		(instances
+			(project ""
+				(path "/93514605-6b24-46cc-859f-51fd06f5909b"
+					(reference "#PWR01")
+					(unit 1)
+				)
+			)
+		)
+	)

Commit message: slumpt
Parts:
- added H1, H2, H3, H4: MountingHole, MountingHole:MountingHole_3mm_Pad, symbol Mechanical:MountingHole
