File: KiCad/EGSE2/bustingballscrazystylenolube/BttChg.kicad_sch (KiCad schematic)
At the start: 30 parts, among them U3 BQ25713BRSNR

Commit message: slumpt
Parts:
- added IN1: IN, TestPoint:TestPoint_Pad_1.0x1.0mm, symbol Connector:TestPoint
- added OUT1: OUT, TestPoint:TestPoint_Pad_1.0x1.0mm, symbol Connector:TestPoint
- added PPHV1: PPHV, TestPoint:TestPoint_Pad_1.0x1.0mm, symbol Connector:TestPoint
- added SW1: SW1, TestPoint:TestPoint_Pad_1.0x1.0mm, symbol Connector:TestPoint
- added SW2: SW2, TestPoint:TestPoint_Pad_1.0x1.0mm, symbol Connector:TestPoint
- added VBATT1: VBATT, TestPoint:TestPoint_Pad_1.0x1.0mm, symbol Connector:TestPoint
- added VDDA1: VDDA, TestPoint:TestPoint_Pad_1.0x1.0mm, symbol Connector:TestPoint
- R16, R22: footprint Resistor_SMD:R_0805_2012Metric_Pad1.20x1.40mm_HandSolder -> Resistor_SMD:R_2512_6332Metric_Pad1.40x3.35mm_HandSolder
- renumbered C8 to C11, C11 to C8
Connections:
- net IN: now also IN1.1
- net OUT: now also OUT1.1
- net PPHV: now also PPHV1.1; no longer C12.1, C13.1, C8.1
- net SW1: now also SW1.1
- net SW2: now also SW2.1
- net VBATT: now also C12.1, C13.1, C8.1, VBATT1.1
- net VDDA: now also VDDA1.1
Other:
- moved on the sheet: C12, C13, C8

Commit message: shmovwe
Parts:
- added R30: 60k, Resistor_SMD:R_0805_2012Metric_Pad1.20x1.40mm_HandSolder, symbol Device:R
- added R31: 40k, Resistor_SMD:R_0805_2012Metric_Pad1.20x1.40mm_HandSolder, symbol Device:R
Connections:
- net OTG/VAP is gone; now on net GND: U3.5 (OTG/VAP)
- net CELL_BATPRESZ: now also R30.1, R31.2
- net GND: now also R31.1
- net OUT: no longer U3.21 (*BATDRV)
- net VDDA: now also R30.2
Changed lines of the file:
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@@
 	)
 	(junction
-		(at 158.75 111.76)
+		(at 166.37 171.45)
 		(diameter 0)
 		(color 0 0 0 0)
@@
 	(wire
 		(pts
-			(xy 158.75 114.3) (xy 158.75 111.76)
+			(xy 166.37 171.45) (xy 182.88 171.45)
 		)
 		(stroke
@@
 	(wire
 		(pts
+			(xy 166.37 162.56) (xy 166.37 160.02)
+		)
+		(stroke
+			(width 0)
+			(type default)
+		)
+	)
+	(wire
+		(pts
 			(xy 152.4 170.18) (xy 152.4 171.45)
 		)
@@
 	(wire
 		(pts
-			(xy 156.21 114.3) (xy 158.75 114.3)
-		)
-		(stroke
-			(width 0)
-			(type default)
-		)
-	)
-	(wire
-		(pts
 			(xy 100.33 60.96) (xy 109.22 60.96)
 		)
@@
 	(wire
 		(pts
-			(xy 152.4 160.02) (xy 162.56 160.02)
+			(xy 152.4 160.02) (xy 166.37 160.02)
 		)
 		(stroke
@@
 	(wire
 		(pts
-			(xy 156.21 111.76) (xy 158.75 111.76)
-		)
-		(stroke
-			(width 0)
-			(type default)
-		)
-	)
-	(wire
-		(pts
 			(xy 152.4 162.56) (xy 152.4 160.02)
 		)
@@
 	(wire
 		(pts
+			(xy 166.37 170.18) (xy 166.37 171.45)
+		)
+		(stroke
+			(width 0)
+			(type default)
+		)
+	)
+	(wire
+		(pts
 			(xy 177.8 142.24) (xy 177.8 138.43)
 		)
@@
 	(wire
 		(pts
+			(xy 166.37 171.45) (xy 166.37 172.72)
+		)
+		(stroke
+			(width 0)
+			(type default)
+		)
+	)
+	(wire
+		(pts
 			(xy 100.33 40.64) (xy 109.22 40.64)
 		)
@@
 	(wire
 		(pts
-			(xy 158.75 111.76) (xy 165.1 111.76)
+			(xy 156.21 111.76) (xy 165.1 111.76)
 		)
 		(stroke
@@
 		)
 	)
-	(label "OTG{slash}VAP"
-		(at 80.01 93.98 0)
-		(effects
-			(font
-				(size 1.27 1.27)
-			)
-			(justify left bottom)
-		)
-	)
 	(label "REGN"
 		(at 165.1 96.52 180)
@@
 		)
 	)
+	(label "CELL_BATPRESZ"
+		(at 182.88 171.45 180)
+		(effects
+			(font
+				(size 1.27 1.27)
+			)
+			(justify right bottom)
+		)
+	)
 	(label "HIDRV1"
 		(at 100.33 43.18 0)
@@
 	(hierarchical_label "GND"
 		(shape output)
+		(at 166.37 180.34 270)
+		(effects
+			(font
+				(size 1.27 1.27)
+			)
+			(justify right)
+		)
+	)
+	(hierarchical_label "GND"
+		(shape output)
+		(at 80.01 93.98 180)
+		(effects
+			(font
+				(size 1.27 1.27)
+			)
+			(justify right)
+		)
+	)
+	(hierarchical_label "GND"
+		(shape output)
 		(at 38.1 190.5 180)
 		(effects
@@
 	)
 	(symbol
+		(lib_id "Device:R")
+		(at 166.37 166.37 180)
+		(unit 1)
+		(exclude_from_sim no)
+		(in_bom yes)
+		(on_board yes)
+		(dnp no)
+		(fields_autoplaced yes)
+		(property "Reference" "R30"
+			(at 168.91 165.0999 0)
+			(effects
+				(font
+					(size 1.27 1.27)
+				)
+				(justify right)
+			)
+		)
+		(property "Value" "60k"
+			(at 168.91 167.6399 0)
+			(effects
+				(font
+					(size 1.27 1.27)
+				)
+				(justify right)
+			)
+		)
+		(property "Footprint" "Resistor_SMD:R_0805_2012Metric_Pad1.20x1.40mm_HandSolder"
+			(at 168.148 166.37 90)
+			(effects
+				(font
+					(size 1.27 1.27)
+				)
+				(hide yes)
+			)
+		)
+		(property "Datasheet" "~"
+			(at 166.37 166.37 0)
+			(effects
+				(font
+					(size 1.27 1.27)
+				)
+				(hide yes)
+			)
+		)
+		(property "Description" "Resistor"
+			(at 166.37 166.37 0)
+			(effects
+				(font
+					(size 1.27 1.27)
+				)
+				(hide yes)
+			)
+		)
+		(pin "1"
+		)
+		(pin "2"
+		)
+		(instances
+			(project "bustingballscrazystylenolube"
+				(path "/93514605-6b24-46cc-859f-51fd06f5909b/7f3a3102-a634-4703-8b8f-f224a071de32"
+					(reference "R30")
+					(unit 1)
+				)
+			)
+		)
+	)
+	(symbol
 		(lib_id "Connector:TestPoint")
 		(at 228.6 63.5 90)
@@
 					(unit 1)
 				)
+			)
+		)
+	)
+	(symbol
+		(lib_id "Device:R")
+		(at 166.37 176.53 180)
+		(unit 1)
+		(exclude_from_sim no)
+		(in_bom yes)
+		(on_board yes)
+		(dnp no)
+		(fields_autoplaced yes)
+		(property "Reference" "R31"
+			(at 168.91 175.2599 0)
+			(effects
+				(font
+					(size 1.27 1.27)
+				)
+				(justify right)
+			)
+		)
+		(property "Value" "40k"
+			(at 168.91 177.7999 0)
+			(effects
+				(font
+					(size 1.27 1.27)
+				)
+				(justify right)
+			)
+		)
+		(property "Footprint" "Resistor_SMD:R_0805_2012Metric_Pad1.20x1.40mm_HandSolder"
+			(at 168.148 176.53 90)
+			(effects
+				(font
+					(size 1.27 1.27)
+				)
+				(hide yes)
+			)
+		)
+		(property "Datasheet" "~"
+			(at 166.37 176.53 0)
+			(effects
+				(font
+					(size 1.27 1.27)
+				)
+				(hide yes)
+			)
+		)
+		(property "Description" "Resistor"
+			(at 166.37 176.53 0)
+			(effects
+				(font
+					(size 1.27 1.27)
+				)
+				(hide yes)
+			)
+		)
+		(pin "1"
+		)
+		(pin "2"
+		)
+		(instances
+			(project "bustingballscrazystylenolube"
+				(path "/93514605-6b24-46cc-859f-51fd06f5909b/7f3a3102-a634-4703-8b8f-f224a071de32"
+					(reference "R31")
+					(unit 1)
+				)
