File: KiCad/Commodore 7/Commodore 7-2025-11-09_234237/Commodore 7.kicad_pcb (KiCad board)
At the start: 2 copper layers, 41 parts, among them IC1 BGU7004,115, J1 M20-6112045, U1 TMP112AIDRLR-Temperature, U10 TCA9543APWR, U2 NEO-M9N-00B, U3 BMI270 - Secondary Accelerome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, U4 MMC5983MA-Magnetomer, U5 MS560702BA03-50 - Barometer, U6 TCA9509DGKR, U7 SN65HVD74DR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

Commit message: doing some routinggggg
Parts:
- E1: moved to B.Cu
- moved U2 30.3 mm to (231.4, 34.0)
- moved C6 29.7 mm to (213.1, 41.9), turned to 135 degrees
- moved E1 28.1 mm to (203.2, 27.1), turned to 180 degrees
- moved R7 27.0 mm to (210.8, 43.6), turned to -45 degrees
- moved R8 26.5 mm to (212.7, 45.4), turned to -45 degrees
- moved U11 25.1 mm to (219.0, 42.8), turned to -45 degrees
- moved IC1 22.2 mm to (216.4, 40.4), turned to 135 degrees
- moved L1 21.7 mm to (216.3, 37.1), turned to -90 degrees
- moved C1 2.51 mm to (41.8, 93.9)
- moved R5 1.72 mm to (37.1, 92.0), turned to 90 degrees
- moved C5 1.52 mm to (105.9, 119.0), turned to 90 degrees
- moved C4 0.22 mm to (115.6, 120.8)
Routing:
- net Net-(U1-V+): track 0.00 -> 8.31 mm
- net Net-(IC1-VCC): track 0.00 -> 7.98 mm
- net Net-(U11-RF_OUT): track 0.00 -> 7.01 mm
- net 3.3v: track 74.1 -> 77.5 mm
- net Net-(U4-CAP): track 0.00 -> 2.93 mm
- net Net-(IC1-RF_OUT): track 0.00 -> 2.75 mm
- net Net-(IC1-RF_IN): track 0.00 -> 2.28 mm

Commit message: organizing some things ig
Parts:
- E1: moved to F.Cu
- U2: moved to B.Cu
- moved R6 141.6 mm to (172.0, 125.2), turned to 180 degrees
- moved C3 139.9 mm to (180.9, 119.6), turned to 90 degrees
- moved U3 134.2 mm to (172.2, 119.4), turned to 90 degrees
- moved C2 131.7 mm to (174.5, 116.4), turned to -45 degrees
- moved C13 110.2 mm to (140.3, 125.3), turned to -90 degrees
- moved C15 107.2 mm to (138.1, 125.0), turned to -90 degrees
- moved C16 106.8 mm to (136.0, 70.2), turned to 90 degrees
- moved C14 104.4 mm to (134.1, 70.2), turned to 90 degrees
- moved C17 103.0 mm to (135.0, 125.0), turned to -90 degrees
- moved U9 102.1 mm to (135.5, 78.3), turned to 180 degrees
- moved C12 101.7 mm to (132.1, 70.3), turned to 90 degrees
- moved U8 101.5 mm to (135.5, 120.3), turned to 0 degrees
- moved R27 100.0 mm to (135.6, 84.6), turned to -90 degrees
- moved R21 96.7 mm to (133.2, 84.7), turned to -90 degrees
- moved U7 93.8 mm to (20.6, 174.7)
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Routing:
- net Net-(U11-RF_OUT): track 7.01 -> 18.3 mm, vias 0 -> 1
- net Net-(E1-Pad1): track 0.00 -> 9.23 mm, vias 0 -> 1

Commit message: updated some labels idk
Changed lines of the file:
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@@
+	)
+	(segment
+		(start 131.085 88.915)
+		(end 131.1 88.9)
+		(width 0.2)
+		(layer "F.Cu")
+		(net 45)
 	)
 	(segment
@@
 	(segment
 		(start 130.725 89.275)
-		(end 131.1 88.9)
+		(end 131.085 88.915)
 		(width 0.2)
 		(layer "F.Cu")
