File: KiCad/Commodore 6/Commodore 6.kicad_pcb (KiCad board)
At the start: 4 copper layers, 127 x 127 mm, 132 parts, among them J1 472192001, J10 FH12-22S-0.5SH55, J11 Conn_01x06, J2 PPTC071LFBN-RC, J3 6130XX11121_61300511121, J4 Conn_01x05_Pin, J5 Conn_01x02_Pin, J6 FTSH-107-01-L-DV-K-A, J7 Conn_01x06, J8 M20-6112045, J9 FH12-24S-0.5SH_55_, Q1 2N2219, Q2 NTR4501NT1G, Q3 PMOS, Q4 PMOS, SW1 SLW-1277545-3A-RA-N-D, SW1A1 SLW-1277545-3A-RA-N-D, SW2 SLW-1277545-3A-RA-N-D, SW3 SLW-1277545-3A-RA-N-D, U1 STM32H562RIT6, U2 STM32H7A3RIT6, U3 SN65HVD74DR, U4 TS3A27518EIPWRQ1, U5 SN74CBT16233DLR, U6 PCA9507DP,118, U7 ADV7280AWBCPZ, U8 TLV1117LV33DCYR, Y1 ABM8AIG-28.63636MHZ

Commit message: Update Commodore 6.kicad_pcb
Connections:
- net Net-(Q3-S) renamed /Power/mosfet_big
Routing:
- net /Power/mosfet_big: track 16.8 -> 0.00 mm, vias 2 -> 7
- net Net-(Q3-G): track 35.2 -> 31.4 mm, vias 4 -> 3
- net I2C_SCL: track 139.3 -> 137.6 mm
- added copper zone on F.Cu, net /Power/mosfet_big
- added copper zone on In1.Cu, net /Power/mosfet_big
Changed lines of the file:
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@@
 	(net 220 "NTSC_SCL")
 	(net 221 "NTSC_D6")
-	(net 222 "Net-(Q3-S)")
+	(net 222 "/Power/mosfet_big")
 	(net 223 "NTSC_SDA")
 	(net 224 "NTSC_D3")
@@
 			(size 1.43 0.6)
 			(layers "F.Cu" "F.Mask" "F.Paste")
-			(net 222 "Net-(Q3-S)")
+			(net 222 "/Power/mosfet_big")
 			(pinfunction "S")
 			(pintype "passive")
@@
 			(size 1.43 0.6)
 			(layers "F.Cu" "F.Mask" "F.Paste")
-			(net 222 "Net-(Q3-S)")
+			(net 222 "/Power/mosfet_big")
 			(pinfunction "S")
 			(pintype "passive")
@@
 	)
 	(via
-		(at 68 78)
-		(size 1)
-		(drill 0.6)
+		(at 69.95 87.4)
+		(size 0.6)
+		(drill 0.3)
 		(layers "F.Cu" "B.Cu")
-		(free yes)
 		(net 5)
 	)
 	(via
-		(at 70 78)
+		(at 53.2 69)
 		(size 1)
 		(drill 0.6)
@@
 	)
 	(via
-		(at 69.95 87.4)
-		(size 0.6)
-		(drill 0.3)
-		(layers "F.Cu" "B.Cu")
-		(net 5)
-	)
-	(via
 		(at 53.213429 70.5)
 		(size 1)
@@
 	)
 	(via
-		(at 57.213429 70.5)
+		(at 55.2 69)
 		(size 1)
 		(drill 0.6)
@@
 	)
 	(via
-		(at 72 78)
+		(at 57.213429 70.5)
 		(size 1)
 		(drill 0.6)
@@
 		(net 5)
 	)
+	(via
+		(at 57.2 69)
+		(size 1)
+		(drill 0.6)
+		(layers "F.Cu" "B.Cu")
+		(free yes)
+		(net 5)
+	)
 	(segment
 		(start 67.45 87.4)
@@
 	)
 	(segment
+		(start 34.740001 104.259999)
+		(end 35.6175 104.259999)
+		(width 0.2)
+		(layer "F.Cu")
+		(net 21)
+	)
+	(segment
+		(start 38.62 109.209999)
+		(end 34.709999 109.209999)
+		(width 0.2)
+		(layer "F.Cu")
+		(net 21)
+	)
+	(segment
+		(start 33.75 108.25)
+		(end 33.75 105.25)
+		(width 0.2)
+		(layer "F.Cu")
+		(net 21)
+	)
+	(segment
+		(start 39.2 110.4)
+		(end 38.62 109.82)
+		(width 0.2)
+		(layer "F.Cu")
+		(net 21)
+	)
+	(segment
 		(start 51.16 103.209999)
 		(end 46.13 103.209999)
@@
 	)
 	(segment
-		(start 35.6175 104.797499)
-		(end 36.08 105.259999)
-		(width 0.5)
+		(start 38.62 109.82)
+		(end 38.62 109.209999)
+		(width 0.2)
+		(layer "F.Cu")
+		(net 21)
+	)
+	(segment
+		(start 34.709999 109.209999)
+		(end 33.75 108.25)
+		(width 0.2)
 		(layer "F.Cu")
 		(net 21)
@@
 	)
 	(segment
+		(start 33.75 105.25)
+		(end 34.740001 104.259999)
+		(width 0.2)
+		(layer "F.Cu")
+		(net 21)
+	)
+	(segment
 		(start 35.605 104.247499)
 		(end 35.6175 104.259999)
@@
 	)
 	(segment
+		(start 41 110.4)
+		(end 39.2 110.4)
+		(width 0.2)
+		(layer "F.Cu")
+		(net 21)
+	)
+	(segment
 		(start 35.605 101.259999)
 		(end 35.605 104.247499)
@@
 	)
 	(via
-		(at 38.62 109.209999)
-		(size 1)
-		(drill 0.6)
+		(at 41 110.4)
+		(size 0.6)
+		(drill 0.3)
 		(layers "F.Cu" "B.Cu")
 		(net 21)
@@
 	)
 	(via
-		(at 36.08 105.259999)
-		(size 0.6)
-		(drill 0.3)
-		(layers "F.Cu" "B.Cu")
-		(net 21)
-	)
-	(via
 		(at 46.08 103.259999)
 		(size 0.6)
@@
 	)
 	(segment
-		(start 38.62 109.209999)
-		(end 38.62 109.182499)
-		(width 0.3)
-		(layer "B.Cu")
-		(net 21)
-	)
-	(segment
-		(start 40.03 109.209999)
-		(end 38.62 109.209999)
-		(width 0.3)
-		(layer "B.Cu")
-		(net 21)
-	)
-	(segment
-		(start 44.57 103.259999)
-		(end 41.04 106.79)
-		(width 0.4)
-		(layer "B.Cu")
-		(net 21)
-	)
-	(segment
-		(start 39.509999 105.259999)
-		(end 41.04 106.79)
+		(start 41.072058 110.4)
+		(end 41 110.4)
 		(width 0.2)
 		(layer "B.Cu")
@@
 	)
 	(segment
-		(start 44.58 113.759999)
-		(end 40.03 109.209999)
-		(width 0.3)
-		(layer "B.Cu")
-		(net 21)
-	)
-	(segment
-		(start 36.08 105.259999)
-		(end 39.509999 105.259999)
+		(start 47.08 113.722499)
+		(end 47.0425 113.759999)
 		(width 0.2)
 		(layer "B.Cu")
@@
 	)
 	(segment
-		(start 47.08 113.722499)
-		(end 47.0425 113.759999)
+		(start 47.0425 113.759999)
+		(end 44.432057 113.759999)
 		(width 0.2)
 		(layer "B.Cu")
@@
 	)
 	(segment
-		(start 41.04 106.79)
-		(end 38.62 109.209999)
-		(width 0.4)
+		(start 44.432057 113.759999)
+		(end 41.072058 110.4)
+		(width 0.2)
 		(layer "B.Cu")
 		(net 21)
@@
 	)
 	(segment
-		(start 47.0425 113.759999)
-		(end 44.58 113.759999)
-		(width 0.3)
-		(layer "B.Cu")
-		(net 21)
-	)
-	(segment
 		(start 104.540601 64.8911)
 		(end 104.540601 62.4286)
@@
 	)
 	(segment
-		(start 62.094314 77.205686)
-		(end 63.844314 77.205686)
-		(width 0.2)
-		(layer "B.Cu")
-		(net 28)
-	)
-	(segment
 		(start 85.75 55.75)
 		(end 85.75 55.3)
@@
 		(net 221)
 	)
-	(segment
-		(start 41.58 108.259999)
-		(end 42.08 107.759999)
-		(width 0.7)
-		(layer "F.Cu")
+	(via
+		(at 53.4 104.6)
+		(size 1)
+		(drill 0.6)
+		(layers "F.Cu" "B.Cu")
+		(free yes)
 		(net 222)
 	)
-	(segment
-		(start 40.54 108.259999)
-		(end 41.58 108.259999)
-		(width 0.7)
-		(layer "F.Cu")
+	(via
+		(at 53.4 101.8)
+		(size 1)
+		(drill 0.6)
+		(layers "F.Cu" "B.Cu")
+		(free yes)
 		(net 222)
 	)
 	(via
-		(at 53.08 102.259999)
+		(at 40.6 107.2)
 		(size 1)
 		(drill 0.6)
 		(layers "F.Cu" "B.Cu")
+		(free yes)
 		(net 222)
 	)
 	(via
-		(at 42.08 107.759999)
+		(at 42 109.2)
 		(size 1)
 		(drill 0.6)
 		(layers "F.Cu" "B.Cu")
+		(free yes)
 		(net 222)
 	)
-	(segment
-		(start 50.58 107.759999)
-		(end 53.08 105.259999)
-		(width 0.7)
-		(layer "B.Cu")
+	(via
+		(at 42 107.2)
+		(size 1)
+		(drill 0.6)
+		(layers "F.Cu" "B.Cu")
+		(free yes)
 		(net 222)
 	)
-	(segment
-		(start 53.08 105.259999)
-		(end 53.08 102.259999)
-		(width 0.7)
-		(layer "B.Cu")
+	(via
+		(at 55.4 104.6)
+		(size 1)
+		(drill 0.6)
+		(layers "F.Cu" "B.Cu")
+		(free yes)
 		(net 222)
 	)
-	(segment
-		(start 42.08 107.759999)
-		(end 50.58 107.759999)
-		(width 0.7)
-		(layer "B.Cu")
+	(via
+		(at 55.4 101.8)
+		(size 1)
+		(drill 0.6)
+		(layers "F.Cu" "B.Cu")
+		(free yes)
 		(net 222)
 	)
@@
 	)
 	(zone
+		(net 222)
+		(net_name "/Power/mosfet_big")
+		(layer "F.Cu")
+		(hatch edge 0.5)
+		(priority 15)
+		(connect_pads yes
+			(clearance 0.5)
+		)
+		(min_thickness 0.25)
+		(filled_areas_thickness no)
+		(fill yes
+			(thermal_gap 0.5)
+			(thermal_bridge_width 0.5)
+		)
+		(polygon
+			(pts
+				(xy 40 106.6) (xy 40 109.8) (xy 42.8 109.8) (xy 42.8 106.6)
+			)
+		)
+	)
+	(zone
 		(net 38)
 		(net_name "+5V")
@@
 	)
 	(zone
+		(net 222)
+		(net_name "/Power/mosfet_big")
+		(layer "F.Cu")
+		(hatch edge 0.5)
+		(priority 16)
+		(connect_pads yes
+			(clearance 0.5)
+		)
+		(min_thickness 0.25)
+		(filled_areas_thickness no)
+		(fill yes
+			(thermal_gap 0.5)
+			(thermal_bridge_width 0.5)
+		)
+		(polygon
+			(pts
+				(xy 52.8 101.2) (xy 56 101.2) (xy 56 105.4) (xy 52.8 105.4)
+			)
+		)
+	)
+	(zone
 		(net 3)
 		(net_name "GNDA")
@@
 		(polygon
 			(pts
-				(xy 14.5 98.5) (xy 58 98.5) (xy 58 124.5) (xy 14.5 124.5)
+				(xy 14.5 98.5) (xy 39.5 98.5) (xy 39.5 124.5) (xy 14.5 124.5)
+			)
+		)
+	)
+	(zone
+		(net 222)
+		(net_name "/Power/mosfet_big")
+		(layer "In1.Cu")
+		(hatch edge 0.5)
+		(priority 14)
+		(connect_pads
+			(clearance 0.5)
+		)
+		(min_thickness 0.25)
+		(filled_areas_thickness no)
+		(fill yes
+			(thermal_gap 0.5)
+			(thermal_bridge_width 0.5)
+		)
+		(polygon
+			(pts
+				(xy 40 106.6) (xy 40 109.8) (xy 56 109.759999) (xy 56 101.2) (xy 51.4 101.2) (xy 51.4 106.4)
 			)
 		)

Commit message: Update Commodore 6.kicad_pcb
Parts:
- moved C25 157.3 mm to (53.7, 64.4), turned to 180 degrees
- moved Payload_Header1 153.2 mm to (41.3, 69.2), turned to 90 degrees
- moved C19 151.0 mm to (53.7, 70.6), turned to 180 degrees
- moved Payload_LoadSwitch1 145.0 mm to (47.5, 68.2), turned to 90 degrees
- moved R10 140.2 mm to (47.5, 65.3)
- moved R5 136.4 mm to (49.4, 68.9), turned to -90 degrees
- moved C22 25.3 mm to (75.0, 97.0)
- moved C24 25.3 mm to (72.0, 97.0)
- moved Current_Monitor1 25.3 mm to (66.0, 96.5)
- moved R9 25.3 mm to (59.0, 98.5)
Connections:
- 1.8LDO1 pad 5: +1.8V -> 1.8V
- C43 pad 2: +1.8V -> 1.8V
- J3 pad 1: +1.8V -> 1.8V
- J7 pad 2: 8.4V -> +8.4V
- R36 pad 1: +1.8V -> 1.8V
Routing:
- net +3.3V: track 210.0 -> 763.9 mm, vias 13 -> 22
- net +5V: track 144.9 -> 426.3 mm, vias 15 -> 24
- net +8.4V: track 15.8 -> 217.7 mm, vias 8 -> 7
- net EGSE_TX: track 19.8 -> 98.0 mm, vias 3 -> 4
- net EGSE_RX: track 21.1 -> 95.3 mm, vias 3 -> 4
- net +2.8V: track 57.0 -> 101.2 mm, vias 3 -> 7
- net 1.8V: track 12.9 -> 51.3 mm, vias 4 -> 9
- net I2C_SCL: track 137.6 -> 156.8 mm
- net +1.8V: track 17.4 -> 0.00 mm
- net Net-(Payload_LoadSwitch1-VOUT): track 0.00 -> 12.6 mm
- net I2C_SDA: track 132.8 -> 145.1 mm
- net Net-(Q3-G): track 31.4 -> 37.0 mm
- net 8.4V_evil: track 5.17 -> 0.00 mm
- net 8.4V: track 4.78 -> 0.00 mm, vias 2 -> 0
- net GNDA: track 283.2 -> 285.5 mm, vias 45 -> 49
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- added copper zone on F.Cu, net +2.8V
- added copper zone on In1.Cu, net +2.8V
- added copper zone on In1.Cu, net +3.3V
- added copper zone on F.Cu, net 1.8V
- added copper zone on In1.Cu, net 1.8V
- added copper zone on F.Cu, net 8.4V_evil
- added copper zone on In2.Cu, net GNDA
- removed copper zone on F.Cu, net 8.4V

Commit message: bruh
Connections:
- DSUB1 pad 11: GND -> GNDA
- DSUB1 pad 12: GND -> GNDA
- DSUB1 pad 3: GND -> GNDA
- DSUB1 pad 4: GND -> GNDA
Routing:
- net +3.3V: track 763.9 -> 764.4 mm
Changed lines of the file:
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@@
 			(layers "*.Cu" "*.Mask")
 			(remove_unused_layers no)
-			(net 73 "GND")
+			(net 2 "GNDA")
 			(pinfunction "3")
 			(pintype "passive")
@@
 			(layers "*.Cu" "*.Mask")
 			(remove_unused_layers no)
-			(net 73 "GND")
+			(net 2 "GNDA")
 			(pinfunction "4")
 			(pintype "passive")
@@
 			(layers "*.Cu" "*.Mask")
 			(remove_unused_layers no)
-			(net 73 "GND")
+			(net 2 "GNDA")
 			(pinfunction "11")
 			(pintype "passive")
@@
 			(layers "*.Cu" "*.Mask")
 			(remove_unused_layers no)
-			(net 73 "GND")
+			(net 2 "GNDA")
 			(pinfunction "12")
 			(pintype "passive")
@@
 	)
 	(segment
+		(start 82.4 45.9)
+		(end 83.139446 45.9)
+		(width 0.3)
+		(layer "F.Cu")
+		(net 9)
+	)
+	(segment
 		(start 69.4467 39.75)
 		(end 68.335519 38.638819)
@@
 	)
 	(segment
+		(start 83.139446 45.9)
+		(end 83.519723 45.519723)
+		(width 0.3)
+		(layer "F.Cu")
+		(net 9)
+	)
+	(segment
 		(start 51.24 26.19)
 		(end 52.405 26.19)
@@
 	)
 	(segment
-		(start 82.4 45.9)
-		(end 83.15 45.9)
-		(width 0.2)
-		(layer "F.Cu")
-		(net 9)
-	)
-	(segment
 		(start 83.610277 45.439723)
 		(end 83.629723 45.439723)
@@
 		(start 97.5 84.5)
 		(end 97.5 83.5)
-		(width 0.2)
+		(width 0.3)
 		(layer "In1.Cu")
 		(net 9)
@@
 		(start 82.75 46.25)
 		(end 82.4 45.9)
-		(width 0.2)
+		(width 0.3)
 		(layer "In1.Cu")
 		(net 9)
@@
 		(start 82.75 68.75)
 		(end 82.75 46.25)
-		(width 0.2)
+		(width 0.3)
 		(layer "In1.Cu")
 		(net 9)
@@
 		(start 97.5 83.5)
 		(end 82.75 68.75)
-		(width 0.2)
+		(width 0.3)
 		(layer "In1.Cu")
 		(net 9)
@@
 	)
 	(segment
-		(start 81.175745 42.993765)
+		(start 82.480277 44.298297)
 		(end 80.603821 42.421841)
-		(width 0.2)
+		(width 0.3)
 		(layer "F.Cu")
 		(net 126)
@@
 	(segment
 		(start 82.480277 44.480277)
-		(end 81.175745 43.175745)
-		(width 0.2)
-		(layer "F.Cu")
-		(net 126)
-	)
-	(segment
-		(start 81.175745 43.175745)
-		(end 81.175745 42.993765)
+		(end 82.480277 44.298297)
 		(width 0.2)
 		(layer "F.Cu")
