File: KiCad/Commodore 7.67/Crystal.kicad_sch (KiCad schematic)
At the start: 4 parts, among them Y1 52MHz

Commit message: its over
Parts:
- renumbered C1 to C40, C2 to C41
Changed lines of the file:
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@@
 		(on_board yes)
 		(dnp no)
-		(property "Reference" "C2"
+		(property "Reference" "C41"
 			(at 151.13 88.9 90)
 			(effects
@@
 			(project "Commodore 7.67"
 				(path "/92fa3f49-0e94-4664-860a-d244369fb976/068aab43-7d3e-4c07-94df-f9ae785d2fce"
-					(reference "C2")
+					(reference "C41")
 					(unit 1)
 				)
@@
 		(dnp no)
 		(fields_autoplaced yes)
-		(property "Reference" "#PWR011"
+		(property "Reference" "#PWR071"
 			(at 137.16 68.58 0)
 			(effects
@@
 			(project "Commodore 7.67"
 				(path "/92fa3f49-0e94-4664-860a-d244369fb976/068aab43-7d3e-4c07-94df-f9ae785d2fce"
-					(reference "#PWR011")
+					(reference "#PWR071")
 					(unit 1)
 				)
@@
 		(dnp no)
 		(fields_autoplaced yes)
-		(property "Reference" "#PWR013"
+		(property "Reference" "#PWR070"
 			(at 111.76 74.93 0)
 			(effects
@@
 			(project "Commodore 7.67"
 				(path "/92fa3f49-0e94-4664-860a-d244369fb976/068aab43-7d3e-4c07-94df-f9ae785d2fce"
-					(reference "#PWR013")
+					(reference "#PWR070")
 					(unit 1)
 				)
@@
 		(on_board yes)
 		(dnp no)
-		(property "Reference" "C1"
+		(property "Reference" "C40"
 			(at 123.19 78.74 90)
 			(effects
@@
 			(project "Commodore 7.67"
 				(path "/92fa3f49-0e94-4664-860a-d244369fb976/068aab43-7d3e-4c07-94df-f9ae785d2fce"
-					(reference "C1")
+					(reference "C40")
 					(unit 1)
 				)
@@
 		(dnp no)
 		(fields_autoplaced yes)
-		(property "Reference" "#PWR012"
+		(property "Reference" "#PWR072"
 			(at 137.16 99.06 0)
 			(effects
@@
 			(project "Commodore 7.67"
 				(path "/92fa3f49-0e94-4664-860a-d244369fb976/068aab43-7d3e-4c07-94df-f9ae785d2fce"
-					(reference "#PWR012")
-					(unit 1)
-				)
+					(reference "#PWR072")
+					(unit 1)
+				)
