File: KiCad/Commodore 7.67/SX1281.kicad_sch (KiCad schematic)
At the start: 17 parts, among them U1 SX1281IMLTRT, U3 LPF-B0R3

Commit message: hello twin backup + commits
Connections:
- net RFIO: now reaches C17.2, C18.2
Changed lines of the file:
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@@
+		)
+	)
+	(hierarchical_label "RFIO"
+		(shape input)
+		(at 218.44 107.95 90)
+		(effects
+			(font
+				(size 1.27 1.27)
+			)
+			(justify left)
 		)
 	)

Commit message: yay done
Parts:
- removed R5, R6: 1k, symbol Device:R_Small_US
Connections:
- net SX_MISO: now reaches U1.16 (MISO_TX)
- net SX_MOSI: now reaches U1.17 (MOSI_RX)
- net SX_SCK: now reaches U1.18 (SCK_~{RTS})
- net SX_CS: now reaches U1.19 (~{SS_CTS})
Changed lines of the file:
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@@
+	(wire
+		(pts
+			(xy 99.06 90.17) (xy 104.14 90.17)
+		)
+		(stroke
+			(width 0)
+			(type default)
+		)
+	)
 	(wire
 		(pts
@@
 	(wire
 		(pts
-			(xy 83.82 92.71) (xy 96.52 92.71)
-		)
-		(stroke
-			(width 0)
-			(type default)
-		)
-	)
-	(wire
-		(pts
 			(xy 167.64 57.15) (xy 167.64 67.31)
 		)
@@
 	(wire
 		(pts
-			(xy 93.98 90.17) (xy 104.14 90.17)
-		)
-		(stroke
-			(width 0)
-			(type default)
-		)
-	)
-	(wire
-		(pts
 			(xy 151.13 115.57) (xy 151.13 118.11)
 		)
@@
 	(wire
 		(pts
+			(xy 88.9 92.71) (xy 104.14 92.71)
+		)
+		(stroke
+			(width 0)
+			(type default)
+		)
+	)
+	(wire
+		(pts
 			(xy 156.21 67.31) (xy 161.29 67.31)
 		)
@@
 	(wire
 		(pts
+			(xy 68.58 97.79) (xy 104.14 97.79)
+		)
+		(stroke
+			(width 0)
+			(type default)
+		)
+	)
+	(wire
+		(pts
 			(xy 177.8 67.31) (xy 180.34 67.31)
 		)
@@
 	(wire
 		(pts
-			(xy 101.6 92.71) (xy 104.14 92.71)
-		)
-		(stroke
-			(width 0)
-			(type default)
-		)
-	)
-	(wire
-		(pts
 			(xy 151.13 123.19) (xy 151.13 125.73)
 		)
@@
 	(wire
 		(pts
+			(xy 78.74 95.25) (xy 104.14 95.25)
+		)
+		(stroke
+			(width 0)
+			(type default)
+		)
+	)
+	(wire
+		(pts
 			(xy 177.8 67.31) (xy 177.8 77.47)
 		)
@@
 		(pts
 			(xy 144.78 128.27) (xy 151.13 128.27)
-		)
-		(stroke
-			(width 0)
-			(type default)
-		)
-	)
-	(wire
-		(pts
-			(xy 83.82 90.17) (xy 88.9 90.17)
 		)
 		(stroke
@@
 		)
 	)
-	(hierarchical_label "SX_1281_TX"
+	(hierarchical_label "SX_CS"
 		(shape output)
-		(at 83.82 90.17 180)
+		(at 68.58 97.79 180)
 		(effects
 			(font
@@
 		)
 	)
-	(hierarchical_label "SX_1281_RX"
-		(shape input)
-		(at 83.82 92.71 180)
+	(hierarchical_label "SX_MOSI"
+		(shape output)
+		(at 88.9 92.71 180)
+		(effects
+			(font
+				(size 1.27 1.27)
+			)
+			(justify right)
+		)
+	)
+	(hierarchical_label "SX_SCK"
+		(shape output)
+		(at 78.74 95.25 180)
+		(effects
+			(font
+				(size 1.27 1.27)
+			)
+			(justify right)
+		)
+	)
+	(hierarchical_label "SX_MISO"
+		(shape output)
+		(at 99.06 90.17 180)
 		(effects
 			(font
@@
 	)
 	(symbol
-		(lib_id "Device:R_Small_US")
-		(at 91.44 90.17 90)
-		(unit 1)
-		(exclude_from_sim no)
-		(in_bom yes)
-		(on_board yes)
-		(dnp no)
-		(fields_autoplaced yes)
-		(property "Reference" "R5"
-			(at 91.44 83.82 90)
-			(effects
-				(font
-					(size 1.27 1.27)
-				)
-			)
-		)
-		(property "Value" "1k"
-			(at 91.44 86.36 90)
-			(effects
-				(font
-					(size 1.27 1.27)
-				)
-			)
-		)
-		(property "Footprint" ""
-			(at 91.44 90.17 0)
-			(effects
-				(font
-					(size 1.27 1.27)
-				)
-				(hide yes)
-			)
-		)
-		(property "Datasheet" "~"
-			(at 91.44 90.17 0)
-			(effects
-				(font
-					(size 1.27 1.27)
-				)
-				(hide yes)
-			)
-		)
-		(property "Description" "Resistor, small US symbol"
-			(at 91.44 90.17 0)
-			(effects
-				(font
-					(size 1.27 1.27)
-				)
-				(hide yes)
-			)
-		)
-		(pin "2"
-		)
-		(pin "1"
-		)
-		(instances
-			(project "Commodore 7.67"
-				(path "/92fa3f49-0e94-4664-860a-d244369fb976/e7924f5e-fb39-4d19-9111-29029f4b1022"
-					(reference "R5")
-					(unit 1)
-				)
-			)
-		)
-	)
-	(symbol
 		(lib_id "power:GND")
 		(at 152.4 67.31 180)
@@
 					(unit 1)
 				)
-			)
-		)
-	)
-	(symbol
-		(lib_id "Device:R_Small_US")
-		(at 99.06 92.71 90)
-		(unit 1)
-		(exclude_from_sim no)
-		(in_bom yes)
-		(on_board yes)
-		(dnp no)
-		(fields_autoplaced yes)
-		(property "Reference" "R6"
-			(at 99.06 86.36 90)
-			(effects
-				(font
-					(size 1.27 1.27)
-				)
-			)
-		)
-		(property "Value" "1k"
-			(at 99.06 88.9 90)
-			(effects
-				(font
-					(size 1.27 1.27)
-				)
-			)
-		)
-		(property "Footprint" ""
-			(at 99.06 92.71 0)
-			(effects
-				(font
-					(size 1.27 1.27)
-				)
-				(hide yes)
-			)
-		)
-		(property "Datasheet" "~"
-			(at 99.06 92.71 0)
-			(effects
-				(font
-					(size 1.27 1.27)
-				)
-				(hide yes)
-			)
-		)
-		(property "Description" "Resistor, small US symbol"
-			(at 99.06 92.71 0)
-			(effects
-				(font
-					(size 1.27 1.27)
-				)
-				(hide yes)
-			)
-		)
-		(pin "2"
-		)
-		(pin "1"
-		)
-		(instances
-			(project "Commodore 7.67"
-				(path "/92fa3f49-0e94-4664-860a-d244369fb976/e7924f5e-fb39-4d19-9111-29029f4b1022"
-					(reference "R6")
-					(unit 1)
-				)

Commit message: oopsies
Parts:
- removed U3: LPF-B0R3, RF_Mini-Circuits:Mini-Circuits_HZ1198_LandPatternPL-247, symbol RF_Filter:LPF-B0R3
Connections:
- net at C16.2, C18.1: now also U1.22 (RFIO)
Other:
- moved on the sheet: C10, C11, C12, C13, C14, C15, C16, C17, C18, L1, R1, R10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

Commit message: its over
Parts:
- renumbered C15 to C1, C11 to C2, C10 to C3, C16 to C4, C12 to C5, C13 to C6, C14 to C7, C18 to C8, C17 to C9, R11 to R2, R10 to R3, U1 to U2
Other:
- moved on the sheet: C1, C2, C3, C4, C5, C6, C7, C8, C9, L1, R1, R2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
