File: KiCad/C6_v1.0/C6v1.0/C6v1.0.kicad_sch (KiCad schematic)
At the start: 0 parts

Commit message: Updated IO on shi
Other:
- added sheet IO_Connections (IO_Connections.kicad_sch)
- sheet STM32 ports: added 3V3, GND; removed none

Commit message: FK TS PMO GGKMSRQTOGIW
Parts:
- added H1, H2, H3, H4: MountingHole, MountingHole:MountingHole_2.2mm_M2_Pad, symbol Mechanical:MountingHole
Other:
- added sheet CameraManagement (CameraManagement.kicad_sch)
- added sheet LevelShifting (LevelShifting.kicad_sch)
- sheet IO_Connections ports: added 8V4, CLK, MISO, MOSI, NSS, RRC3_RX, RRC3_TX; removed none
- sheet STM32 ports: added 2V8, CAM_D0, CAM_D1, CAM_D2, CAM_D3, CAM_D4, CAM_D5, CAM_D6, CAM_D7, CAM_HSYNC, CAM_PIXCLK, CAM_PWDN, CAM_RST, CAM_RX, CAM_SCL, CAM_SDA, CAM_TX, CAM_VSYNC, DCD_PWDN, DCD_RST, NTSC_INTR, OV_OE, PPS, RRC3_RX, RRC3_TX, RX+, RX-, SPLIT_OE, TRX_SPI_MISO, TRX_SPI_MOSI*, TRX_SPI_NSS*, TRX_SPI_SCK*, TX+, TX-; removed none
