File: KiCad/C6_v1.0/C6v1.0/IO_Connections.kicad_sch (KiCad schematic)
At the start: 2 parts, among them J1 FH12-24S-0.5SH_55_, J2 Conn_01x06

Commit message: FK TS PMO GGKMSRQTOGIW
Parts:
- added J3: Conn_01x06, Connector_JST:JST_XA_B06B-XASK-1_1x06_P2.50mm_Vertical, symbol Connector_Generic:Conn_01x06
- added J5: Conn_01x05_Socket, Connector_PinSocket_2.00mm:PinSocket_1x05_P2.00mm_Vertical, symbol Connector:Conn_01x05_Socket
Connections:
- net GND: now also J3.5 (Pin_5), J5.5 (Pin_5)
- new net 8V4: J3.6 (Pin_6)
- new net CLK: J3.2 (Pin_2)
- new net MISO: J3.3 (Pin_3)
- new net MOSI: J3.4 (Pin_4)
- new net NSS: J3.1 (Pin_1)
- new net RRC3_RX: J5.3 (Pin_3)
- new net RRC3_TX: J5.4 (Pin_4)
Other:
- note added: "Straight up transmittin my shi I got modulation all over my shi"
