File: KiCad/C6_v1.0/C6v1.0/STM32.kicad_sch (KiCad schematic)
At the start: 22 parts, among them J1 Conn_01x06_Pin, J2 Conn_01x06_Pin, U1 STM32H562RITx, U2 STM32H7A3RITx

Commit message: Updated IO on shi
Connections:
- net CAM_SCL*: now reaches U2.8 (PC0)
- net CAM_SDA*: now reaches U2.9 (PC1)
Other:
- sheet Peripheral ports: added CAM_SCL, CAM_SCL*, CAM_SDA, CAM_SDA*; removed none

Commit message: FK TS PMO GGKMSRQTOGIW
Parts:
- added R23, R24: 10k, Resistor_SMD:R_0805_2012Metric, symbol Device:R
- added U7: MAX3490xSA, Package_SO:SOIC-8_3.9x4.9mm_P1.27mm, symbol Interface_UART:MAX3490xSA
Connections:
- net CAM_SCL* is gone; now on net CAM_SCL: U2.8 (PC0)
- net CAM_SDA* is gone; now on net CAM_SDA: U2.9 (PC1)
- net 3V3: now also R23.2, R24.2, U7.1 (VCC)
- net GND: now also U7.4 (GND)
- net TRX_SPI_MISO: now also U1.43 (PA10); no longer U1.52 (PC11)
- net TRX_SPI_MOSI: now also U1.44 (PA11); no longer U1.53 (PC12)
- net TRX_SPI_NSS: now also U1.41 (PA8); no longer U1.50 (PA15(JTDI))
- net TRX_SPI_SCK: now also U1.42 (PA9); no longer U1.51 (PC10)
- net SPLIT_OE: now reaches U2.10 (PC2)
- net SPLIT_OE: now also R23.1
- net OV_OE: now reaches U2.11 (PC3)
- net OV_OE: now also R24.1
- net PPS: now reaches U2.21 (PA5)
- net PPS: now also U1.21 (PA5)
- net DCD_RST: now reaches U2.26 (PB0)
- net DCD_PWDN: now reaches U2.27 (PB1)
- net TX: now reaches U1.14 (PA0)
- net TX: now also U7.3 (DI)
- net RX: now reaches U1.15 (PA1)
- net RX: now also U7.2 (RO)
- net RRC3_TX: now reaches U1.37 (PC6)
- net RRC3_RX: now reaches U1.38 (PC7)
- net SDMMC1_D0: now reaches U1.39 (PC8)
- net SDMMC1_D1: now reaches U1.40 (PC9)
- net SDMMC1_CMD: now reaches U1.54 (PD2)
- new net RX+: U7.6 (Z)
- new net RX-: U7.5 (Y)
- new net SDMMC1_CK: U1.53 (PC12)
- new net SDMMC1_D2: U1.51 (PC10)
- new net SDMMC1_D3: U1.52 (PC11)
- new net TX+: U7.8 (A)
- new net TX-: U7.7 (B)
Other:
- added sheet SDCardBS (SDCARDBS.kicad_sch)
- sheet Peripheral ports: added none; removed CAM_SCL, CAM_SCL*, CAM_SDA, CAM_SDA*
