File: KiCad/G6/G6.kicad_sch (KiCad schematic)
At the start: 0 parts

Commit message: uhhh idk
Parts:
- added D1: IR26-21C_L110_TR8, LED_SMD:LED_1206_3216Metric, symbol LED:IR26-21C_L110_TR8
- added J2: Conn_02x20_Odd_Even_MountingPin, Connector_PinHeader_2.54mm:PinHeader_2x20_P2.54mm_Vertical, symbol Connector_Generic_MountingPin:Conn_02x20_Odd_Even_MountingPin
- added Q1: 2N3904, Package_TO_SOT_THT:TO-92_Inline, symbol Transistor_BJT:2N3904
- added R10: 10k, Resistor_SMD:R_1206_3216Metric, symbol Device:R
- added R11, R12: 1k, Resistor_SMD:R_1206_3216Metric, symbol Device:R
- added U11: SN74HC74DRG4 (SOIC14), Package_SO:SOIC-14_3.9x8.7mm_P1.27mm, symbol MCU_Microchip_PIC16:PIC16F18324-xSL
Connections:
- new net: R10.2, U11.1 (VDD)
- new net: D1.1 (K), R12.2
- new net: Q1.2 (B), R11.2
- new net: Q1.3 (C), R12.1
- new net: U11.2 (RA5), U11.6 (RC4)
- new net: R11.1, U11.5 (RC5)
- new net 3.3v: D1.2 (A), J2.5 (Pin_5), J2.6 (Pin_6), R10.1, U11.14 (VSS)
- new net 5v: J2.10 (Pin_10), J2.9 (Pin_9)
- new net GNDD: J2.1 (Pin_1), J2.15 (Pin_15), J2.16 (Pin_16), J2.19 (Pin_19), J2.2 (Pin_2), J2.20 (Pin_20), J2.27 (Pin_27), J2.28 (Pin_28), J2.35 (Pin_35), J2.36 (Pin_36), J2.7 (Pin_7), J2.8 (Pin_8), Q1.1 (E), U11.7 (RC3)
- new net GPIO: J2.24 (Pin_24), J2.25 (Pin_25)
- new net I2C-MAIN-RESET: J2.31 (Pin_31)
- new net I2C-SCL-MAIN: J2.4 (Pin_4)
- new net I2C-SDA-MAIN: J2.3 (Pin_3)
- new net IIM-MAIN-INT: J2.29 (Pin_29)
- new net INT-MMC: J2.30 (Pin_30)
- new net INT1-BMI: J2.32 (Pin_32)
- new net INT2-BMI: J2.34 (Pin_34)
- new net MISO: J2.11 (Pin_11)
- new net MOSI: J2.12 (Pin_12)
- new net PPS: J2.23 (Pin_23), U11.3 (RA4)
- new net SCK: J2.26 (Pin_26)
- new net VBATT: J2.13 (Pin_13), J2.14 (Pin_14)
- new net a+: J2.22 (Pin_22)
- new net a-: J2.21 (Pin_21)
- new net y+: J2.17 (Pin_17)
- new net y-: J2.18 (Pin_18)
Other:
- added sheet BMI270 (BMI270.kicad_sch)
- added sheet GPS (GPS.kicad_sch)
- added sheet I2C Buffer (I2C Buffer.kicad_sch)
- added sheet IIM-42652 (MAIN CONNECTION.kicad_sch)
- added sheet MMC5983 (MMC5983.kicad_sch)
- added sheet MS560702 (MS560702.kicad_sch)
- added sheet TMP112 (TMP112.kicad_sch)
- added sheet Transceiver (Transceiver.kicad_sch)
- note added: "BMI: 0X69"
- note added: "I2C ADDRESS:"
- note added: "MMC: 0X30"
- note added: "MS5: 0X76"
- note added: "MUX: 0x70 IIM: 0x68"
- note added: "PPS Status"
- note added: "Temp: 0x48"

Commit message: i finally finished routing everything to spi
Other:
- added sheet IIM-42653 (IIM-42653.kicad_sch)
- added sheet STM (STM.kicad_sch)
Changed lines of the file:
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@@
+	)
+	(sheet
+		(at 137.16 173.99)
+		(size 33.02 16.51)
+		(exclude_from_sim no)
+		(in_bom yes)
+		(on_board yes)
+		(dnp no)
+		(fields_autoplaced yes)
+		(stroke
+			(width 0.1524)
+			(type solid)
+		)
+		(fill
+			(color 0 0 0 0.0000)
+		)
+		(property "Sheetname" "IIM-42653"
+			(at 137.16 173.2784 0)
+			(effects
+				(font
+					(size 1.27 1.27)
+				)
+				(justify left bottom)
+			)
+		)
+		(property "Sheetfile" "IIM-42653.kicad_sch"
+			(at 137.16 191.0846 0)
+			(effects
+				(font
+					(size 1.27 1.27)
+				)
+				(justify left top)
+			)
+		)
+		(instances
+			(project "G6"
+				(path "/99017594-210d-4d15-87a7-3152ef0d7b7c"
+					(page "10")
+				)
+			)
+		)
 	)
 	(sheet
@@
 				)
 			)
+		)
+	)
+	(sheet
+		(at 102.87 149.86)
+		(size 26.67 22.86)
+		(exclude_from_sim no)
+		(in_bom yes)
+		(on_board yes)
+		(dnp no)
+		(fields_autoplaced yes)
+		(stroke
+			(width 0.1524)
+			(type solid)
+		)
+		(fill
+			(color 0 0 0 0.0000)
+		)
+		(property "Sheetname" "STM"
+			(at 102.87 149.1484 0)
+			(effects
+				(font
+					(size 1.27 1.27)
+				)
+				(justify left bottom)
+			)
+		)
+		(property "Sheetfile" "STM.kicad_sch"
+			(at 102.87 173.3046 0)
+			(effects
+				(font
+					(size 1.27 1.27)
+				)
+				(justify left top)
+			)
+		)
+		(instances
+			(project "G6"
+				(path "/99017594-210d-4d15-87a7-3152ef0d7b7c"
+					(page "11")
+				)
+			)

Commit message: I think the schematics done uhhh idrk
Parts:
- added J1: Conn_02x10_Odd_Even, Connector_PinHeader_2.54mm:PinHeader_2x10_P2.54mm_Vertical, symbol Connector_Generic:Conn_02x10_Odd_Even
- added U8: ISL83488IBZ, CC0603KRXQRQBB104:SOIC8_4X5_INR, symbol ISL83488IBZ:ISL83488IBZ
Connections:
- net 3.3v: now also J1.3 (Pin_3), J1.4 (Pin_4)
- net 5v: now also J1.7 (Pin_7), J1.8 (Pin_8)
- net GNDD: now also J1.1 (Pin_1), J1.10 (Pin_10), J1.15 (Pin_15), J1.16 (Pin_16), J1.18 (Pin_18), J1.19 (Pin_19), J1.2 (Pin_2), J1.20 (Pin_20), J1.5 (Pin_5), J1.6 (Pin_6), J1.9 (Pin_9)
- net PPS: now also J1.17 (Pin_17)
- net a+: now also J1.12 (Pin_12)
- net a-: now also J1.14 (Pin_14)
- net y+: now also J1.11 (Pin_11)
- net y-: now also J1.13 (Pin_13)
Other:
- removed sheet IIM-42652
- sheet BMI270 ports: added CS-BMI, MISO-BMI, MOSI-BMI, SCK-MAIN; removed none
- sheet IIM-42653 ports: added CS-IIM1, CS-IIM2, MISO-IIM1, MISO-IIM2, MOSI-IIM1, MOSI-IIM2, SCK-MAIN; removed none
- sheet MMC5983 ports: added CS-MMC, MISO-MMC, MOSI-MMC, SCK-MAIN; removed none
- sheet MS560702 ports: added CS-MS5, MISO-MS5, MOSI-MS5, SCK-MAIN; removed none
- sheet STM ports: added CS-BMI, CS-IIM1, CS-IIM2, CS-MMC, CS-MS5, CS-TMP, MISO-BMI, MISO-IIM1, MISO-IIM2, MISO-MMC, MISO-MS5, MISO-TMP, MOSI-BMI, MOSI-IIM1, MOSI-IIM2, MOSI-MMC, MOSI-MS5, MOSI-TMP, SCK-MAIN; removed none
- sheet TMP112 ports: added CS-TMP, MISO-TMP, MOSI-TMP, SCK-MAIN; removed none
- note removed: "BMI: 0X69"
- note removed: "I2C ADDRESS:"
- note removed: "MMC: 0X30"
- note removed: "MS5: 0X76"
- note removed: "MUX: 0x70 IIM: 0x68"
- note removed: "Temp: 0x48"

Commit message: im sorry parsa :/
Parts:
- removed J2: Conn_02x20_Odd_Even_MountingPin, Connector_PinHeader_2.54mm:PinHeader_2x20_P2.54mm_Vertical, symbol Connector_Generic_MountingPin:Conn_02x20_Odd_Even_MountingPin
Other:
- removed sheet I2C Buffer
- moved on the sheet: J1

Commit message: sasha sneaky academic
Parts:
- removed R10: 10k, Resistor_SMD:R_1206_3216Metric, symbol Device:R
- removed U8: ISL83488IBZ, CC0603KRXQRQBB104:SOIC8_4X5_INR, symbol ISL83488IBZ:ISL83488IBZ
- renumbered R11 to R1, R12 to R2, U11 to U2
Connections:
- net 3.3v: now also U2.1 (VDD); no longer U2.14 (VSS)
- net GNDD: no longer Q1.1 (E), U2.7 (RC3)
- new net GND: Q1.1 (E), U2.14 (VSS)

Commit message: errrrrr i cant find a umcx connector they all say there like $50??
Other:
- sheet GPS ports: added CS-GPS, GPIO, MISO-GPS, MOSI-GPS, PPS, SCK-MAIN; removed none
- sheet STM ports: added CS-GPS, MISO-GPS, MOSI-GPS; removed none

Commit message: i have no idea whats going on, everything crashed and nothing will open
Other:
- sheet STM ports: added RX, TX; removed none
- sheet Transceiver ports: added RX, TX; removed none

Commit message: g6
Connections:
- net GNDD is gone; now on net GND: J1.1 (Pin_1), J1.10 (Pin_10), J1.15 (Pin_15), J1.16 (Pin_16), J1.18 (Pin_18), J1.19 (Pin_19), J1.2 (Pin_2), J1.20 (Pin_20), J1.5 (Pin_5), J1.6 (Pin_6), J1.9 (Pin_9)
- net a+: now also J1.14 (Pin_14); no longer J1.12 (Pin_12)
- net a-: now also J1.12 (Pin_12); no longer J1.14 (Pin_14)
- net y+: now also J1.13 (Pin_13); no longer J1.11 (Pin_11)
- net y-: now also J1.11 (Pin_11); no longer J1.13 (Pin_13)
Other:
- sheet STM ports: added GPIO; removed none
- moved on the sheet: J1
