File: KiCad/G6/MS560702.kicad_sch (KiCad schematic)
At the start: 1 part, among them U5 MS560702BA03-50 - Barometer

Commit message: i finally finished routing everything to spi
Parts:
- added C18: .01uF, CC0603KRXQRQBB104:.01YAG_CC1206_YAG, symbol Device:C
Connections:
- net 3.3v: now also C18.2; no longer U5.2 (PS)
- net GNDD: now also U5.2 (PS), C18.1; no longer U5.4 (~{CSB}), U5.6 (SDO)
- net I2C-SCL-MAIN renamed SPI-SCK-MAIN
- net I2C-SDA-MAIN renamed SPI-SDI-MAIN
- new net CS-MS5: U5.4 (~{CSB})
- new net SPI-SDO-MAIN: U5.6 (SDO)
Changed lines of the file:
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@@
 	(generator_version "9.0")
 	(paper "A4")
+	(junction
+		(at 165.1 82.55)
+		(diameter 0)
+		(color 0 0 0 0)
+	)
 	(wire
 		(pts
@@
 	(wire
 		(pts
-			(xy 158.75 82.55) (xy 167.64 82.55)
+			(xy 165.1 82.55) (xy 167.64 82.55)
 		)
 		(stroke
@@
 	(wire
 		(pts
-			(xy 110.49 90.17) (xy 128.27 90.17)
+			(xy 158.75 82.55) (xy 165.1 82.55)
 		)
 		(stroke
@@
 	(wire
 		(pts
-			(xy 125.73 87.63) (xy 128.27 87.63)
+			(xy 110.49 90.17) (xy 128.27 90.17)
 		)
 		(stroke
@@
 		)
 	)
-	(global_label "I2C-SCL-MAIN"
+	(global_label "SPI-SCK-MAIN"
 		(shape input)
 		(at 110.49 90.17 180)
@@
 		)
 		(property "Intersheetrefs" "${INTERSHEET_REFS}"
-			(at 93.2928 90.17 0)
+			(at 93.0509 90.17 0)
 			(effects
 				(font
@@
 		)
 	)
-	(global_label "I2C-SDA-MAIN"
+	(global_label "CS-MS5"
 		(shape input)
-		(at 110.49 95.25 180)
+		(at 128.27 82.55 180)
 		(fields_autoplaced yes)
 		(effects
@@
 		)
 		(property "Intersheetrefs" "${INTERSHEET_REFS}"
-			(at 93.2323 95.25 0)
+			(at 117.3625 82.55 0)
 			(effects
 				(font
@@
 		)
 	)
-	(global_label "3.3v"
+	(global_label "SPI-SDI-MAIN"
 		(shape input)
-		(at 125.73 87.63 180)
+		(at 110.49 95.25 180)
 		(fields_autoplaced yes)
 		(effects
@@
 		)
 		(property "Intersheetrefs" "${INTERSHEET_REFS}"
-			(at 118.7534 87.63 0)
+			(at 93.7161 95.25 0)
 			(effects
 				(font
@@
 		)
 	)
+	(global_label "SPI-SDO-MAIN"
+		(shape input)
+		(at 158.75 87.63 0)
+		(fields_autoplaced yes)
+		(effects
+			(font
+				(size 1.27 1.27)
+			)
+			(justify left)
+		)
+		(property "Intersheetrefs" "${INTERSHEET_REFS}"
+			(at 176.2496 87.63 0)
+			(effects
+				(font
+					(size 1.27 1.27)
+				)
+				(justify left)
+				(hide yes)
+			)
+		)
+	)
 	(symbol
-		(lib_id "power:GNDD")
-		(at 128.27 82.55 270)
+		(lib_id "Device:C")
+		(at 165.1 78.74 0)
 		(unit 1)
 		(exclude_from_sim no)
@@
 		(dnp no)
 		(fields_autoplaced yes)
-		(property "Reference" "#PWR021"
-			(at 121.92 82.55 0)
+		(property "Reference" "C18"
+			(at 168.91 77.4699 0)
+			(effects
+				(font
+					(size 1.27 1.27)
+				)
+				(justify left)
+			)
+		)
+		(property "Value" ".01uF"
+			(at 168.91 80.0099 0)
+			(effects
+				(font
+					(size 1.27 1.27)
+				)
+				(justify left)
+			)
+		)
+		(property "Footprint" "CC0603KRXQRQBB104:.01YAG_CC1206_YAG"
+			(at 166.0652 82.55 0)
+			(effects
+				(font
+					(size 1.27 1.27)
+				)
+				(hide yes)
+			)
+		)
+		(property "Datasheet" "~"
+			(at 165.1 78.74 0)
+			(effects
+				(font
+					(size 1.27 1.27)
+				)
+				(hide yes)
+			)
+		)
+		(property "Description" "Unpolarized capacitor"
+			(at 165.1 78.74 0)
+			(effects
+				(font
+					(size 1.27 1.27)
+				)
+				(hide yes)
+			)
+		)
+		(pin "1"
+		)
+		(pin "2"
+		)
+		(instances
+			(project ""
+				(path "/99017594-210d-4d15-87a7-3152ef0d7b7c/d6c1a486-cb9f-412b-8709-54bd623c2a86"
+					(reference "C18")
+					(unit 1)
+				)
+			)
+		)
+	)
+	(symbol
+		(lib_id "power:GNDD")
+		(at 128.27 87.63 270)
+		(unit 1)
+		(exclude_from_sim no)
+		(in_bom yes)
+		(on_board yes)
+		(dnp no)
+		(fields_autoplaced yes)
+		(property "Reference" "#PWR066"
+			(at 121.92 87.63 0)
 			(effects
 				(font
@@
 		)
 		(property "Value" "GNDD"
-			(at 124.46 82.5499 90)
+			(at 124.46 87.6299 90)
 			(effects
 				(font
@@
 		)
 		(property "Footprint" ""
-			(at 128.27 82.55 0)
+			(at 128.27 87.63 0)
 			(effects
 				(font
@@
 		)
 		(property "Datasheet" ""
-			(at 128.27 82.55 0)
+			(at 128.27 87.63 0)
 			(effects
 				(font
@@
 		)
 		(property "Description" "Power symbol creates a global label with name \"GNDD\" , digital ground"
-			(at 128.27 82.55 0)
+			(at 128.27 87.63 0)
 			(effects
 				(font
@@
 		)
 		(instances
-			(project "G6"
+			(project ""
 				(path "/99017594-210d-4d15-87a7-3152ef0d7b7c/d6c1a486-cb9f-412b-8709-54bd623c2a86"
-					(reference "#PWR021")
+					(reference "#PWR066")
 					(unit 1)
 				)
@@
 	)
 	(symbol
-		(lib_id "power:GNDD")
-		(at 158.75 87.63 90)
-		(unit 1)
-		(exclude_from_sim no)
-		(in_bom yes)
-		(on_board yes)
-		(dnp no)
-		(fields_autoplaced yes)
-		(property "Reference" "#PWR023"
-			(at 165.1 87.63 0)
-			(effects
-				(font
-					(size 1.27 1.27)
-				)
-				(hide yes)
-			)
-		)
-		(property "Value" "GNDD"
-			(at 162.56 87.6299 90)
-			(effects
-				(font
-					(size 1.27 1.27)
-				)
-				(justify right)
-			)
-		)
-		(property "Footprint" ""
-			(at 158.75 87.63 0)
-			(effects
-				(font
-					(size 1.27 1.27)
-				)
-				(hide yes)
-			)
-		)
-		(property "Datasheet" ""
-			(at 158.75 87.63 0)
-			(effects
-				(font
-					(size 1.27 1.27)
-				)
-				(hide yes)
-			)
-		)
-		(property "Description" "Power symbol creates a global label with name \"GNDD\" , digital ground"
-			(at 158.75 87.63 0)
-			(effects
-				(font
-					(size 1.27 1.27)
-				)
-				(hide yes)
-			)
-		)
-		(pin "1"
-		)
-		(instances
-			(project "G6"
-				(path "/99017594-210d-4d15-87a7-3152ef0d7b7c/d6c1a486-cb9f-412b-8709-54bd623c2a86"
-					(reference "#PWR023")
-					(unit 1)
-				)
-			)
-		)
-	)
-	(symbol
 		(lib_id "MS560702BA03-50:MS560702BA03-50")
 		(at 143.51 87.63 0)
@@
 					(unit 1)
 				)
+			)
+		)
+	)
+	(symbol
+		(lib_id "power:GNDD")
+		(at 165.1 74.93 180)
+		(unit 1)
+		(exclude_from_sim no)
+		(in_bom yes)
+		(on_board yes)
+		(dnp no)
+		(fields_autoplaced yes)
+		(property "Reference" "#PWR021"
+			(at 165.1 68.58 0)
+			(effects
+				(font
+					(size 1.27 1.27)
+				)
+				(hide yes)
+			)
+		)
+		(property "Value" "GNDD"
+			(at 165.1 69.85 0)
+			(effects
+				(font
+					(size 1.27 1.27)
+				)
+			)
+		)
+		(property "Footprint" ""
+			(at 165.1 74.93 0)
+			(effects
+				(font
+					(size 1.27 1.27)
+				)
+				(hide yes)
+			)
+		)
+		(property "Datasheet" ""
+			(at 165.1 74.93 0)
+			(effects
+				(font
+					(size 1.27 1.27)
+				)
+				(hide yes)
+			)
+		)
+		(property "Description" "Power symbol creates a global label with name \"GNDD\" , digital ground"
+			(at 165.1 74.93 0)
+			(effects
+				(font
+					(size 1.27 1.27)
+				)
+				(hide yes)
+			)
+		)
+		(pin "1"
+		)
+		(instances
+			(project ""
+				(path "/99017594-210d-4d15-87a7-3152ef0d7b7c/d6c1a486-cb9f-412b-8709-54bd623c2a86"
+					(reference "#PWR021")
+					(unit 1)
+				)

Commit message: uhhhh im confused gang
Connections:
- net SPI-SDI-MAIN renamed SPI-SDI-MS5
- net SPI-SDO-MAIN renamed SPI-SDO-MS5
Changed lines of the file:
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@@
 		)
 	)
-	(global_label "SPI-SDI-MAIN"
+	(global_label "SPI-SDI-MS5"
 		(shape input)
 		(at 110.49 95.25 180)
@@
 		)
 		(property "Intersheetrefs" "${INTERSHEET_REFS}"
-			(at 93.7161 95.25 0)
+			(at 94.321 95.25 0)
 			(effects
 				(font
@@
 		)
 	)
-	(global_label "SPI-SDO-MAIN"
+	(global_label "SPI-SDO-MS5"
 		(shape input)
 		(at 158.75 87.63 0)
@@
 		)
 		(property "Intersheetrefs" "${INTERSHEET_REFS}"
-			(at 176.2496 87.63 0)
+			(at 175.6447 87.63 0)
 			(effects
 				(font

Commit message: I think the schematics done uhhh idrk
Connections:
- net SPI-SCK-MAIN renamed SCK-MAIN
- net SPI-SDI-MS5 renamed MOSI-MS5
- net SPI-SDO-MS5 renamed MISO-MS5
Changed lines of the file:
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@@
 		)
 	)
-	(global_label "SPI-SCK-MAIN"
+	(hierarchical_label "MISO-MS5"
 		(shape input)
-		(at 110.49 90.17 180)
-		(fields_autoplaced yes)
+		(at 158.75 87.63 0)
+		(effects
+			(font
+				(size 1.27 1.27)
+			)
+			(justify left)
+		)
+	)
+	(hierarchical_label "MOSI-MS5"
+		(shape input)
+		(at 110.49 95.25 180)
 		(effects
 			(font
@@
 			(justify right)
 		)
-		(property "Intersheetrefs" "${INTERSHEET_REFS}"
-			(at 93.0509 90.17 0)
-			(effects
-				(font
-					(size 1.27 1.27)
-				)
-				(justify right)
-				(hide yes)
-			)
-		)
 	)
-	(global_label "CS-MS5"
+	(hierarchical_label "CS-MS5"
 		(shape input)
 		(at 128.27 82.55 180)
-		(fields_autoplaced yes)
 		(effects
 			(font
@@
 			(justify right)
 		)
-		(property "Intersheetrefs" "${INTERSHEET_REFS}"
-			(at 117.3625 82.55 0)
-			(effects
-				(font
-					(size 1.27 1.27)
-				)
-				(justify right)
-				(hide yes)
-			)
-		)
 	)
-	(global_label "SPI-SDI-MS5"
+	(hierarchical_label "SCK-MAIN"
 		(shape input)
-		(at 110.49 95.25 180)
-		(fields_autoplaced yes)
+		(at 110.49 90.17 180)
 		(effects
 			(font
@@
 			(justify right)
 		)
-		(property "Intersheetrefs" "${INTERSHEET_REFS}"
-			(at 94.321 95.25 0)
-			(effects
-				(font
-					(size 1.27 1.27)
-				)
-				(justify right)
-				(hide yes)
-			)
-		)
 	)
-	(global_label "SPI-SDO-MS5"
-		(shape input)
-		(at 158.75 87.63 0)
-		(fields_autoplaced yes)
-		(effects
-			(font
-				(size 1.27 1.27)
-			)
-			(justify left)
-		)
-		(property "Intersheetrefs" "${INTERSHEET_REFS}"
-			(at 175.6447 87.63 0)
-			(effects
-				(font
-					(size 1.27 1.27)
-				)
-				(justify left)
-				(hide yes)
-			)
-		)
-	)

Commit message: sasha sneaky academic
Parts:
- renumbered C18 to C6, U5 to U7
Changed lines of the file:
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@@
 		(dnp no)
 		(fields_autoplaced yes)
-		(property "Reference" "C18"
+		(property "Reference" "C6"
 			(at 168.91 77.4699 0)
 			(effects
@@
 			(project ""
 				(path "/99017594-210d-4d15-87a7-3152ef0d7b7c/d6c1a486-cb9f-412b-8709-54bd623c2a86"
-					(reference "C18")
+					(reference "C6")
 					(unit 1)
 				)
@@
 		(dnp no)
 		(fields_autoplaced yes)
-		(property "Reference" "#PWR066"
+		(property "Reference" "#PWR035"
 			(at 121.92 87.63 0)
 			(effects
@@
 			(project ""
 				(path "/99017594-210d-4d15-87a7-3152ef0d7b7c/d6c1a486-cb9f-412b-8709-54bd623c2a86"
-					(reference "#PWR066")
+					(reference "#PWR035")
 					(unit 1)
 				)
@@
 		(dnp no)
 		(fields_autoplaced yes)
-		(property "Reference" "#PWR022"
+		(property "Reference" "#PWR034"
 			(at 121.92 85.09 0)
 			(effects
@@
 			(project "G6"
 				(path "/99017594-210d-4d15-87a7-3152ef0d7b7c/d6c1a486-cb9f-412b-8709-54bd623c2a86"
-					(reference "#PWR022")
+					(reference "#PWR034")
 					(unit 1)
 				)
@@
 		(dnp no)
 		(fields_autoplaced yes)
-		(property "Reference" "U5"
+		(property "Reference" "U7"
 			(at 143.51 74.93 0)
 			(effects
@@
 			(project "G6"
 				(path "/99017594-210d-4d15-87a7-3152ef0d7b7c/d6c1a486-cb9f-412b-8709-54bd623c2a86"
-					(reference "U5")
+					(reference "U7")
 					(unit 1)
 				)
@@
 		(dnp no)
 		(fields_autoplaced yes)
-		(property "Reference" "#PWR021"
+		(property "Reference" "#PWR037"
 			(at 165.1 68.58 0)
 			(effects
@@
 			(project ""
 				(path "/99017594-210d-4d15-87a7-3152ef0d7b7c/d6c1a486-cb9f-412b-8709-54bd623c2a86"
-					(reference "#PWR021")
+					(reference "#PWR037")
 					(unit 1)
 				)
@@
 		(dnp no)
 		(fields_autoplaced yes)
-		(property "Reference" "#PWR024"
+		(property "Reference" "#PWR036"
 			(at 165.1 92.71 0)
 			(effects
@@
 			(project "G6"
 				(path "/99017594-210d-4d15-87a7-3152ef0d7b7c/d6c1a486-cb9f-412b-8709-54bd623c2a86"
-					(reference "#PWR024")
-					(unit 1)
-				)
+					(reference "#PWR036")
+					(unit 1)
+				)

Commit message: g6
Connections:
- net GNDD renamed GND
Changed lines of the file:
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@@
 	)
 	(symbol
-		(lib_id "power:GNDD")
+		(lib_id "power:GND")
 		(at 128.27 87.63 270)
 		(unit 1)
@@
 			)
 		)
-		(property "Value" "GNDD"
+		(property "Value" "GND"
 			(at 124.46 87.6299 90)
 			(effects
@@
 			)
 		)
-		(property "Description" "Power symbol creates a global label with name \"GNDD\" , digital ground"
+		(property "Description" "Power symbol creates a global label with name \"GND\" , ground"
 			(at 128.27 87.63 0)
 			(effects
@@
 		)
 		(instances
-			(project ""
+			(project "G6"
 				(path "/99017594-210d-4d15-87a7-3152ef0d7b7c/d6c1a486-cb9f-412b-8709-54bd623c2a86"
 					(reference "#PWR035")
@@
 	)
 	(symbol
-		(lib_id "power:GNDD")
+		(lib_id "power:GND")
 		(at 128.27 85.09 270)
 		(unit 1)
@@
 			)
 		)
-		(property "Value" "GNDD"
+		(property "Value" "GND"
 			(at 124.46 85.0899 90)
 			(effects
@@
 			)
 		)
-		(property "Description" "Power symbol creates a global label with name \"GNDD\" , digital ground"
+		(property "Description" "Power symbol creates a global label with name \"GND\" , ground"
 			(at 128.27 85.09 0)
 			(effects
@@
 		)
 		(instances
+			(project ""
+				(path "/99017594-210d-4d15-87a7-3152ef0d7b7c/d6c1a486-cb9f-412b-8709-54bd623c2a86"
+					(reference "#PWR034")
+					(unit 1)
+				)
+			)
+		)
+	)
+	(symbol
+		(lib_id "power:GND")
+		(at 165.1 74.93 180)
+		(unit 1)
+		(exclude_from_sim no)
+		(in_bom yes)
+		(on_board yes)
+		(dnp no)
+		(fields_autoplaced yes)
+		(property "Reference" "#PWR037"
+			(at 165.1 68.58 0)
+			(effects
+				(font
+					(size 1.27 1.27)
+				)
+				(hide yes)
+			)
+		)
+		(property "Value" "GND"
+			(at 165.1 69.85 0)
+			(effects
+				(font
+					(size 1.27 1.27)
+				)
+			)
+		)
+		(property "Footprint" ""
+			(at 165.1 74.93 0)
+			(effects
+				(font
+					(size 1.27 1.27)
+				)
+				(hide yes)
+			)
+		)
+		(property "Datasheet" ""
+			(at 165.1 74.93 0)
+			(effects
+				(font
+					(size 1.27 1.27)
+				)
+				(hide yes)
+			)
+		)
+		(property "Description" "Power symbol creates a global label with name \"GND\" , ground"
+			(at 165.1 74.93 0)
+			(effects
+				(font
+					(size 1.27 1.27)
+				)
+				(hide yes)
+			)
+		)
+		(pin "1"
+		)
+		(instances
 			(project "G6"
 				(path "/99017594-210d-4d15-87a7-3152ef0d7b7c/d6c1a486-cb9f-412b-8709-54bd623c2a86"
-					(reference "#PWR034")
+					(reference "#PWR037")
+					(unit 1)
+				)
+			)
+		)
+	)
+	(symbol
+		(lib_id "power:GND")
+		(at 158.75 92.71 90)
+		(unit 1)
+		(exclude_from_sim no)
+		(in_bom yes)
+		(on_board yes)
+		(dnp no)
+		(fields_autoplaced yes)
+		(property "Reference" "#PWR036"
+			(at 165.1 92.71 0)
+			(effects
+				(font
+					(size 1.27 1.27)
+				)
+				(hide yes)
+			)
+		)
+		(property "Value" "GND"
+			(at 162.56 92.7099 90)
+			(effects
+				(font
+					(size 1.27 1.27)
+				)
+				(justify right)
+			)
+		)
+		(property "Footprint" ""
+			(at 158.75 92.71 0)
+			(effects
+				(font
+					(size 1.27 1.27)
+				)
+				(hide yes)
+			)
+		)
+		(property "Datasheet" ""
+			(at 158.75 92.71 0)
+			(effects
+				(font
+					(size 1.27 1.27)
+				)
+				(hide yes)
+			)
+		)
+		(property "Description" "Power symbol creates a global label with name \"GND\" , ground"
+			(at 158.75 92.71 0)
+			(effects
+				(font
+					(size 1.27 1.27)
+				)
+				(hide yes)
+			)
+		)
+		(pin "1"
+		)
+		(instances
+			(project "G6"
+				(path "/99017594-210d-4d15-87a7-3152ef0d7b7c/d6c1a486-cb9f-412b-8709-54bd623c2a86"
+					(reference "#PWR036")
 					(unit 1)
 				)
@@
 					(unit 1)
 				)
-			)
-		)
-	)
-	(symbol
-		(lib_id "power:GNDD")
-		(at 165.1 74.93 180)
-		(unit 1)
-		(exclude_from_sim no)
-		(in_bom yes)
-		(on_board yes)
-		(dnp no)
-		(fields_autoplaced yes)
-		(property "Reference" "#PWR037"
-			(at 165.1 68.58 0)
-			(effects
-				(font
-					(size 1.27 1.27)
-				)
-				(hide yes)
-			)
-		)
-		(property "Value" "GNDD"
-			(at 165.1 69.85 0)
-			(effects
-				(font
-					(size 1.27 1.27)
-				)
-			)
-		)
-		(property "Footprint" ""
-			(at 165.1 74.93 0)
-			(effects
-				(font
-					(size 1.27 1.27)
-				)
-				(hide yes)
-			)
-		)
-		(property "Datasheet" ""
-			(at 165.1 74.93 0)
-			(effects
-				(font
-					(size 1.27 1.27)
-				)
-				(hide yes)
-			)
-		)
-		(property "Description" "Power symbol creates a global label with name \"GNDD\" , digital ground"
-			(at 165.1 74.93 0)
-			(effects
-				(font
-					(size 1.27 1.27)
-				)
-				(hide yes)
-			)
-		)
-		(pin "1"
-		)
-		(instances
-			(project ""
-				(path "/99017594-210d-4d15-87a7-3152ef0d7b7c/d6c1a486-cb9f-412b-8709-54bd623c2a86"
-					(reference "#PWR037")
-					(unit 1)
-				)
-			)
-		)
-	)
-	(symbol
-		(lib_id "power:GNDD")
-		(at 158.75 92.71 90)
-		(unit 1)
-		(exclude_from_sim no)
-		(in_bom yes)
-		(on_board yes)
-		(dnp no)
-		(fields_autoplaced yes)
-		(property "Reference" "#PWR036"
-			(at 165.1 92.71 0)
-			(effects
-				(font
-					(size 1.27 1.27)
-				)
-				(hide yes)
-			)
-		)
-		(property "Value" "GNDD"
-			(at 162.56 92.7099 90)
-			(effects
-				(font
-					(size 1.27 1.27)
-				)
-				(justify right)
-			)
-		)
-		(property "Footprint" ""
-			(at 158.75 92.71 0)
-			(effects
-				(font
-					(size 1.27 1.27)
-				)
-				(hide yes)
-			)
-		)
-		(property "Datasheet" ""
-			(at 158.75 92.71 0)
-			(effects
-				(font
-					(size 1.27 1.27)
-				)
-				(hide yes)
-			)
-		)
-		(property "Description" "Power symbol creates a global label with name \"GNDD\" , digital ground"
-			(at 158.75 92.71 0)
-			(effects
-				(font
-					(size 1.27 1.27)
-				)
-				(hide yes)
-			)
-		)
-		(pin "1"
-		)
-		(instances
-			(project "G6"
-				(path "/99017594-210d-4d15-87a7-3152ef0d7b7c/d6c1a486-cb9f-412b-8709-54bd623c2a86"
-					(reference "#PWR036")
-					(unit 1)
-				)
