File: KiCad/G6/G6.kicad_pcb (KiCad board)
At the start: 4 copper layers, 42 parts, among them IC1 BGU7004,115, J1 Conn_02x10_Odd_Even, Q1 2N3904, U1 ISL83488IBZ, U10 IIM-42653, U11 IIM-42653, U12 STM32C051K8T6, U13 REG1117A-1.8, U2 SN74HC74DRG4 (SOIC14), U3 BMI270 - Secondary Accelerome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

Commit message: sneaky commit
Parts:
- moved J1 77.3 mm to (164.3, 101.7), turned to 180 degrees
Changed lines of the file:
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@@
 	(footprint "Connector_PinHeader_2.54mm:PinHeader_2x10_P2.54mm_Vertical"
 		(layer "F.Cu")
-		(at 119.26 38.83 90)
+		(at 164.255 101.69 180)
 		(descr "Through hole straight pin header, 2x10, 2.54mm pitch, double rows")
 		(tags "Through hole pin header THT 2x10 2.54mm double row")
 		(property "Reference" "J1"
-			(at 1.27 -2.38 90)
+			(at 1.27 -2.38 0)
 			(layer "F.SilkS")
 			(effects
@@
 		)
 		(property "Value" "Conn_02x10_Odd_Even"
-			(at 1.27 25.24 90)
+			(at 1.27 25.24 0)
 			(layer "F.Fab")
 			(effects
@@
 		)
 		(property "Datasheet" ""
-			(at 0 0 90)
+			(at 0 0 0)
 			(layer "F.Fab")
 			(hide yes)
@@
 		)
 		(property "Description" ""
-			(at 0 0 90)
+			(at 0 0 0)
 			(layer "F.Fab")
 			(hide yes)
@@
 		)
 		(fp_line
+			(start 1.27 1.27)
+			(end 1.27 -1.38)
+			(stroke
+				(width 0.12)
+				(type solid)
+			)
+			(layer "F.SilkS")
+		)
+		(fp_line
 			(start 1.27 -1.38)
 			(end 3.92 -1.38)
@@
 		)
 		(fp_line
+			(start -1.38 24.24)
+			(end 3.92 24.24)
+			(stroke
+				(width 0.12)
+				(type solid)
+			)
+			(layer "F.SilkS")
+		)
+		(fp_line
+			(start -1.38 1.27)
+			(end 1.27 1.27)
+			(stroke
+				(width 0.12)
+				(type solid)
+			)
+			(layer "F.SilkS")
+		)
+		(fp_line
+			(start -1.38 1.27)
+			(end -1.38 24.24)
+			(stroke
+				(width 0.12)
+				(type solid)
+			)
+			(layer "F.SilkS")
+		)
+		(fp_line
+			(start -1.38 0)
+			(end -1.38 -1.38)
+			(stroke
+				(width 0.12)
+				(type solid)
+			)
+			(layer "F.SilkS")
+		)
+		(fp_line
 			(start -1.38 -1.38)
 			(end 0 -1.38)
@@
 		)
 		(fp_line
-			(start -1.38 0)
-			(end -1.38 -1.38)
-			(stroke
-				(width 0.12)
-				(type solid)
-			)
-			(layer "F.SilkS")
-		)
-		(fp_line
-			(start 1.27 1.27)
-			(end 1.27 -1.38)
-			(stroke
-				(width 0.12)
-				(type solid)
-			)
-			(layer "F.SilkS")
-		)
-		(fp_line
-			(start -1.38 1.27)
-			(end 1.27 1.27)
-			(stroke
-				(width 0.12)
-				(type solid)
-			)
-			(layer "F.SilkS")
-		)
-		(fp_line
-			(start -1.38 1.27)
-			(end -1.38 24.24)
-			(stroke
-				(width 0.12)
-				(type solid)
-			)
-			(layer "F.SilkS")
-		)
-		(fp_line
-			(start -1.38 24.24)
-			(end 3.92 24.24)
-			(stroke
-				(width 0.12)
-				(type solid)
-			)
-			(layer "F.SilkS")
+			(start 4.32 24.63)
+			(end 4.32 -1.77)
+			(stroke
+				(width 0.05)
+				(type solid)
+			)
+			(layer "F.CrtYd")
 		)
 		(fp_line
@@
 		)
 		(fp_line
+			(start -1.77 24.63)
+			(end 4.32 24.63)
+			(stroke
+				(width 0.05)
+				(type solid)
+			)
+			(layer "F.CrtYd")
+		)
+		(fp_line
 			(start -1.77 -1.77)
 			(end -1.77 24.63)
@@
 		)
 		(fp_line
-			(start 4.32 24.63)
-			(end 4.32 -1.77)
-			(stroke
-				(width 0.05)
-				(type solid)
-			)
-			(layer "F.CrtYd")
-		)
-		(fp_line
-			(start -1.77 24.63)
-			(end 4.32 24.63)
-			(stroke
-				(width 0.05)
-				(type solid)
-			)
-			(layer "F.CrtYd")
+			(start 3.81 24.13)
+			(end -1.27 24.13)
+			(stroke
+				(width 0.1)
+				(type solid)
+			)
+			(layer "F.Fab")
 		)
 		(fp_line
@@
 		)
 		(fp_line
+			(start -1.27 24.13)
+			(end -1.27 0)
+			(stroke
+				(width 0.1)
+				(type solid)
+			)
+			(layer "F.Fab")
+		)
+		(fp_line
 			(start -1.27 0)
 			(end 0 -1.27)
@@
 			(layer "F.Fab")
 		)
-		(fp_line
-			(start 3.81 24.13)
-			(end -1.27 24.13)
-			(stroke
-				(width 0.1)
-				(type solid)
-			)
-			(layer "F.Fab")
-		)
-		(fp_line
-			(start -1.27 24.13)
-			(end -1.27 0)
-			(stroke
-				(width 0.1)
-				(type solid)
-			)
-			(layer "F.Fab")
-		)
 		(fp_text user "${REFERENCE}"
-			(at 1.27 11.43 0)
+			(at 1.27 11.43 90)
 			(layer "F.Fab")
 			(effects
@@
 		)
 		(pad "1" thru_hole rect
-			(at 0 0 90)
+			(at 0 0 180)
 			(size 1.7 1.7)
 			(drill 1)
@@
 		)
 		(pad "2" thru_hole circle
-			(at 2.54 0 90)
+			(at 2.54 0 180)
 			(size 1.7 1.7)
 			(drill 1)
@@
 		)
 		(pad "3" thru_hole circle
-			(at 0 2.54 90)
+			(at 0 2.54 180)
 			(size 1.7 1.7)
 			(drill 1)
@@
 		)
 		(pad "4" thru_hole circle
-			(at 2.54 2.54 90)
+			(at 2.54 2.54 180)
 			(size 1.7 1.7)
 			(drill 1)
@@
 		)
 		(pad "5" thru_hole circle
-			(at 0 5.08 90)
+			(at 0 5.08 180)
 			(size 1.7 1.7)
 			(drill 1)
@@
 		)
 		(pad "6" thru_hole circle
-			(at 2.54 5.08 90)
+			(at 2.54 5.08 180)
 			(size 1.7 1.7)
 			(drill 1)
@@
 		)
 		(pad "7" thru_hole circle
-			(at 0 7.62 90)
+			(at 0 7.62 180)
 			(size 1.7 1.7)
 			(drill 1)
@@
 		)
 		(pad "8" thru_hole circle
-			(at 2.54 7.62 90)
+			(at 2.54 7.62 180)
 			(size 1.7 1.7)
 			(drill 1)
@@
 		)
 		(pad "9" thru_hole circle
-			(at 0 10.16 90)
+			(at 0 10.16 180)
 			(size 1.7 1.7)
 			(drill 1)
@@
 		)
 		(pad "10" thru_hole circle
-			(at 2.54 10.16 90)
+			(at 2.54 10.16 180)
 			(size 1.7 1.7)
 			(drill 1)
@@
 		)
 		(pad "11" thru_hole circle
-			(at 0 12.7 90)
+			(at 0 12.7 180)
 			(size 1.7 1.7)
 			(drill 1)
@@
 		)
 		(pad "12" thru_hole circle
-			(at 2.54 12.7 90)
+			(at 2.54 12.7 180)
 			(size 1.7 1.7)
 			(drill 1)
@@
 		)
 		(pad "13" thru_hole circle
-			(at 0 15.24 90)
+			(at 0 15.24 180)
 			(size 1.7 1.7)
 			(drill 1)
@@
 		)
 		(pad "14" thru_hole circle
-			(at 2.54 15.24 90)
+			(at 2.54 15.24 180)
 			(size 1.7 1.7)
 			(drill 1)
@@
 		)
 		(pad "15" thru_hole circle
-			(at 0 17.78 90)
+			(at 0 17.78 180)
 			(size 1.7 1.7)
 			(drill 1)
@@
 		)
 		(pad "16" thru_hole circle
-			(at 2.54 17.78 90)
+			(at 2.54 17.78 180)
 			(size 1.7 1.7)
 			(drill 1)
@@
 		)
 		(pad "17" thru_hole circle
-			(at 0 20.32 90)
+			(at 0 20.32 180)
 			(size 1.7 1.7)
 			(drill 1)
@@
 		)
 		(pad "18" thru_hole circle
-			(at 2.54 20.32 90)
+			(at 2.54 20.32 180)
 			(size 1.7 1.7)
 			(drill 1)
@@
 		)
 		(pad "19" thru_hole circle
-			(at 0 22.86 90)
+			(at 0 22.86 180)
 			(size 1.7 1.7)
 			(drill 1)
@@
 		)
 		(pad "20" thru_hole circle
-			(at 2.54 22.86 90)
-			(size 1.7 1.7)
-			(drill 1)
+			(at 2.54 22.86 180)
+			(size 1.7 1.7)
+			(drill 1)

Commit message: g6
Parts:
- removed R6, R7: 10k, CC0603KRXQRQBB104:10kRC1206N_YAG
- added J2: CONMHF1-SMD-T, CONMHF1_SMD_T:TE_CONMHF1-SMD-T, F.Cu at (79.1, 69.7)
- added J3: FTSH-107-01-L-DV-K-A, FTSH_107_01_L_DV_K_A:SAMTEC_FTSH-107-01-L-DV-K-A, F.Cu at (142.0, 80.5)
- added R10: 10k, Resistor_SMD:R_0805_2012Metric, F.Cu at (92.7, 87.2)
- added R4: 100, Resistor_SMD:R_0805_2012Metric, F.Cu at (148.0, 79.1)
- added R5: 1k, Resistor_SMD:R_0805_2012Metric, F.Cu at (97.7, 87.2)
- moved R2 85.6 mm to (161.2, 145.4), turned to -90 degrees
- moved Q1 85.5 mm to (167.0, 141.7), turned to -90 degrees
- moved R1 84.4 mm to (161.0, 139.5), turned to -90 degrees
- moved D1 80.5 mm to (162.6, 150.0)
- moved U2 73.3 mm to (153.0, 142.0), turned to 180 degrees
- moved U1 66.1 mm to (163.0, 114.5), turned to 90 degrees
- moved U4 65.8 mm to (82.2, 75.9), turned to -90 degrees
- moved L1 63.6 mm to (82.2, 81.9), turned to -90 degrees
- moved R8 62.1 mm to (160.5, 107.5), turned to 0 degrees
- moved IC1 58.8 mm to (85.5, 82.4), turned to -90 degrees
- moved U13 57.6 mm to (85.5, 89.4), turned to 0 degrees
- moved R9 56.7 mm to (165.5, 107.5), turned to 180 degrees
- moved U5 48.7 mm to (95.0, 76.5), turned to 0 degrees
- moved C3 43.6 mm to (104.0, 69.6), turned to -90 degrees
- moved C15 12.7 mm to (116.5, 97.5), turned to 90 degrees
Connections:
- net Net-(U12-PF2-NRST) renamed /STM/NRST
- C16 pad 2: Net-(U12-PC15-OSCX_OUT) -> /STM/OSCX_IN
- C17 pad 2: Net-(U12-PC14-OSCX_IN) -> /STM/OSCX_IN
- C6 pad 1: GNDD -> GND
- IC1 pad 5: unconnected-(IC1-ENABLE-Pad5) -> /GPS/ENABLE
- J1 pad 1: GNDD -> GND
- J1 pad 10: GNDD -> GND
- J1 pad 11: y+ -> y-
- J1 pad 12: a+ -> a-
- J1 pad 13: y- -> y+
- J1 pad 14: a- -> a+
- J1 pad 15: GNDD -> GND
- J1 pad 16: GNDD -> GND
- J1 pad 18: GNDD -> GND
- J1 pad 19: GNDD -> GND
- J1 pad 2: GNDD -> GND
- J1 pad 20: GNDD -> GND
- J1 pad 5: GNDD -> GND
- J1 pad 6: GNDD -> GND
- J1 pad 9: GNDD -> GND
- U12 pad 2: Net-(U12-PC14-OSCX_IN) -> /STM/OSCX_IN
- U12 pad 24: Net-(U12-PA13) -> /STM/SWDIO
- U12 pad 25: unconnected-(U12-PA13-BOOT0-Pad25) -> /STM/SWCLK
- U12 pad 29: /STM/CS-GPS -> /GPS/CS-GPS
- U12 pad 3: Net-(U12-PC15-OSCX_OUT) -> /STM/OSCX_OUT
- U12 pad 32: unconnected-(U12-PB8-Pad32) -> /GPS/GPIO
- U4 pad 1: GNDD -> GND
- U4 pad 3: GNDD -> GND
- U4 pad 4: GNDD -> GND
- U4 pad 6: GNDD -> GND
- U5 pad 19: /GPS/SCK-MAIN -> /SCK-MAIN
- U5 pad 20: /GPS/MISO-GPS -> /BMI270/MISO-BMI
- U5 pad 21: /GPS/MOSI-GPS -> /BMI270/MOSI-BMI
- U5 pad 3: /GPS/PPS -> PPS
- U7 pad 2: GNDD -> GND
- U7 pad 3: GNDD -> GND
- U7 pad 5: GNDD -> GND
- Y1 pad 1: Net-(U12-PC14-OSCX_IN) -> /STM/OSCX_IN
- Y1 pad 2: Net-(U12-PC15-OSCX_OUT) -> /STM/OSCX_IN
Routing:
- net PPS: track 0.00 -> 176.0 mm, vias 0 -> 1
- net /GPS/GPIO: track 0.00 -> 38.0 mm, vias 0 -> 2
- net /GPS/CS-GPS: track 0.00 -> 30.2 mm, vias 0 -> 2
- net y+: track 5.13 -> 30.9 mm
- net 3.3v: track 78.8 -> 104.1 mm, vias 0 -> 11
- net a+: track 5.13 -> 30.2 mm
- net y-: track 5.67 -> 29.6 mm
- net /BMI270/MOSI-BMI: track 81.2 -> 104.7 mm
- net a-: track 5.67 -> 28.8 mm
- net /BMI270/MISO-BMI: track 79.1 -> 99.2 mm, vias 8 -> 9
- net /SCK-MAIN: track 82.3 -> 102.1 mm, vias 6 -> 7
- net /STM/SWCLK: track 0.00 -> 14.5 mm, vias 0 -> 2
- net /GPS/ENABLE: track 0.00 -> 14.0 mm
- net /STM/SWDIO: track 0.00 -> 13.2 mm, vias 0 -> 2
- net Net-(U2-RA5): track 0.00 -> 7.35 mm
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- added copper zone on F.Cu, net 3.3v
- added copper zone on In2.Cu, net 3.3v
- added copper zone on B.Cu, net GND
- added copper zone on F.Cu, net GND
- added copper zone on In1.Cu, net GND
Other:
- board outline added: 127 x 127 mm

Commit message: netclasses SUCK
Parts:
- moved R8 1.12 mm to (160.9, 108.5)
- moved R9 1.12 mm to (165.9, 108.5)
- moved U1 1.12 mm to (163.4, 115.5)
Connections:
- net a+ renamed rx+
- net a- renamed rx-
- net y+ renamed tx+
- net y- renamed tx-
- U1 pad 2: /Transceiver/RX -> /STM/RX
- U1 pad 3: /Transceiver/TX -> /STM/TX
Routing:
- net /STM/TX: track 0.00 -> 55.2 mm, vias 0 -> 2
- net /STM/RX: track 0.00 -> 51.4 mm, vias 0 -> 2
- net GND: track 0.00 -> 15.6 mm, vias 0 -> 5
- net /BMI270/MISO-BMI: track 99.2 -> 103.6 mm
- net rx-: track 28.8 -> 30.3 mm
- net rx+: track 30.2 -> 31.1 mm
- net PPS: vias 1 -> 2
