File: KiCad/EGSE2/EGSE2/PDControl.kicad_sch (KiCad schematic)
At the start: 25 parts, among them J5 Conn_01x03_Pin, U1 TPS25730DREFR, U2 TLV76033DBZR

Commit message: gooning
Parts:
- added C12, C13: 10uF, Capacitor_SMD:C_0805_2012Metric_Pad1.18x1.45mm_HandSolder, symbol Device:C
Connections:
- net GND: now also C12.2, C13.2
- net LDO_1V5: now also C12.1
- net LDO_3V3: now also C13.1
Other:
- moved on the sheet: J5
