File: KiCad/EGSE2/EGSE2/EGSE2.kicad_sch (KiCad schematic)
At the start: 4 parts

Commit message: gamig on this EGSE type hsi
Other:
- sheet USBHELL renamed USB_config
Changed lines of the file:
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@@
 			(color 0 0 0 0.0000)
 		)
-		(property "Sheetname" "USBHELL"
+		(property "Sheetname" "USB_config"
 			(at 104.14 60.2484 0)
 			(effects
