File: KiCad/C6_v1.0/CameraManagement.kicad_sch (KiCad schematic)
At the start: 19 parts, among them U4 SN74CB3T3384PWR, U5 SN74CB3T3384PWR, U6 ADV7280AWBCPZ, Y3 ABM8AIG-28.63636MHZ

Commit message: gooning
Parts:
- R17, R18: footprint YC164-JR-0733RL:RESCAXE80P320X160X70-8N -> YC124-JR-0733RL:RES_YC124_2X1_YAG-L
- U4, U5: footprint PW24 -> SN74CB3T3384PWR:PW24
Changed lines of the file:
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@@
 			)
 		)
-		(property "Footprint" "YC164-JR-0733RL:RESCAXE80P320X160X70-8N"
+		(property "Footprint" "YC124-JR-0733RL:RES_YC124_2X1_YAG-L"
 			(at 59.69 135.89 0)
 			(effects
@@
 			)
 		)
-		(property "Footprint" "PW24"
+		(property "Footprint" "SN74CB3T3384PWR:PW24"
 			(at 43.18 81.28 0)
 			(effects
@@
 			)
 		)
-		(property "Footprint" "PW24"
+		(property "Footprint" "SN74CB3T3384PWR:PW24"
 			(at 43.18 30.48 0)
 			(effects
@@
 			)
 		)
-		(property "Footprint" "YC164-JR-0733RL:RESCAXE80P320X160X70-8N"
+		(property "Footprint" "YC124-JR-0733RL:RES_YC124_2X1_YAG-L"
 			(at 59.69 176.53 0)
 			(effects

Commit message: im scared
Parts:
- R17, R18: footprint YC124-JR-0733RL:RES_YC124_2X1_YAG-L -> C6:RES_YC124_2X1_YAG-L
- U4, U5: footprint SN74CB3T3384PWR:PW24 -> C6:PW24-L
- U6: footprint ADV7280AWBCPZ NTSC:CP-32-12_ADI -> C6:CP-32-12_ADI-L
- Y3: footprint ABM8AIG_28_63636MHZ_12_2Z_T3 Crystal:XTAL_ABM8AIG-28.63636MHZ-12-2Z-T3 -> C6:XTAL_ABM8AIG-28.63636MHZ-12-2Z-T3
Changed lines of the file:
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@@
 			)
 		)
-		(property "Footprint" "ADV7280AWBCPZ NTSC:CP-32-12_ADI"
+		(property "Footprint" "C6:CP-32-12_ADI-L"
 			(at 195.58 30.48 0)
 			(effects
@@
 			)
 		)
-		(property "Footprint" "YC124-JR-0733RL:RES_YC124_2X1_YAG-L"
+		(property "Footprint" "C6:RES_YC124_2X1_YAG-L"
 			(at 59.69 135.89 0)
 			(effects
@@
 			)
 		)
-		(property "Footprint" "SN74CB3T3384PWR:PW24"
+		(property "Footprint" "C6:PW24-L"
 			(at 43.18 81.28 0)
 			(effects
@@
 			)
 		)
-		(property "Footprint" "SN74CB3T3384PWR:PW24"
+		(property "Footprint" "C6:PW24-L"
 			(at 43.18 30.48 0)
 			(effects
@@
 			)
 		)
-		(property "Footprint" "YC124-JR-0733RL:RES_YC124_2X1_YAG-L"
+		(property "Footprint" "C6:RES_YC124_2X1_YAG-L"
 			(at 59.69 176.53 0)
 			(effects
@@
 			)
 		)
-		(property "Footprint" "ABM8AIG_28_63636MHZ_12_2Z_T3 Crystal:XTAL_ABM8AIG-28.63636MHZ-12-2Z-T3"
+		(property "Footprint" "C6:XTAL_ABM8AIG-28.63636MHZ-12-2Z-T3"
 			(at 182.88 96.52 0)
 			(effects

Commit message: DCMI1-Me0
Parts:
- C10, C11, C12, C13, C15, C16, C17: footprint Capacitor_SMD:C_0805_2012Metric -> Capacitor_SMD:C_0402_1005Metric_Pad0.74x0.62mm_HandSolder
- C14: footprint Capacitor_SMD:C_0201_0603Metric_Pad0.64x0.40mm_HandSolder -> Capacitor_SMD:C_0402_1005Metric_Pad0.74x0.62mm_HandSolder
- R20, R21, R22: footprint Resistor_SMD:R_0805_2012Metric -> Resistor_SMD:R_0402_1005Metric_Pad0.72x0.64mm_HandSolder
Connections:
- net 1V8: no longer U6.21 (AVDD)
- net 1V8*: now also U6.21 (AVDD)
- net CAM_D0: now also U4.20 (2B4); no longer U4.2 (1B1)
- net CAM_D1: now also U4.23 (2B5); no longer U4.5 (1B2)
- net CAM_D2: now also U4.2 (1B1); no longer U4.6 (1B3)
- net CAM_D3: now also U4.5 (1B2); no longer U4.9 (1B4)
- net CAM_D4: now also U4.6 (1B3); no longer U4.10 (1B5)
- net CAM_D5: now also U4.9 (1B4); no longer U4.15 (2B1)
- net CAM_D7: now also U4.15 (2B1); no longer U4.19 (2B3)
- net CAM_PCLK: now also U4.19 (2B3); no longer U4.20 (2B4)
- net GND: now also U4.11 (1A5); no longer U4.22 (2A5)
- net OV_D0: now also U4.21 (2A4); no longer U4.3 (1A1)
- net OV_D1: now also U4.22 (2A5); no longer U4.4 (1A2)
- net OV_D2: now also U4.3 (1A1); no longer U4.7 (1A3)
- net OV_D3: now also U4.4 (1A2); no longer U4.8 (1A4)
- net OV_D4: now also U4.7 (1A3); no longer U4.11 (1A5)
- net OV_D5: now also U4.8 (1A4); no longer U4.14 (2A1)
- net OV_D7: now also U4.14 (2A1); no longer U4.18 (2A3)
- net OV_PCLK: now also U4.18 (2A3); no longer U4.21 (2A4)
Changed lines of the file:
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@@
-	(wire
-		(pts
-			(xy 40.64 53.34) (xy 43.18 53.34)
-		)
-		(stroke
-			(width 0)
-			(type default)
-		)
-	)
 	(wire
 		(pts
@@
 	)
 	(label "1V8*"
+		(at 259.08 60.96 0)
+		(effects
+			(font
+				(size 1.27 1.27)
+			)
+			(justify left bottom)
+		)
+	)
+	(label "1V8*"
 		(at 173.99 25.4 0)
 		(effects
@@
 			)
 			(justify left bottom)
-		)
-	)
-	(label "CAM_D4"
-		(at 40.64 53.34 180)
-		(effects
-			(font
-				(size 1.27 1.27)
-			)
-			(justify right bottom)
 		)
 	)
@@
 		)
 	)
-	(label "CAM_D0"
+	(label "CAM_D2"
 		(at 40.64 33.02 180)
 		(effects
@@
 		)
 	)
-	(label "CAM_D1"
+	(label "CAM_D3"
 		(at 40.64 40.64 180)
 		(effects
@@
 		)
 	)
-	(label "CAM_D2"
+	(label "CAM_D4"
 		(at 40.64 43.18 180)
 		(effects
@@
 		)
 	)
-	(label "CAM_D3"
+	(label "CAM_D5"
 		(at 40.64 50.8 180)
 		(effects
@@
 		)
 	)
-	(label "CAM_D7"
+	(label "CAM_PCLK"
 		(at 106.68 43.18 0)
 		(effects
@@
 		)
 	)
-	(label "CAM_PCLK"
+	(label "CAM_D0"
 		(at 106.68 40.64 0)
 		(effects
@@
 		)
 	)
+	(label "CAM_D1"
+		(at 106.68 33.02 0)
+		(effects
+			(font
+				(size 1.27 1.27)
+			)
+			(justify left bottom)
+		)
+	)
 	(label "CAM_D6"
 		(at 106.68 99.06 0)
@@
 		)
 	)
-	(label "CAM_D5"
+	(label "CAM_D7"
 		(at 106.68 53.34 0)
 		(effects
@@
 		)
 	)
-	(hierarchical_label "GND"
+	(hierarchical_label "OV_D1"
 		(shape output)
 		(at 106.68 35.56 0)
@@
 		)
 	)
-	(hierarchical_label "OV_D5"
+	(hierarchical_label "OV_D7"
 		(shape input)
 		(at 106.68 55.88 0)
@@
 		)
 	)
-	(hierarchical_label "OV_D0"
+	(hierarchical_label "OV_D2"
 		(shape input)
 		(at 40.64 35.56 180)
@@
 		)
 	)
-	(hierarchical_label "1V8"
-		(shape input)
-		(at 259.08 60.96 0)
-		(effects
-			(font
-				(size 1.27 1.27)
-			)
-			(justify left)
-		)
-	)
-	(hierarchical_label "OV_D4"
+	(hierarchical_label "GND"
 		(shape input)
 		(at 40.64 55.88 180)
@@
 		)
 	)
-	(hierarchical_label "OV_PCLK"
+	(hierarchical_label "OV_D0"
 		(shape input)
 		(at 106.68 38.1 0)
@@
 		)
 	)
-	(hierarchical_label "OV_D2"
+	(hierarchical_label "OV_D4"
 		(shape input)
 		(at 40.64 45.72 180)
@@
 		)
 	)
-	(hierarchical_label "OV_D7"
+	(hierarchical_label "OV_PCLK"
 		(shape input)
 		(at 106.68 45.72 0)
@@
 		)
 	)
-	(hierarchical_label "OV_D3"
+	(hierarchical_label "OV_D5"
 		(shape input)
 		(at 40.64 48.26 180)
@@
 		)
 	)
-	(hierarchical_label "OV_D1"
+	(hierarchical_label "OV_D3"
 		(shape input)
 		(at 40.64 38.1 180)
@@
 			)
 		)
-		(property "Footprint" "Capacitor_SMD:C_0805_2012Metric"
+		(property "Footprint" "Capacitor_SMD:C_0402_1005Metric_Pad0.74x0.62mm_HandSolder"
 			(at 168.6052 35.56 0)
 			(effects
@@
 			)
 		)
-		(property "Footprint" "Capacitor_SMD:C_0805_2012Metric"
+		(property "Footprint" "Capacitor_SMD:C_0402_1005Metric_Pad0.74x0.62mm_HandSolder"
 			(at 196.5452 106.68 0)
 			(effects
@@
 			)
 		)
-		(property "Footprint" "Capacitor_SMD:C_0805_2012Metric"
+		(property "Footprint" "Capacitor_SMD:C_0402_1005Metric_Pad0.74x0.62mm_HandSolder"
 			(at 104.4448 20.32 0)
 			(effects
@@
 			)
 		)
-		(property "Footprint" "Resistor_SMD:R_0805_2012Metric"
+		(property "Footprint" "Resistor_SMD:R_0402_1005Metric_Pad0.72x0.64mm_HandSolder"
 			(at 277.368 46.99 90)
 			(effects
@@
 			)
 		)
-		(property "Footprint" "Capacitor_SMD:C_0201_0603Metric_Pad0.64x0.40mm_HandSolder"
+		(property "Footprint" "Capacitor_SMD:C_0402_1005Metric_Pad0.74x0.62mm_HandSolder"
 			(at 178.7652 35.56 0)
 			(effects
@@
 			)
 		)
-		(property "Footprint" "Capacitor_SMD:C_0805_2012Metric"
+		(property "Footprint" "Capacitor_SMD:C_0402_1005Metric_Pad0.74x0.62mm_HandSolder"
 			(at 171.1452 106.68 0)
 			(effects
@@
 			)
 		)
-		(property "Footprint" "Capacitor_SMD:C_0805_2012Metric"
+		(property "Footprint" "Capacitor_SMD:C_0402_1005Metric_Pad0.74x0.62mm_HandSolder"
 			(at 104.4448 71.12 0)
 			(effects
@@
 			)
 		)
-		(property "Footprint" "Resistor_SMD:R_0805_2012Metric"
+		(property "Footprint" "Resistor_SMD:R_0402_1005Metric_Pad0.72x0.64mm_HandSolder"
 			(at 237.998 102.87 90)
 			(effects
@@
 			)
 		)
-		(property "Footprint" "Capacitor_SMD:C_0805_2012Metric"
+		(property "Footprint" "Capacitor_SMD:C_0402_1005Metric_Pad0.74x0.62mm_HandSolder"
 			(at 246.38 95.5548 0)
 			(effects
@@
 			)
 		)
-		(property "Footprint" "Capacitor_SMD:C_0805_2012Metric"
+		(property "Footprint" "Capacitor_SMD:C_0402_1005Metric_Pad0.74x0.62mm_HandSolder"
 			(at 274.0152 68.58 0)
 			(effects
@@
 			)
 		)
-		(property "Footprint" "Resistor_SMD:R_0805_2012Metric"
+		(property "Footprint" "Resistor_SMD:R_0402_1005Metric_Pad0.72x0.64mm_HandSolder"
 			(at 201.93 98.298 90)
 			(effects

Commit message: finaly
Parts:
- removed C10, C11: 0.1u, Capacitor_SMD:C_0402_1005Metric_Pad0.74x0.62mm_HandSolder, symbol Device:C
- removed R19: R33, Resistor_SMD:R_0402_1005Metric_Pad0.72x0.64mm_HandSolder, symbol Device:R
- removed U4, U5: SN74CB3T3384PWR, C6:PW24-L, symbol SN74CB3T3384PWR:SN74CB3T3384PWR
- added R62: YC164-JR-0733RL, C6:RES_YC124_2X1_YAG-L, symbol YC164-JR-0733RL:YC164-JR-0733RL
- added U11: SN74CBTLV16292VR, C6:DGV56-L, symbol SN74CBTLV16292VR:SN74CBTLV16292VR
Connections:
- net 3V3: now also U11.17 (VCC)
- net CAM_D0: now also R62.6, U11.25 (11A); no longer R17.1, R17.8
- net CAM_D1: now also R62.7, U11.23 (10A); no longer R17.2, R17.7
- net CAM_D2: now also R62.5, U11.27 (12A); no longer R17.3, R17.6
- net CAM_D3: now also R62.8, U11.21 (9A); no longer R17.4, R17.5
- net CAM_D4: now also R18.7, U11.13 (6A); no longer R18.1, R18.8
- net CAM_D5: now also R18.8, U11.11 (5A); no longer R18.2, R18.7
- net CAM_D6: now also R17.6, U11.6 (3A); no longer R18.3, R18.6
- net CAM_D7: now also R17.7, U11.4 (2A); no longer R18.4, R18.5
- net CAM_PCLK: now also R18.5, U11.18 (8A)
- net GND: now also U11.19 (GND), U11.38 (GND), U11.49 (GND), U11.8 (GND)
- net OV_D0: now also U11.31 (11B2)
- net OV_D1: now also U11.33 (10B2)
- net OV_D2: now also U11.29 (12B2)
- net OV_D3: now also U11.35 (9B2)
- net OV_D4: now also U11.42 (6B2)
- net OV_D5: now also U11.44 (5B2)
- net OV_D6: now also U11.48 (3B2)
- net OV_D7: now also U11.51 (2B2)
- net OV_PCLK: now also U11.37 (8B2)
- net SPLIT_D0: now also U11.32 (11B1)
- net SPLIT_D1: now also U11.34 (10B1)
- net SPLIT_D2: now also U11.30 (12B1)
- net SPLIT_D3: now also U11.36 (9B1)
- net SPLIT_D4: now also U11.43 (6B1)
- net SPLIT_D5: now also U11.45 (5B1)
- net SPLIT_D6: now also U11.50 (3B1)
- net SPLIT_D7: now also U11.52 (2B1)
- net SPLIT_PCLK: now also U11.39 (8B1)
- net DCD_VSYNC: now reaches U6.29 (VS/FIELD/SFL)
- net DCD_VSYNC: now also U11.47 (4B1)
- net DCD_HSYNC: now reaches U6.30 (HS)
- net DCD_HSYNC: now also U11.41 (7B1)
- net DCD_PDWN renamed DCD_PWDN
- net DCD_PWDN: now also U11.54 (1B1)
- new net CAM_D0*: R62.3
- new net CAM_D1*: R62.2
- new net CAM_D2*: R62.4
- new net CAM_D3*: R62.1
- new net CAM_D4*: R18.2
- new net CAM_D5*: R18.1
- new net CAM_D6*: R17.3
- new net CAM_D7*: R17.2
- new net CAM_HSYNC: R18.6, U11.15 (7A)
- new net CAM_HSYNC*: R18.3
- new net CAM_PCLK*: R18.4
- new net CAM_PDWN: R17.8, U11.2 (1A)
- new net CAM_PDWN*: R17.1
- new net CAM_S: U11.1 (S)
- new net CAM_VSYNC: R17.5, U11.9 (4A)
- new net CAM_VSYNC*: R17.4
- new net OV_HSYNC: U11.40 (7B2)
- new net OV_PWDN: U11.53 (1B2)
- new net OV_VSYNC: U11.46 (4B2)
