File: KiCad/C6_v1.0/IO_Connections.kicad_sch (KiCad schematic)
At the start: 4 parts, among them J1 FH12-24S-0.5SH_55_, J2 Conn_01x06, J3 Conn_01x06, J5 Conn_01x05_Socket

Commit message: mar
Parts:
- renumbered J2 to J6, J1 to J7
Changed lines of the file:
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@@
 		(on_board yes)
 		(dnp no)
-		(property "Reference" "J1"
+		(property "Reference" "J7"
 			(at 31.75 31.496 0)
 			(effects
@@
 			(project "C6v1.0"
 				(path "/8737aa07-2805-4383-a805-a4fb57529a3e/bc81c9ac-f01c-4dc3-bedd-d5929ac8ec00"
-					(reference "J1")
+					(reference "J7")
 					(unit 1)
 				)
@@
 		(on_board yes)
 		(dnp no)
-		(property "Reference" "J2"
+		(property "Reference" "J6"
 			(at 27.432 144.018 90)
 			(effects
@@
 			(project "C6v1.0"
 				(path "/8737aa07-2805-4383-a805-a4fb57529a3e/bc81c9ac-f01c-4dc3-bedd-d5929ac8ec00"
-					(reference "J2")
+					(reference "J6")
 					(unit 1)
 				)

Commit message: gooning
Parts:
- J7: footprint FH12_24S_0_5SH_55 Camera Connector:HRS_FH12-24S-0.5SH_55_ -> FH12-24S-0.5S_55_:CONN_FH12-22S-0.5SH55_HIR
Changed lines of the file:
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@@
 			)
 		)
-		(property "Footprint" "FH12_24S_0_5SH_55 Camera Connector:HRS_FH12-24S-0.5SH_55_"
+		(property "Footprint" "FH12-24S-0.5S_55_:CONN_FH12-22S-0.5SH55_HIR"
 			(at 35.56 71.12 0)
 			(effects

Commit message: im scared
Parts:
- J7: footprint FH12-24S-0.5S_55_:CONN_FH12-22S-0.5SH55_HIR -> C6:CONN_FH12-22S-0.5SH55_HIR
Changed lines of the file:
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@@
 			)
 		)
-		(property "Footprint" "FH12-24S-0.5S_55_:CONN_FH12-22S-0.5SH55_HIR"
+		(property "Footprint" "C6:CONN_FH12-22S-0.5SH55_HIR"
 			(at 35.56 71.12 0)
 			(effects

Commit message: DCMI1-Me0
Parts:
- added J10: Conn_01x03, Connector_JST:JST_XA_S03B-XASK-1_1x03_P2.50mm_Horizontal, symbol Connector_Generic:Conn_01x03
- added J11: Conn_01x06, Connector_JST:JST_XA_S06B-XASK-1_1x06_P2.50mm_Horizontal, symbol Connector_Generic:Conn_01x06
- added J12: Conn_02x10_Odd_Even, Connector_PinHeader_2.54mm:PinHeader_2x10_P2.54mm_Vertical, symbol Connector_Generic:Conn_02x10_Odd_Even
- J3, J6: footprint Connector_JST:JST_XA_B06B-XASK-1_1x06_P2.50mm_Vertical -> Connector_JST:JST_XA_S06B-XASK-1_1x06_P2.50mm_Horizontal
Connections:
- net 5V: now also J12.7 (Pin_7), J12.8 (Pin_8)
- net GND: now also J10.1 (Pin_1), J11.1 (Pin_1), J12.1 (Pin_1), J12.10 (Pin_10), J12.15 (Pin_15), J12.16 (Pin_16), J12.18 (Pin_18), J12.19 (Pin_19), J12.2 (Pin_2), J12.20 (Pin_20), J12.5 (Pin_5), J12.6 (Pin_6), J12.9 (Pin_9)
- new net 3V3: J11.6 (Pin_6), J12.3 (Pin_3), J12.4 (Pin_4)
- new net ESC_TLM: J10.2 (Pin_2)
- new net HALL_A: J11.4 (Pin_4)
- new net HALL_B: J11.3 (Pin_3)
- new net HALL_C: J11.2 (Pin_2)
- new net PPS: J12.17 (Pin_17)
- new net PWM_IN: J10.3 (Pin_3)
- new net RX+: J12.11 (Pin_11)
- new net RX-: J12.13 (Pin_13)
- new net TX+: J12.14 (Pin_14)
- new net TX-: J12.12 (Pin_12)

Commit message: finaly
Parts:
- added R51, R52, R53, R54, R55, R56, R57, R58, R59, R60, R61: R33, Resistor_SMD:R_0402_1005Metric_Pad0.72x0.64mm_HandSolder, symbol Device:R
Connections:
- net DCMI_D0: now also R54.2; no longer J7.19 (Y2)
- net DCMI_D1: now also R52.2; no longer J7.21 (Y3)
- net DCMI_D2: now also R51.2; no longer J7.22 (Y4)
- net DCMI_D3: now also R53.2; no longer J7.20 (Y5)
- net DCMI_D4: now also R55.2; no longer J7.18 (Y6)
- net DCMI_D5: now also R57.2; no longer J7.16 (Y7)
- net DCMI_D6: now also R58.2; no longer J7.14 (Y8)
- net DCMI_D7: now also R59.2; no longer J7.12 (Y9)
- net DCMI_HSYNC: now also R60.2; no longer J7.9 (HSYNC)
- net DCMI_PCLK: now also R56.2; no longer J7.17 (PCLK)
- net DCMI_VSYNC: now also R61.2; no longer J7.7 (VSYNC)
- new net D0: J7.19 (Y2), R54.1
- new net D1: J7.21 (Y3), R52.1
- new net D2: J7.22 (Y4), R51.1
- new net D3: J7.20 (Y5), R53.1
- new net D4: J7.18 (Y6), R55.1
- new net D5: J7.16 (Y7), R57.1
- new net D6: J7.14 (Y8), R58.1
- new net D7: J7.12 (Y9), R59.1
- new net HSYNC: J7.9 (HSYNC), R60.1
- new net PCLK: J7.17 (PCLK), R56.1
- new net VSYNC: J7.7 (VSYNC), R61.1
Other:
- moved on the sheet: J10, J11, J5
