File: KiCad/C6_v1.0/LDOs.kicad_sch (KiCad schematic)
At the start: 15 parts

Commit message: pingus
Parts:
- gave numbers to parts that had none: 6
Changed lines of the file:
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@@
 		(dnp no)
 		(fields_autoplaced yes)
-		(property "Reference" "LED?"
+		(property "Reference" "LED2"
 			(at 154.94 91.4399 90)
 			(effects
@@
 			(project "C6v1.0"
 				(path "/8737aa07-2805-4383-a805-a4fb57529a3e/4d3c3eea-62ea-4a75-81f8-713bd295f2ea/4f1b91fb-2ee2-4864-a62f-28af09a89974"
-					(reference "LED?")
+					(reference "LED2")
 					(unit 1)
 				)
@@
 		(dnp no)
 		(fields_autoplaced yes)
-		(property "Reference" "LED?"
+		(property "Reference" "LED4"
 			(at 186.69 60.9599 90)
 			(effects
@@
 			(project "C6v1.0"
 				(path "/8737aa07-2805-4383-a805-a4fb57529a3e/4d3c3eea-62ea-4a75-81f8-713bd295f2ea/4f1b91fb-2ee2-4864-a62f-28af09a89974"
-					(reference "LED?")
+					(reference "LED4")
 					(unit 1)
 				)
@@
 		(on_board yes)
 		(dnp no)
-		(property "Reference" "2.8LDO?"
+		(property "Reference" "2.8LDO1"
 			(at 138.43 64.77 0)
 			(effects
@@
 			(project "C6v1.0"
 				(path "/8737aa07-2805-4383-a805-a4fb57529a3e/4d3c3eea-62ea-4a75-81f8-713bd295f2ea/4f1b91fb-2ee2-4864-a62f-28af09a89974"
-					(reference "2.8LDO?")
+					(reference "2.8LDO1")
 					(unit 1)
 				)
@@
 		(on_board yes)
 		(dnp no)
-		(property "Reference" "1.8LDO?"
+		(property "Reference" "1.8LDO1"
 			(at 139.7 102.87 0)
 			(effects
@@
 			(project "C6v1.0"
 				(path "/8737aa07-2805-4383-a805-a4fb57529a3e/4d3c3eea-62ea-4a75-81f8-713bd295f2ea/4f1b91fb-2ee2-4864-a62f-28af09a89974"
-					(reference "1.8LDO?")
+					(reference "1.8LDO1")
 					(unit 1)
 				)
@@
 		(dnp no)
 		(fields_autoplaced yes)
-		(property "Reference" "LED?"
+		(property "Reference" "LED3"
 			(at 160.02 133.3499 90)
 			(effects
@@
 			(project "C6v1.0"
 				(path "/8737aa07-2805-4383-a805-a4fb57529a3e/4d3c3eea-62ea-4a75-81f8-713bd295f2ea/4f1b91fb-2ee2-4864-a62f-28af09a89974"
-					(reference "LED?")
+					(reference "LED3")
 					(unit 1)
 				)
@@
 		(dnp no)
 		(fields_autoplaced yes)
-		(property "Reference" "U?"
+		(property "Reference" "U8"
 			(at 149.86 29.21 0)
 			(effects
@@
 			(project "C6v1.0"
 				(path "/8737aa07-2805-4383-a805-a4fb57529a3e/4d3c3eea-62ea-4a75-81f8-713bd295f2ea/4f1b91fb-2ee2-4864-a62f-28af09a89974"
-					(reference "U?")
-					(unit 1)
-				)
+					(reference "U8")
+					(unit 1)
+				)

Commit message: save
Parts:
- LED2, LED3, LED4: footprint LTST_C190KRKT red led:LED_LTST-C190_LTO -> LTST_C190KRKT:LED_LTST-C190_LTO
- U8: footprint TLV1117LV33DCYR 3.3 ldo:VREG_TLV1117LV33DCYR -> TLV1117LV33DCYR:VREG_TLV1117LV33DCYR
Changed lines of the file:
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@@
 			)
 		)
-		(property "Footprint" "LTST_C190KRKT red led:LED_LTST-C190_LTO"
+		(property "Footprint" "LTST_C190KRKT:LED_LTST-C190_LTO"
 			(at 148.59 86.36 0)
 			(effects
@@
 			)
 		)
-		(property "Footprint" "LTST_C190KRKT red led:LED_LTST-C190_LTO"
+		(property "Footprint" "LTST_C190KRKT:LED_LTST-C190_LTO"
 			(at 180.34 55.88 0)
 			(effects
@@
 			)
 		)
-		(property "Footprint" "LTST_C190KRKT red led:LED_LTST-C190_LTO"
+		(property "Footprint" "LTST_C190KRKT:LED_LTST-C190_LTO"
 			(at 153.67 128.27 0)
 			(effects
@@
 			)
 		)
-		(property "Footprint" "TLV1117LV33DCYR 3.3 ldo:VREG_TLV1117LV33DCYR"
+		(property "Footprint" "TLV1117LV33DCYR:VREG_TLV1117LV33DCYR"
 			(at 149.86 41.91 0)
 			(effects

Commit message: im scared
Connections:
- net GNDD renamed GND

Commit message: finaly
Connections:
- net +2.8V renamed 2V8
- net +3.3V renamed 3V3
- net +5V renamed 5V
- net 1.8V renamed 1V8
Changed lines of the file:
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@@
 		)
 	)
-	(global_label "+3.3V"
+	(hierarchical_label "2V8"
 		(shape input)
-		(at 106.68 72.39 180)
-		(fields_autoplaced yes)
+		(at 107.95 110.49 180)
 		(effects
 			(font
@@
 			(justify right)
 		)
-		(property "Intersheetrefs" "${INTERSHEET_REFS}"
-			(at 98.01 72.39 0)
-			(effects
-				(font
-					(size 1.27 1.27)
-				)
-				(justify right)
-				(hide yes)
-			)
-		)
 	)
-	(global_label "+2.8V"
+	(hierarchical_label "3V3"
 		(shape input)
-		(at 187.96 72.39 0)
-		(fields_autoplaced yes)
+		(at 203.2 36.83 0)
 		(effects
 			(font
@@
 			(justify left)
 		)
-		(property "Intersheetrefs" "${INTERSHEET_REFS}"
-			(at 196.63 72.39 0)
-			(effects
-				(font
-					(size 1.27 1.27)
-				)
-				(justify left)
-				(hide yes)
+	)
+	(hierarchical_label "1V8"
+		(shape input)
+		(at 166.37 110.49 0)
+		(effects
+			(font
+				(size 1.27 1.27)
 			)
+			(justify left)
 		)
 	)
-	(global_label "+2.8V"
+	(hierarchical_label "3V3"
 		(shape input)
-		(at 107.95 110.49 180)
-		(fields_autoplaced yes)
+		(at 106.68 72.39 180)
 		(effects
 			(font
@@
 			(justify right)
 		)
-		(property "Intersheetrefs" "${INTERSHEET_REFS}"
-			(at 99.28 110.49 0)
-			(effects
-				(font
-					(size 1.27 1.27)
-				)
-				(justify right)
-				(hide yes)
-			)
-		)
 	)
-	(global_label "1.8V"
+	(hierarchical_label "2V8"
 		(shape input)
-		(at 166.37 110.49 0)
-		(fields_autoplaced yes)
+		(at 187.96 72.39 0)
 		(effects
 			(font
@@
 			(justify left)
 		)
-		(property "Intersheetrefs" "${INTERSHEET_REFS}"
-			(at 173.4676 110.49 0)
-			(effects
-				(font
-					(size 1.27 1.27)
-				)
-				(justify left)
-				(hide yes)
-			)
-		)
 	)
-	(global_label "+3.3V"
-		(shape input)
-		(at 203.2 36.83 0)
-		(fields_autoplaced yes)
-		(effects
-			(font
-				(size 1.27 1.27)
-			)
-			(justify left)
-		)
-		(property "Intersheetrefs" "${INTERSHEET_REFS}"
-			(at 211.87 36.83 0)
-			(effects
-				(font
-					(size 1.27 1.27)
-				)
-				(justify left)
-				(hide yes)
-			)
-		)
-	)
-	(global_label "+5V"
+	(hierarchical_label "5V"
 		(shape input)
 		(at 107.95 36.83 180)
-		(fields_autoplaced yes)
 		(effects
 			(font
@@
 			(justify right)
 		)
-		(property "Intersheetrefs" "${INTERSHEET_REFS}"
-			(at 101.0943 36.83 0)
-			(effects
-				(font
-					(size 1.27 1.27)
-				)
-				(justify right)
-				(hide yes)
-			)
-		)
 	)
