File: KiCad/C6_v1.0/LevelShifting.kicad_sch (KiCad schematic)
At the start: 6 parts, among them U3 PCA9306

Commit message: gooning
Parts:
- U3: footprint (none) -> Package_SON:X2SON-8_1.4x1mm_P0.35mm
Changed lines of the file:
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@@
 			)
 		)
-		(property "Footprint" ""
+		(property "Footprint" "Package_SON:X2SON-8_1.4x1mm_P0.35mm"
 			(at 46.99 39.37 0)
 			(effects

Commit message: DCMI1-Me0
Parts:
- R3, R4, R5, R6, R7: footprint Resistor_SMD:R_0805_2012Metric -> Resistor_SMD:R_0402_1005Metric_Pad0.72x0.64mm_HandSolder
Changed lines of the file:
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@@
 			)
 		)
-		(property "Footprint" "Resistor_SMD:R_0805_2012Metric"
+		(property "Footprint" "Resistor_SMD:R_0402_1005Metric_Pad0.72x0.64mm_HandSolder"
 			(at 89.662 38.1 90)
 			(effects
@@
 			)
 		)
-		(property "Footprint" "Resistor_SMD:R_0805_2012Metric"
+		(property "Footprint" "Resistor_SMD:R_0402_1005Metric_Pad0.72x0.64mm_HandSolder"
 			(at 37.338 38.1 90)
 			(effects
@@
 			)
 		)
-		(property "Footprint" "Resistor_SMD:R_0805_2012Metric"
+		(property "Footprint" "Resistor_SMD:R_0402_1005Metric_Pad0.72x0.64mm_HandSolder"
 			(at 68.072 38.1 90)
 			(effects
@@
 			)
 		)
-		(property "Footprint" "Resistor_SMD:R_0805_2012Metric"
+		(property "Footprint" "Resistor_SMD:R_0402_1005Metric_Pad0.72x0.64mm_HandSolder"
 			(at 47.498 38.1 90)
 			(effects
@@
 			)
 		)
-		(property "Footprint" "Resistor_SMD:R_0805_2012Metric"
+		(property "Footprint" "Resistor_SMD:R_0402_1005Metric_Pad0.72x0.64mm_HandSolder"
 			(at 76.962 38.1 90)
 			(effects

Commit message: finaly
Parts:
- U3: footprint Package_SON:X2SON-8_1.4x1mm_P0.35mm -> Package_SO:SSOP-8_2.95x2.8mm_P0.65mm
Changed lines of the file:
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@@
 			)
 		)
-		(property "Footprint" "Package_SON:X2SON-8_1.4x1mm_P0.35mm"
+		(property "Footprint" "Package_SO:SSOP-8_2.95x2.8mm_P0.65mm"
 			(at 46.99 39.37 0)
 			(effects
