File: KiCad/ENIAC/Power.kicad_sch (KiCad schematic)
At the start: 16 parts, among them U10 LM317BD2TR4G, U11 S-13A1A00-U5T1U3, U9 TPS7A2033PDQNRM3

Commit message: john d tickle
Changed lines of the file:
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@@
 	(generator_version "9.0")
 	(paper "A4")
-	(text_box "current draws:\ntx 12.5dBm 24mA\nrx high sens 8.2mA\nLNA 12mA\nPA +28dBm 660mA max"
+	(text_box "current draws:\nidfk\nLO/mixer stuff: 17mA\nSX1281: 80mA\n"
 		(exclude_from_sim no)
 		(at 40.64 151.13 0)

Commit message: funny commit message
Parts:
- removed C32, C33, C37: 1uF, symbol Device:C_Small
- removed C34, C35, C38, C39: 2.2uF, symbol Device:C_Small
- removed C36: 0.1uF, symbol Device:C_Small
- removed R10: 1k, symbol Device:R_Small_US
- removed R11, R12: 10k, symbol Device:R_Small
- removed R13: 39.2k, symbol Device:R_Small
- removed R9: 33.2k, symbol Device:R_Small
- removed U10: LM317BD2TR4G, D2PAK3_ONS, symbol 2025-11-11_05-35-23:LM317BD2TR4G
- removed U11: S-13A1A00-U5T1U3, SOT-89_5MC_MCH, symbol 2025-11-11_05-05-23:MCP1804T-3302I_MT
- removed U9: TPS7A2033PDQNRM3, DQN0004A-MFG, symbol 2025-10-22_05-18-30:TPS7A2033PDQNRM3
- added C32, C35: .33uF, symbol Device:C
- added C33, C34: .22uF, symbol Device:C
- added C36, C37, C38, C39: 1uF, symbol Device:C
- added U10, U11: NCV8163ASN330T1G, Package_TO_SOT_SMD:TSOT-23-5, symbol Regulator_Linear:NCV8114ASN120T1G
- added U7, U9: TL780-05CKTTR, KTT3_6P22X6P6_TEX, symbol 2026-03-09_03-52-00:TL780-05CKTTR
Connections:
- net GND: now also C32.2, C33.1, C34.1, C35.2, C36.1, C37.1, C38.1, C39.1, U10.2 (GND), U11.2 (GND), U7.2 (COMMON), U7.4 (EPAD), U9.2 (COMMON), U9.4 (EPAD)
- net VBATT: now also C32.1, C35.1, U7.3 (INPUT), U9.3 (INPUT)
- new net +3.3VA: C37.2, U10.5 (OUT)
- new net +3.3VD: C39.2, U11.5 (OUT)
- new net +5VA: C33.2, U7.1 (OUTPUT)
- new net +5V_poor: C34.2, C36.2, C38.2, U10.1 (IN), U10.3 (EN), U11.1 (IN), U11.3 (EN), U9.1 (OUTPUT)

Commit message: netclasses SUCK
Parts:
- C42: renamed from C33; footprint (none) -> Capacitor_SMD:C_0603_1608Metric
- C43: renamed from C34; footprint (none) -> Capacitor_SMD:C_0603_1608Metric
- C44: renamed from C36; footprint (none) -> Capacitor_SMD:C_0603_1608Metric
- C45: renamed from C38; footprint (none) -> Capacitor_SMD:C_0603_1608Metric
- C46: renamed from C37; footprint (none) -> Capacitor_SMD:C_0603_1608Metric
- C47: renamed from C39; footprint (none) -> Capacitor_SMD:C_0603_1608Metric
- C48: renamed from C32; footprint (none) -> Capacitor_SMD:C_0603_1608Metric
- C49: renamed from C35; footprint (none) -> Capacitor_SMD:C_0603_1608Metric
- U5: renamed from U7; footprint KTT3_6P22X6P6_TEX -> Package_TO_SOT_SMD:TO-263-3_TabPin4
- U6: renamed from U9; footprint KTT3_6P22X6P6_TEX -> Package_TO_SOT_SMD:TO-263-3_TabPin4
- renumbered U10 to U7, U11 to U8
