File: KiCad/ENIAC/SX1281.kicad_sch (KiCad schematic)
At the start: 13 parts, among them U2 SX1281IMLTRT

Commit message: john d tickle
Other:
- added sheet Crystal (Crystal.kicad_sch)
Changed lines of the file:
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@@
+		)
+	)
+	(sheet
+		(at 88.9 123.19)
+		(size 15.24 27.94)
+		(exclude_from_sim no)
+		(in_bom yes)
+		(on_board yes)
+		(dnp no)
+		(fields_autoplaced yes)
+		(stroke
+			(width 0.1524)
+			(type solid)
+		)
+		(fill
+			(color 0 0 0 0.0000)
+		)
+		(property "Sheetname" "Crystal"
+			(at 88.9 122.4784 0)
+			(effects
+				(font
+					(size 1.27 1.27)
+				)
+				(justify left bottom)
+			)
+		)
+		(property "Sheetfile" "Crystal.kicad_sch"
+			(at 88.9 151.7146 0)
+			(effects
+				(font
+					(size 1.27 1.27)
+				)
+				(justify left top)
+			)
+		)
+		(instances
+			(project "ENIAC"
+				(path "/028e33f3-2d21-4744-a260-423608f4c0b7/d2a65d20-6114-460a-836d-d801263d62de"
+					(page "3")
+				)
+			)
 		)
 	)

Commit message: funny commit message
Parts:
- added Y2: ABM11-142-27.120MHZ-T3, ABM11-142-27.120MHZ-T3:XTAL_ABM11-142-27.120MHZ-T3, symbol ABM11-142-27.120MHZ-T3:ABM11-142-27.120MHZ-T3
Connections:
- net GND: now also Y2.2 (GND), Y2.4 (GND)
- net at U2.4 (XTA): now also Y2.1
- net at U2.6 (XTB): now also Y2.3
Other:
- removed sheet Crystal

Commit message: netclasses SUCK
Parts:
- removed R2, R3: 1k, symbol Device:R_Small_US
- added R13: 22, Resistor_SMD:R_0603_1608Metric, symbol Device:R_Small_US
- added TP1: TestPoint, symbol Connector:TestPoint
- C50: renamed from C1; footprint (none) -> Capacitor_SMD:C_0603_1608Metric
- C51: renamed from C2; footprint (none) -> Capacitor_SMD:C_0603_1608Metric
- C52: renamed from C3; footprint (none) -> Capacitor_SMD:C_0603_1608Metric
- C53: renamed from C4; footprint (none) -> Capacitor_SMD:C_0603_1608Metric
- C54: renamed from C5; footprint (none) -> Capacitor_SMD:C_0603_1608Metric
- C55: renamed from C6; footprint (none) -> Capacitor_SMD:C_0603_1608Metric
- C56: renamed from C7; footprint (none) -> Capacitor_SMD:C_0603_1608Metric
- C57: renamed from C8; value 18pF -> 47pF; footprint (none) -> Capacitor_SMD:C_0603_1608Metric
- C58: renamed from C9; footprint (none) -> Capacitor_SMD:C_0603_1608Metric
- L5: renamed from L1; footprint (none) -> Inductor_SMD:L_0603_1608Metric
- U9: renamed from U2; footprint SX1281IMLTRT:XCVR_SX1281IMLTRT -> Package_DFN_QFN:QFN-24-1EP_4x4mm_P0.5mm_EP2.6x2.6mm_ThermalVias
- Y2: footprint ABM11-142-27.120MHZ-T3:XTAL_ABM11-142-27.120MHZ-T3 -> ABM11_142_27_120MHZ_T3 (1):XTAL_ABM11-142-27.120MHZ-T3
Connections:
- net SX_MISO: now also R13.2; no longer U9.16 (MISO_TX)
- net SX_RST: now also U9.3 (~{RESET}), TP1.1
- net rfio: now reaches C53.2, C57.1, U9.22 (RFIO)
- net +3.3V_RF renamed +3.3VA
- new net MISO_TX: R13.1, U9.16 (MISO_TX)
