File: KiCad/ENIAC/ENIAC.kicad_sch (KiCad schematic)
At the start: 1 part, among them J1 B6B-XH-A

Commit message: john d tickle
Other:
- removed sheet 2_4GHz_Frontend
- removed sheet Crystal
- sheet 1_2GHz_Frontend ports: added GP1, RFIO; removed none
Changed lines of the file:
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@@
-	(wire
-		(pts
-			(xy 209.55 74.93) (xy 209.55 71.12)
-		)
-		(stroke
-			(width 0)
-			(type default)
-		)
-	)
 	(wire
 		(pts
@@
 	(wire
 		(pts
-			(xy 227.33 71.12) (xy 227.33 74.93)
-		)
-		(stroke
-			(width 0)
-			(type default)
-		)
-	)
-	(wire
-		(pts
 			(xy 111.76 88.9) (xy 111.76 36.83)
 		)
@@
 	(wire
 		(pts
-			(xy 209.55 71.12) (xy 227.33 71.12)
-		)
-		(stroke
-			(width 0)
-			(type default)
-		)
-	)
-	(wire
-		(pts
 			(xy 196.85 74.93) (xy 196.85 66.04)
 		)
@@
 	(wire
 		(pts
+			(xy 77.47 138.43) (xy 77.47 146.05)
+		)
+		(stroke
+			(width 0)
+			(type default)
+		)
+	)
+	(wire
+		(pts
+			(xy 72.39 138.43) (xy 72.39 146.05)
+		)
+		(stroke
+			(width 0)
+			(type default)
+		)
+	)
+	(wire
+		(pts
 			(xy 114.3 86.36) (xy 114.3 36.83)
 		)
@@
 			(width 0)
 			(type default)
+		)
+	)
+	(label "RFIO_RF"
+		(at 72.39 138.43 90)
+		(effects
+			(font
+				(size 1.27 1.27)
+			)
+			(justify left bottom)
+		)
+	)
+	(label "GP1"
+		(at 196.85 66.04 90)
+		(effects
+			(font
+				(size 1.27 1.27)
+			)
+			(justify left bottom)
+		)
+	)
+	(label "GP1"
+		(at 77.47 138.43 90)
+		(effects
+			(font
+				(size 1.27 1.27)
+			)
+			(justify left bottom)
+		)
+	)
+	(label "GP1"
+		(at 196.85 66.04 90)
+		(effects
+			(font
+				(size 1.27 1.27)
+			)
+			(justify left bottom)
+		)
+	)
+	(label "RFIO_RF"
+		(at 191.77 66.04 90)
+		(effects
+			(font
+				(size 1.27 1.27)
+			)
+			(justify left bottom)
 		)
 	)
@@
 		)
 	)
-	(hierarchical_label "CLK_REF"
-		(shape output)
-		(at 209.55 74.93 270)
-		(effects
-			(font
-				(size 1.27 1.27)
-			)
-			(justify right)
-		)
-	)
 	(hierarchical_label "SX_MISO"
 		(shape input)
@@
 		)
 	)
-	(hierarchical_label "CLK_REF"
-		(shape output)
-		(at 227.33 74.93 270)
-		(effects
-			(font
-				(size 1.27 1.27)
-			)
-			(justify right)
-		)
-	)
 	(hierarchical_label "RFIO_RF"
 		(shape bidirectional)
@@
 		(shape input)
 		(at 187.96 92.71 0)
-		(effects
-			(font
-				(size 1.27 1.27)
-			)
-			(justify left)
-		)
-	)
-	(hierarchical_label "GP1"
-		(shape input)
-		(at 196.85 66.04 90)
-		(effects
-			(font
-				(size 1.27 1.27)
-			)
-			(justify left)
-		)
-	)
-	(hierarchical_label "RFIO_RF"
-		(shape bidirectional)
-		(at 191.77 66.04 90)
 		(effects
 			(font
@@
 	)
 	(sheet
-		(at 179.07 22.86)
-		(size 100.33 43.18)
-		(exclude_from_sim no)
-		(in_bom yes)
-		(on_board yes)
-		(dnp no)
-		(stroke
-			(width 0.1524)
-			(type solid)
-		)
-		(fill
-			(color 0 0 0 0.0000)
-		)
-		(property "Sheetname" "2_4GHz_Frontend"
-			(at 179.07 18.796 0)
-			(effects
-				(font
-					(size 1.27 1.27)
-				)
-				(justify left bottom)
-			)
-		)
-		(property "Sheetfile" "2_4GHz_Frontend.kicad_sch"
-			(at 178.816 20.828 0)
-			(effects
-				(font
-					(size 1.27 1.27)
-				)
-				(justify left top)
-			)
-		)
-		(instances
-			(project "ENIAC"
-				(path "/028e33f3-2d21-4744-a260-423608f4c0b7"
-					(page "3")
-				)
-			)
-		)
-	)
-	(sheet
 		(at 26.035 22.86)
 		(size 33.655 67.31)
@@
 				(path "/028e33f3-2d21-4744-a260-423608f4c0b7"
 					(page "5")
-				)
-			)
-		)
-	)
-	(sheet
-		(at 222.25 74.93)
-		(size 15.24 27.94)
-		(exclude_from_sim no)
-		(in_bom yes)
-		(on_board yes)
-		(dnp no)
-		(fields_autoplaced yes)
-		(stroke
-			(width 0.1524)
-			(type solid)
-		)
-		(fill
-			(color 0 0 0 0.0000)
-		)
-		(property "Sheetname" "Crystal"
-			(at 222.25 74.2184 0)
-			(effects
-				(font
-					(size 1.27 1.27)
-				)
-				(justify left bottom)
-			)
-		)
-		(property "Sheetfile" "Crystal.kicad_sch"
-			(at 222.25 103.4546 0)
-			(effects
-				(font
-					(size 1.27 1.27)
-				)
-				(justify left top)
-			)
-		)
-		(instances
-			(project "ENIAC"
-				(path "/028e33f3-2d21-4744-a260-423608f4c0b7"
-					(page "4")
 				)
 			)
@@
 			)
 		)
+		(pin "RFIO" input
+			(at 72.39 146.05 90)
+			(effects
+				(font
+					(size 1.27 1.27)
+				)
+				(justify right)
+			)
+		)
+		(pin "GP1" input
+			(at 77.47 146.05 90)
+			(effects
+				(font
+					(size 1.27 1.27)
+				)
+				(justify right)
+			)
+		)

Commit message: funny commit message
Changed lines of the file:
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@@
 	(generator_version "9.0")
 	(paper "A4")
+	(junction
+		(at 109.22 99.06)
+		(diameter 0)
+		(color 0 0 0 0)
+	)
+	(junction
+		(at 111.76 96.52)
+		(diameter 0)
+		(color 0 0 0 0)
+	)
 	(wire
 		(pts
@@
 	(wire
 		(pts
+			(xy 109.22 99.06) (xy 109.22 146.05)
+		)
+		(stroke
+			(width 0)
+			(type default)
+		)
+	)
+	(wire
+		(pts
 			(xy 104.14 36.83) (xy 104.14 44.45)
 		)
@@
 	(wire
 		(pts
-			(xy 111.76 88.9) (xy 111.76 36.83)
+			(xy 111.76 96.52) (xy 111.76 36.83)
+		)
+		(stroke
+			(width 0)
+			(type default)
+		)
+	)
+	(wire
+		(pts
+			(xy 111.76 96.52) (xy 111.76 146.05)
 		)
 		(stroke
@@
 	(wire
 		(pts
-			(xy 187.96 95.25) (xy 106.68 95.25)
-		)
-		(stroke
-			(width 0)
-			(type default)
-		)
-	)
-	(wire
-		(pts
-			(xy 109.22 36.83) (xy 109.22 92.71)
+			(xy 187.96 88.9) (xy 106.68 88.9)
+		)
+		(stroke
+			(width 0)
+			(type default)
+		)
+	)
+	(wire
+		(pts
+			(xy 111.76 96.52) (xy 187.96 96.52)
+		)
+		(stroke
+			(width 0)
+			(type default)
+		)
+	)
+	(wire
+		(pts
+			(xy 109.22 36.83) (xy 109.22 99.06)
+		)
+		(stroke
+			(width 0)
+			(type default)
+		)
+	)
+	(wire
+		(pts
+			(xy 109.22 99.06) (xy 187.96 99.06)
 		)
 		(stroke
@@
 	(wire
 		(pts
-			(xy 187.96 92.71) (xy 109.22 92.71)
-		)
-		(stroke
-			(width 0)
-			(type default)
-		)
-	)
-	(wire
-		(pts
-			(xy 106.68 36.83) (xy 106.68 95.25)
+			(xy 106.68 36.83) (xy 106.68 88.9)
 		)
 		(stroke
@@
 		(pts
 			(xy 114.3 86.36) (xy 114.3 36.83)
-		)
-		(stroke
-			(width 0)
-			(type default)
-		)
-	)
-	(wire
-		(pts
-			(xy 187.96 88.9) (xy 111.76 88.9)
 		)
 		(stroke
@@
 	(hierarchical_label "SX_MOSI"
 		(shape output)
+		(at 111.76 146.05 270)
+		(effects
+			(font
+				(size 1.27 1.27)
+			)
+			(justify right)
+		)
+	)
+	(hierarchical_label "SX_MOSI"
+		(shape output)
+		(at 187.96 96.52 0)
+		(effects
+			(font
+				(size 1.27 1.27)
+			)
+			(justify left)
+		)
+	)
+	(hierarchical_label "SX_SCK"
+		(shape input)
+		(at 109.22 146.05 270)
+		(effects
+			(font
+				(size 1.27 1.27)
+			)
+			(justify right)
+		)
+	)
+	(hierarchical_label "SX_MISO"
+		(shape input)
+		(at 187.96 86.36 0)
+		(effects
+			(font
+				(size 1.27 1.27)
+			)
+			(justify left)
+		)
+	)
+	(hierarchical_label "GP1"
+		(shape input)
+		(at 196.85 74.93 270)
+		(effects
+			(font
+				(size 1.27 1.27)
+			)
+			(justify right)
+		)
+	)
+	(hierarchical_label "SX_CS"
+		(shape input)
 		(at 187.96 88.9 0)
-		(effects
-			(font
-				(size 1.27 1.27)
-			)
-			(justify left)
-		)
-	)
-	(hierarchical_label "SX_MISO"
-		(shape input)
-		(at 187.96 86.36 0)
-		(effects
-			(font
-				(size 1.27 1.27)
-			)
-			(justify left)
-		)
-	)
-	(hierarchical_label "GP1"
-		(shape input)
-		(at 196.85 74.93 270)
-		(effects
-			(font
-				(size 1.27 1.27)
-			)
-			(justify right)
-		)
-	)
-	(hierarchical_label "SX_CS"
-		(shape input)
-		(at 187.96 95.25 0)
 		(effects
 			(font
@@
 	(hierarchical_label "SX_SCK"
 		(shape input)
-		(at 187.96 92.71 0)
-		(effects
-			(font
+		(at 187.96 99.06 0)
+		(effects
+			(font

Commit message: netclasses SUCK
Parts:
- J1: footprint B6B-XH-A:JST_B6B-XH-A -> Connector_JST:JST_EH_S6B-EH_1x06_P2.50mm_Horizontal
Connections:
- net SX_CS renamed SX1281/SX_CS
- net SX_MISO renamed SX1281/SX_MISO
Other:
- sheet SX1281 ports: added GP1, RFIO, SX_CS, SX_MISO, SX_MOSI, SX_SCK; removed none
Changed lines of the file:
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@@
-		)
-	)
-	(hierarchical_label "SX_MOSI"
-		(shape output)
-		(at 187.96 96.52 0)
-		(effects
-			(font
-				(size 1.27 1.27)
-			)
-			(justify left)
 		)
 	)
@@
 		)
 	)
-	(hierarchical_label "SX_MISO"
-		(shape input)
-		(at 187.96 86.36 0)
-		(effects
-			(font
-				(size 1.27 1.27)
-			)
-			(justify left)
-		)
-	)
-	(hierarchical_label "GP1"
-		(shape input)
-		(at 196.85 74.93 270)
-		(effects
-			(font
-				(size 1.27 1.27)
-			)
-			(justify right)
-		)
-	)
-	(hierarchical_label "SX_CS"
-		(shape input)
-		(at 187.96 88.9 0)
-		(effects
-			(font
-				(size 1.27 1.27)
-			)
-			(justify left)
-		)
-	)
-	(hierarchical_label "RFIO_RF"
-		(shape bidirectional)
-		(at 191.77 74.93 270)
-		(effects
-			(font
-				(size 1.27 1.27)
-			)
-			(justify right)
-		)
-	)
-	(hierarchical_label "SX_SCK"
-		(shape input)
-		(at 187.96 99.06 0)
-		(effects
-			(font
-				(size 1.27 1.27)
-			)
-			(justify left)
-		)
-	)
 	(symbol
 		(lib_id "power:+5V")
@@
 			)
 		)
-		(property "Footprint" "B6B-XH-A:JST_B6B-XH-A"
+		(property "Footprint" "Connector_JST:JST_EH_S6B-EH_1x06_P2.50mm_Horizontal"
 			(at 106.68 29.21 0)
 			(effects
@@
 			)
 		)
+		(pin "SX_MOSI" output
+			(at 187.96 96.52 180)
+			(effects
+				(font
+					(size 1.27 1.27)
+				)
+				(justify left)
+			)
+		)
+		(pin "SX_MISO" output
+			(at 187.96 86.36 180)
+			(effects
+				(font
+					(size 1.27 1.27)
+				)
+				(justify left)
+			)
+		)
+		(pin "GP1" input
+			(at 196.85 74.93 90)
+			(effects
+				(font
+					(size 1.27 1.27)
+				)
+				(justify right)
+			)
+		)
+		(pin "RFIO" input
+			(at 191.77 74.93 90)
+			(effects
+				(font
+					(size 1.27 1.27)
+				)
+				(justify right)
+			)
+		)
+		(pin "SX_CS" output
+			(at 187.96 88.9 180)
+			(effects
+				(font
+					(size 1.27 1.27)
+				)
+				(justify left)
+			)
+		)
+		(pin "SX_SCK" output
+			(at 187.96 99.06 180)
+			(effects
+				(font
+					(size 1.27 1.27)
+				)
+				(justify left)
+			)
+		)

Commit message: finally............
Connections:
- net SX_MOSI renamed 1_2GHz_Frontend/SX_MOSI
- net SX_SCK renamed 1_2GHz_Frontend/SX_SCK
Other:
- sheet 1_2GHz_Frontend ports: added SX_MOSI, SX_SCK; removed none
Changed lines of the file:
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@@
-		)
-	)
-	(hierarchical_label "SX_MOSI"
-		(shape output)
-		(at 111.76 146.05 270)
-		(effects
-			(font
-				(size 1.27 1.27)
-			)
-			(justify right)
-		)
-	)
-	(hierarchical_label "SX_SCK"
-		(shape input)
-		(at 109.22 146.05 270)
-		(effects
-			(font
-				(size 1.27 1.27)
-			)
-			(justify right)
 		)
 	)
@@
 			(effects
 				(font
+					(size 1.27 1.27)
+				)
+				(justify right)
+			)
+		)
+		(pin "SX_MOSI" output
+			(at 111.76 146.05 90)
+			(effects
+				(font
+					(size 1.27 1.27)
+				)
+				(justify right)
+			)
+		)
+		(pin "SX_SCK" input
+			(at 109.22 146.05 90)
+			(effects
+				(font
