File: KiCad/ENIAC/RX_path.kicad_sch (KiCad schematic)
At the start: 39 parts, among them Q1 MMBT3904, U13 LT5560, U4 QPC6713, U5 PCA9536DP, U8 QPL9504

Commit message: netclasses SUCK
Parts:
- removed C11, C12, C13: C, symbol Device:C
- removed L4: L, symbol Device:L
- C59: renamed from C31; value C -> 68pF; footprint (none) -> Capacitor_SMD:C_0603_1608Metric
- C60: renamed from C10; value C -> 1pF; footprint (none) -> Capacitor_SMD:C_0603_1608Metric
- C61: renamed from C46; value C -> NC; footprint (none) -> Capacitor_SMD:C_0603_1608Metric
- C62: renamed from C66; value C -> 10pF; footprint (none) -> Capacitor_SMD:C_0603_1608Metric
- C63: renamed from C68; value C -> 1nF; footprint (none) -> Capacitor_SMD:C_0603_1608Metric
- C64: renamed from C67; value C -> 1uF; footprint (none) -> Capacitor_SMD:C_0603_1608Metric
- C65: renamed from C48; value C -> 1nF; footprint (none) -> Capacitor_SMD:C_0603_1608Metric
- C66: renamed from C63; value C -> 10pF; footprint (none) -> Capacitor_SMD:C_0603_1608Metric
- C67: renamed from C49; value C -> NC; footprint (none) -> Capacitor_SMD:C_0603_1608Metric
- C68: renamed from C47; value C -> 0.1uF; footprint (none) -> Capacitor_SMD:C_0603_1608Metric
- C69: renamed from C64; value C -> NC; footprint (none) -> Capacitor_SMD:C_0603_1608Metric
- C70: renamed from C65; value C -> NC; footprint (none) -> Capacitor_SMD:C_0603_1608Metric
- C71: renamed from C69; value C -> 1nF; footprint (none) -> Capacitor_SMD:C_0603_1608Metric
- C72: renamed from C50; value C -> 68pF; footprint (none) -> Capacitor_SMD:C_0603_1608Metric
- C73: renamed from C15; value C -> 1uF; footprint (none) -> Capacitor_SMD:C_0603_1608Metric
- C74: renamed from C14; value C -> 2.2pF; footprint (none) -> Capacitor_SMD:C_0603_1608Metric
- C75: renamed from C16; value C -> 1uF; footprint (none) -> Capacitor_SMD:C_0603_1608Metric
- FL3: renamed from FL1; footprint SMD5_SAW-B7520_QUA -> AFS14A04_1575_42_T3:FIL_AFS14A04-1575.42-T3
- L10: renamed from L5; value L -> JP; footprint (none) -> Inductor_SMD:L_0603_1608Metric
- L11: renamed from L6; value L -> JP; footprint (none) -> Inductor_SMD:L_0603_1608Metric
- L6: renamed from L2; value L -> 3.9nH; footprint (none) -> Inductor_SMD:L_0603_1608Metric
- L7: renamed from L3; value L -> 3.9nH; footprint (none) -> Inductor_SMD:L_0603_1608Metric
- L8: renamed from L10; value L -> JP; footprint (none) -> Inductor_SMD:L_0603_1608Metric
- L9: renamed from L7; value L -> 18nH; footprint (none) -> Inductor_SMD:L_0603_1608Metric
- R14: renamed from R18; footprint (none) -> Resistor_SMD:R_0603_1608Metric
- R15: renamed from R19; footprint (none) -> Resistor_SMD:R_0603_1608Metric
- R16: renamed from R20; footprint (none) -> Resistor_SMD:R_0603_1608Metric
- R17: renamed from R4; value R -> 3; footprint (none) -> Resistor_SMD:R_0603_1608Metric
- TR1, TR2: footprint 0896BM15A0001E:FIL_0896BM15E0025E -> TRANSGENDE:SMT_15B0050E_JOT
- U13: renamed from U4; footprint HCP_16_1_ADI -> Package_DFN_QFN:QFN-16-1EP_3x3mm_P0.5mm_EP1.7x1.7mm_ThermalVias
- renumbered U13 to U10, U8 to U11, U5 to U12
Connections:
- net in_bal+: now reaches C74.2, L10.2, TR2.3
- net in_bal-: now reaches C74.1, L11.2, TR2.4
- net LNA out: now reaches C67.1, C72.1, L9.2, U11.7 (RF_OUT)
- net evil1: now reaches C66.2, C69.1, L8.2
- net bal_out+: now reaches L6.2, TR1.3
- net bal_out-: now reaches L7.2, TR1.4
- net LNA in: now reaches C59.2, C61.1, U11.2 (RF_IN)
Other:
- moved on the sheet: L6, L7

Commit message: PEAK PLL ROUTING
Connections:
- net OUT+ renamed OUT_p
- net OUT- renamed OUT_n
- net bal_out+ renamed bal_out_p
- net bal_out- renamed bal_out_n
Changed lines of the file:
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@@
 		)
 	)
-	(label "OUT-"
+	(label "OUT_n"
 		(at 31.75 101.6 180)
 		(effects
@@
 		)
 	)
-	(label "OUT+"
+	(label "OUT_p"
 		(at 31.75 104.14 180)
 		(effects
@@
 		)
 	)
-	(label "OUT-"
+	(label "OUT_n"
 		(at 68.58 160.02 0)
 		(effects
@@
 		)
 	)
-	(label "OUT+"
+	(label "OUT_p"
 		(at 68.58 149.86 0)
 		(effects
@@
 		)
 	)
-	(label "bal_out+"
+	(label "bal_out_p"
 		(at 58.42 149.86 0)
 		(effects
@@
 		)
 	)
-	(label "bal_out-"
+	(label "bal_out_n"
 		(at 58.42 160.02 0)
 		(effects

Commit message: finally............
Connections:
- net +3.3VA: no longer U11.5 (~{EN})
- net at Q1.3 (C), R15.1: now also U11.5 (~{EN})
- net 3.3VD renamed +3.3VD
- net IN+ renamed IN_p
- net IN- renamed IN_n
- net in_bal+ renamed in_bal_p
- net in_bal- renamed in_bal_n
Other:
- moved on the sheet: Q1, R15, R16
Changed lines of the file:
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@@
 	)
 	(junction
-		(at 57.15 57.15)
-		(diameter 0)
-		(color 0 0 0 0)
-	)
-	(junction
 		(at 233.68 118.11)
 		(diameter 0)
@@
 	)
 	(junction
+		(at 57.15 66.04)
+		(diameter 0)
+		(color 0 0 0 0)
+	)
+	(junction
 		(at 233.68 110.49)
 		(diameter 0)
@@
 	(wire
 		(pts
+			(xy 57.15 57.15) (xy 57.15 66.04)
+		)
+		(stroke
+			(width 0)
+			(type default)
+		)
+	)
+	(wire
+		(pts
 			(xy 38.1 149.86) (xy 48.26 149.86)
 		)
@@
 	(wire
 		(pts
+			(xy 48.26 66.04) (xy 44.45 66.04)
+		)
+		(stroke
+			(width 0)
+			(type default)
+		)
+	)
+	(wire
+		(pts
+			(xy 57.15 66.04) (xy 64.77 66.04)
+		)
+		(stroke
+			(width 0)
+			(type default)
+		)
+	)
+	(wire
+		(pts
 			(xy 41.91 49.53) (xy 41.91 46.99)
 		)
@@
 	(wire
 		(pts
-			(xy 88.9 66.04) (xy 93.98 66.04)
+			(xy 74.93 66.04) (xy 80.01 66.04)
 		)
 		(stroke
@@
 	(wire
 		(pts
-			(xy 80.01 77.47) (xy 83.82 77.47)
+			(xy 66.04 77.47) (xy 69.85 77.47)
 		)
 		(stroke
@@
 	(wire
 		(pts
-			(xy 215.9 146.05) (xy 217.17 146.05)
+			(xy 185.42 127) (xy 187.96 127)
 		)
 		(stroke
@@
 		)
 	)
-	(polyline
+	(wire
 		(pts
-			(xy 132.08 121.92) (xy 181.61 121.92)
+			(xy 215.9 146.05) (xy 217.17 146.05)
 		)
 		(stroke
@@
 		)
 	)
-	(wire
+	(polyline
 		(pts
-			(xy 146.05 102.87) (xy 157.48 102.87)
+			(xy 132.08 121.92) (xy 181.61 121.92)
 		)
 		(stroke
@@
 	(wire
 		(pts
-			(xy 157.48 102.87) (xy 158.75 102.87)
+			(xy 146.05 102.87) (xy 157.48 102.87)
 		)
 		(stroke
@@
 	(wire
 		(pts
-			(xy 57.15 57.15) (xy 57.15 66.04)
+			(xy 157.48 102.87) (xy 158.75 102.87)
 		)
 		(stroke
@@
 	(wire
 		(pts
-			(xy 64.77 66.04) (xy 57.15 66.04)
+			(xy 44.45 66.04) (xy 44.45 68.58)
 		)
 		(stroke
@@
 	(wire
 		(pts
-			(xy 72.39 66.04) (xy 78.74 66.04)
+			(xy 55.88 66.04) (xy 57.15 66.04)
 		)
 		(stroke
@@
 	(wire
 		(pts
-			(xy 83.82 77.47) (xy 83.82 73.66)
+			(xy 69.85 77.47) (xy 69.85 73.66)
 		)
 		(stroke
@@
 	(wire
 		(pts
+			(xy 236.22 127) (xy 233.68 127)
+		)
+		(stroke
+			(width 0)
+			(type default)
+		)
+	)
+	(wire
+		(pts
 			(xy 57.15 31.75) (xy 59.69 31.75)
 		)
@@
 	(wire
 		(pts
-			(xy 68.58 77.47) (xy 72.39 77.47)
+			(xy 54.61 77.47) (xy 58.42 77.47)
 		)
 		(stroke
@@
 	(wire
 		(pts
-			(xy 57.15 57.15) (xy 64.77 57.15)
-		)
-		(stroke
-			(width 0)
-			(type default)
-		)
-	)
-	(wire
-		(pts
 			(xy 80.01 99.06) (xy 80.01 97.79)
 		)
@@
 		)
 	)
-	(label "in_bal+"
+	(label "in_bal_p"
 		(at 149.86 92.71 0)
 		(effects
@@
 		)
 	)
-	(label "IN+"
+	(label "IN_p"
 		(at 167.64 92.71 0)
 		(effects
@@
 	)
 	(label "RX_att"
-		(at 187.96 127 180)
+		(at 185.42 127 180)
 		(effects
 			(font
@@
 		)
 	)
-	(label "IN-"
+	(label "IN_n"
 		(at 167.64 102.87 0)
 		(effects
@@
 		)
 	)
-	(label "IN+"
+	(label "IN_p"
 		(at 52.07 106.68 0)
 		(effects
@@
 		)
 	)
-	(label "IN-"
+	(label "IN_n"
 		(at 52.07 104.14 0)
 		(effects
@@
 		)
 	)
-	(label "in_bal-"
+	(label "in_bal_n"
 		(at 148.59 102.87 0)
 		(effects
@@
 	)
 	(label "1.2RX_BPF"
-		(at 233.68 127 0)
+		(at 236.22 127 0)
 		(effects
 			(font
@@
 	(hierarchical_label "GP1"
 		(shape input)
-		(at 68.58 77.47 180)
+		(at 54.61 77.47 180)
 		(effects
 			(font
@@
 			)
 		)
-		(property "Value" "3.3VD"
+		(property "Value" "+3.3VD"
 			(at 233.68 99.568 90)
 			(effects
@@
 	(symbol
 		(lib_id "power:+3.3VA")
-		(at 64.77 57.15 270)
+		(at 44.45 68.58 180)
 		(unit 1)
 		(exclude_from_sim no)
@@
 		(dnp no)
 		(property "Reference" "#PWR0110"
-			(at 60.96 57.15 0)
+			(at 44.45 64.77 0)
 			(effects
 				(font
@@
 		)
 		(property "Value" "+3.3VA"
-			(at 68.58 57.1499 90)
+			(at 44.4501 72.39 90)
 			(effects
 				(font
@@
 		)
 		(property "Footprint" ""
-			(at 64.77 57.15 0)
+			(at 44.45 68.58 0)
 			(effects
 				(font
@@
 		)
 		(property "Datasheet" ""
-			(at 64.77 57.15 0)
+			(at 44.45 68.58 0)
 			(effects
 				(font
@@
 		)
 		(property "Description" "Power symbol creates a global label with name \"+3.3VA\""
-			(at 64.77 57.15 0)
+			(at 44.45 68.58 0)
 			(effects
 				(font
@@
 	(symbol
 		(lib_id "power:GND")
-		(at 93.98 66.04 90)
+		(at 80.01 66.04 90)
 		(unit 1)
 		(exclude_from_sim no)
@@
 		(fields_autoplaced yes)
 		(property "Reference" "#PWR0120"
-			(at 100.33 66.04 0)
+			(at 86.36 66.04 0)
 			(effects
 				(font
@@
 		)
 		(property "Value" "GND"
-			(at 97.79 66.0399 90)
+			(at 83.82 66.0399 90)
 			(effects
 				(font
@@
 		)
 		(property "Footprint" ""
-			(at 93.98 66.04 0)
+			(at 80.01 66.04 0)
 			(effects
 				(font
@@
 		)
 		(property "Datasheet" ""
-			(at 93.98 66.04 0)
+			(at 80.01 66.04 0)
 			(effects
 				(font
@@
 		)
 		(property "Description" "Power symbol creates a global label with name \"GND\" , ground"
-			(at 93.98 66.04 0)
+			(at 80.01 66.04 0)
 			(effects
 				(font
@@
 	(symbol
 		(lib_id "Transistor_BJT:MMBT3904")
-		(at 83.82 68.58 90)
+		(at 69.85 68.58 90)
 		(unit 1)
 		(exclude_from_sim no)
@@
 		(fields_autoplaced yes)
 		(property "Reference" "Q1"
-			(at 83.82 59.69 90)
+			(at 69.85 59.69 90)
 			(effects
 				(font
@@
 		)
 		(property "Value" "MMBT3904"
-			(at 83.82 62.23 90)
+			(at 69.85 62.23 90)
 			(effects
 				(font
@@
 		)
 		(property "Footprint" "Package_TO_SOT_SMD:SOT-23"
-			(at 85.725 63.5 0)
+			(at 71.755 63.5 0)
 			(effects
 				(font
@@
 		)
 		(property "Datasheet" "https://www.onsemi.com/pdf/datasheet/pzt3904-d.pdf"
-			(at 83.82 68.58 0)
+			(at 69.85 68.58 0)
 			(effects
 				(font
@@
 		)
 		(property "Description" "0.2A Ic, 40V Vce, Small Signal NPN Transistor, SOT-23"
-			(at 83.82 68.58 0)
+			(at 69.85 68.58 0)
 			(effects
 				(font
@@
 	(symbol
 		(lib_id "Device:R")
-		(at 76.2 77.47 270)
+		(at 62.23 77.47 270)
 		(unit 1)
 		(exclude_from_sim no)
@@
 		(fields_autoplaced yes)
 		(property "Reference" "R16"
-			(at 76.2 71.12 90)
+			(at 62.23 71.12 90)
 			(effects
 				(font
@@
 		)
 		(property "Value" "1k"
-			(at 76.2 73.66 90)
+			(at 62.23 73.66 90)
 			(effects
 				(font
@@
 		)
 		(property "Footprint" "Resistor_SMD:R_0603_1608Metric"
-			(at 76.2 75.692 90)
+			(at 62.23 75.692 90)
 			(effects
 				(font
@@
 		)
 		(property "Datasheet" "~"
-			(at 76.2 77.47 0)
+			(at 62.23 77.47 0)
 			(effects
 				(font
@@
 		)
 		(property "Description" "Resistor"
-			(at 76.2 77.47 0)
+			(at 62.23 77.47 0)
 			(effects
 				(font
@@
 	(symbol
 		(lib_id "Device:R")
-		(at 68.58 66.04 270)
+		(at 52.07 66.04 270)
 		(unit 1)
 		(exclude_from_sim no)
@@
 		(on_board yes)
 		(dnp no)
-		(fields_autoplaced yes)
 		(property "Reference" "R15"
-			(at 68.58 59.69 90)
+			(at 52.07 69.342 90)
 			(effects
 				(font
@@
 		)
 		(property "Value" "10k"
-			(at 68.58 62.23 90)
+			(at 52.07 71.882 90)
 			(effects
 				(font
@@
 		)
 		(property "Footprint" "Resistor_SMD:R_0603_1608Metric"
-			(at 68.58 64.262 90)
+			(at 52.07 64.262 90)
 			(effects
 				(font
@@
 		)
 		(property "Datasheet" "~"
-			(at 68.58 66.04 0)
+			(at 52.07 66.04 0)
 			(effects
 				(font
@@
 		)
 		(property "Description" "Resistor"
-			(at 68.58 66.04 0)
+			(at 52.07 66.04 0)
 			(effects
 				(font
@@
 			)
 		)
-		(property "Value" "3.3VD"
+		(property "Value" "+3.3VD"
 			(at 168.402 130.81 90)
 			(effects
