File: KiCad/ENIAC/1_2GHz_Frontend.kicad_sch (KiCad schematic)
At the start: 1 part, among them U12 HMC361S8GE

Commit message: john d tickle
Parts:
- added C63, C64, C65, C66, C67, C68, C69: C, symbol Device:C
- added L10: L, symbol Device:L
- added U13: LT5560, Package_DFN_QFN:DFN-8-1EP_3x3mm_P0.5mm_EP1.66x2.38mm, symbol RF_Mixer:LT5560
- added U3: 4259-63, SC-70-6_PSM, symbol 2025-11-10_00-05-56:4259-63
Connections:
- net GP1: now also U3.4 (CTRL)
- new net: C63.2, C64.1, L10.2
- new net: C66.1, U13.8 (LO+)
- new net +3.3VA: C67.1, C68.1, C69.1, U13.7 (VCC)
- new net +3.3V_RF: U3.6 (*CTRL/VDD)
- new net 2.4GHZ_RX: U3.1 (RF1)
- new net 2.4GHz_TX: U3.3 (RF2)
- new net GND: C64.2, C65.2, C66.2, C67.2, C68.2, C69.2, U3.2 (GND)
- new net IN+: U13.3 (IN+)
- new net IN-: U13.4 (IN-)
- new net LO: C63.1
- new net LO-: C65.1, L10.1, U13.1 (LO-)
- new net RFIO: U3.5 (RFC)
Other:
- sheet 3.6GHz LO ports: added RFOut; removed none

Commit message: funny commit message
Parts:
- removed C63, C64, C65, C66, C67, C68, C69: C, symbol Device:C
- removed L10: L, symbol Device:L
- removed U13: LT5560, Package_DFN_QFN:DFN-8-1EP_3x3mm_P0.5mm_EP1.66x2.38mm, symbol RF_Mixer:LT5560
- added C51, C52, C53, C54, C55, C56, C57, C58, C59, C60, C61, C62, C70, C71, C72, C73, C74, C75, C76, C77, C78, C79, C80, C81: C, symbol Device:C
- added FL3: AFII-SW-0059, SMD5_SAW-B7520_QUA, symbol 2026-03-09_02-05-18:B39242B7520P810
- added L11, L12, L13, L14: L, symbol Device:L
- added R21, R22, R23: R, symbol Device:R
- added U6: BMT321, Package_DFN_QFN:VQFN-12-1EP_4x4mm_P0.8mm_EP2.1x2.1mm_ThermalVias, symbol Driver_Motor:EMC2303-x-KP
Connections:
- net GND: now also U12.8 (GND), U12.9 (GND), C52.2, C53.2, C54.2, C59.1, C60.1, C62.2, C70.1, C71.1, C72.1, C73.1, C74.2, C75.1, C76.2, C77.2, C78.2, C79.1, C80.1, C81.1, FL3.2 (GROUND), FL3.3 (GROUND), FL3.5 (GROUND), L11.1, U6.13 (GND)
- net at U12.1 (*OUT): now also C55.1
- net at U12.3 (OUT): now also C56.2
- net +5VA: now reaches U12.4 (VCC)
- net +5VA: now also C53.1, C54.1, C62.1, C70.2, C72.2, C73.2, C74.1, C75.2, C79.2, C80.2, C81.2, L13.1, L14.1, R21.1, R22.1, R23.1
- net at U12.5 (IN): now also C51.2
- net at U12.7 (*IN): now also C52.1
- net 2.4GHZ_RX renamed RX_path/RX_OUT
- new net: C57.2, C58.1, L11.2
- new net: C59.2, C61.1, L12.2
- new net: C71.2, L13.2, U6.11 (VCC)
- new net: C58.2, U6.2 (RF_IN), U6.3 (RF_IN)
- new net 1.2TX: C56.1
- new net 1.2TX_BPF: C57.1, FL3.4 (OUTPUT)
- new net 1.2_FD: FL3.1 (INPUT)
- new net I_REF1: C78.1, R23.2, U6.4 (I_REF1)
- new net I_REF2: C77.1, R22.2, U6.5 (I_REF2)
- new net OUT_BIAS: C60.2, L12.1, L14.2, U6.7 (RF_OUT), U6.8 (RF_OUT), U6.9 (RF_OUT)
- new net TX_ANT: C61.2
- new net V_BIAS: C76.1, R21.2, U6.6 (V_BIAS)
Other:
- removed sheet 3.6GHz LO
- added sheet RX_path (RX_path.kicad_sch)
- note added: "1 2 3"
- moved on the sheet: U12, U3

Commit message: netclasses SUCK
Parts:
- added FL1: B39242B9413K610, AFS14A04_1575_42_T3:FIL_AFS14A04-1575.42-T3, symbol 2026-03-09_02-05-18:B39242B7520P810
- C1: renamed from C52; value C -> 100pF; footprint (none) -> Capacitor_SMD:C_0603_1608Metric
- C10: renamed from C75; value C -> NC; footprint (none) -> Capacitor_SMD:C_0603_1608Metric
- C11: renamed from C78; value C -> NC; footprint (none) -> Capacitor_SMD:C_0603_1608Metric
- C12: renamed from C77; value C -> NC; footprint (none) -> Capacitor_SMD:C_0603_1608Metric
- C13: renamed from C76; value C -> NC; footprint (none) -> Capacitor_SMD:C_0603_1608Metric
- C14: renamed from C57; value C -> 47nF; footprint (none) -> Capacitor_SMD:C_0603_1608Metric
- C15: renamed from C81; value C -> NC; footprint (none) -> Capacitor_SMD:C_0603_1608Metric
- C16: renamed from C80; value C -> 100pF; footprint (none) -> Capacitor_SMD:C_0603_1608Metric
- C17: renamed from C79; value C -> 1uF; footprint (none) -> Capacitor_SMD:C_0603_1608Metric
- C18: renamed from C62; value C -> 1uF; footprint (none) -> Capacitor_SMD:C_0603_1608Metric
- C19: renamed from C58; value C -> 1.2pF; footprint (none) -> Capacitor_SMD:C_0603_1608Metric
- C2: renamed from C51; value C -> 100pF; footprint (none) -> Capacitor_SMD:C_0603_1608Metric
- C20: renamed from C70; value C -> 100pF; footprint (none) -> Capacitor_SMD:C_0603_1608Metric
- C21: renamed from C71; value C -> NC; footprint (none) -> Capacitor_SMD:C_0603_1608Metric
- C22: renamed from C59; value C -> 6.8pF; footprint (none) -> Capacitor_SMD:C_0603_1608Metric
- C23: renamed from C60; value C -> 3.3pF; footprint (none) -> Capacitor_SMD:C_0603_1608Metric
- C24: renamed from C61; value C -> 47pF; footprint (none) -> Capacitor_SMD:C_0603_1608Metric
- C3: renamed from C55; value C -> 100pF; footprint (none) -> Capacitor_SMD:C_0603_1608Metric
- C4: renamed from C56; value C -> 100pF; footprint (none) -> Capacitor_SMD:C_0603_1608Metric
- C5: renamed from C54; value C -> 10uF; footprint (none) -> Capacitor_SMD:C_0603_1608Metric
- C6: renamed from C53; value C -> 1nF; footprint (none) -> Capacitor_SMD:C_0603_1608Metric
- C7: renamed from C72; value C -> 1uF; footprint (none) -> Capacitor_SMD:C_0603_1608Metric
- C8: renamed from C73; value C -> 47pF; footprint (none) -> Capacitor_SMD:C_0603_1608Metric
- C9: renamed from C74; value C -> NC; footprint (none) -> Capacitor_SMD:C_0603_1608Metric
- FL2: renamed from FL3; footprint SMD5_SAW-B7520_QUA -> AFS14A04_1575_42_T3:FIL_AFS14A04-1575.42-T3
- L1: renamed from L11; value L -> 10nH; footprint (none) -> Inductor_SMD:L_0603_1608Metric
- L2: renamed from L14; value L -> 22nH; footprint (none) -> Inductor_SMD:L_0603_1608Metric
- L3: renamed from L13; value L -> 33nH; footprint (none) -> Inductor_SMD:L_0603_1608Metric
- L4: renamed from L12; value L -> 3.9nH; footprint (none) -> Inductor_SMD:L_0603_1608Metric
- R1: renamed from R23; value R -> 300; footprint (none) -> Resistor_SMD:R_0603_1608Metric
- R2: renamed from R22; value R -> 430; footprint (none) -> Resistor_SMD:R_0603_1608Metric
- R3: renamed from R21; value R -> 82; footprint (none) -> Resistor_SMD:R_0603_1608Metric
- U1: renamed from U3; footprint SC-70-6_PSM -> Package_TO_SOT_SMD:SOT-363_SC-70-6_Handsoldering
- U2: renamed from U12; footprint RD-8-3_ADI -> Package_SO:SOIC-8-1EP_3.9x4.9mm_P1.27mm_EP2.41x3.3mm_ThermalVias
- renumbered U6 to U3
Connections:
- net 1.2TX is gone; now on net 1.2_FD: C4.1
- net 2.4GHz_TX: now also C2.1
- net GND: now also C3.2, FL1.2 (GROUND), FL1.3 (GROUND), FL1.5 (GROUND)
- net RX_path/RX_OUT: now also FL1.4 (OUTPUT); no longer U1.1 (RF1)
- net HGH: now reaches C14.2, C19.1, L1.2
- net csnc: now reaches C22.2, C24.1, L4.2
- net 2.4ejfsdn: now reaches C2.2, U2.5 (IN)
- net LABE: now reaches C4.2, U2.3 (OUT)
- net MOMG: now reaches C19.2, U3.2 (RF_IN), U3.3 (RF_IN)
- new net 2.4rxx: FL1.1 (INPUT), U1.1 (RF1)
Other:
- moved on the sheet: C2

Commit message: finally............
Connections:
- net +3.3V_RF renamed +3.3VA
Changed lines of the file:
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@@
 			)
 		)
-		(property "Value" "+3.3V_RF"
+		(property "Value" "+3.3VA"
 			(at 25.4 124.46 0)
 			(effects

Commit message: i hate sims
Parts:
- U1: value 4259-63 -> AS215-92
Connections:
- net +3.3VA is gone; now on net GND: U1.6 (*CTRL/VDD)
Changed lines of the file:
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@@
 		(fields_autoplaced yes)
 		(property "Reference" "U1"
-			(at 50.8 125.73 0)
+			(at 50.8 100.33 0)
 			(effects
 				(font
@@
 			)
 		)
-		(property "Value" "4259-63"
-			(at 50.8 123.19 0)
+		(property "Value" "AS215-92"
+			(at 50.8 102.87 0)
 			(effects
 				(font
@@
 	)
 	(symbol
+		(lib_id "power:GND")
+		(at 25.4 119.38 0)
+		(unit 1)
+		(exclude_from_sim no)
+		(in_bom yes)
+		(on_board yes)
+		(dnp no)
+		(fields_autoplaced yes)
+		(property "Reference" "#PWR03"
+			(at 25.4 125.73 0)
+			(effects
+				(font
+					(size 1.27 1.27)
+				)
+				(hide yes)
+			)
+		)
+		(property "Value" "GND"
+			(at 25.4 124.46 0)
+			(effects
+				(font
+					(size 1.27 1.27)
+				)
+			)
+		)
+		(property "Footprint" ""
+			(at 25.4 119.38 0)
+			(effects
+				(font
+					(size 1.27 1.27)
+				)
+				(hide yes)
+			)
+		)
+		(property "Datasheet" ""
+			(at 25.4 119.38 0)
+			(effects
+				(font
+					(size 1.27 1.27)
+				)
+				(hide yes)
+			)
+		)
+		(property "Description" "Power symbol creates a global label with name \"GND\" , ground"
+			(at 25.4 119.38 0)
+			(effects
+				(font
+					(size 1.27 1.27)
+				)
+				(hide yes)
+			)
+		)
+		(pin "1"
+		)
+		(instances
+			(project "ENIAC"
+				(path "/028e33f3-2d21-4744-a260-423608f4c0b7/cea77956-cbc5-4ddc-8ead-a341e8686604"
+					(reference "#PWR03")
+					(unit 1)
+				)
+			)
+		)
+	)
+	(symbol
 		(lib_id "Device:C")
 		(at 222.25 102.87 90)
@@
 					(unit 1)
 				)
-			)
-		)
-	)
-	(symbol
-		(lib_id "power:+3.3VA")
-		(at 25.4 119.38 180)
-		(unit 1)
-		(exclude_from_sim no)
-		(in_bom yes)
-		(on_board yes)
-		(dnp no)
-		(fields_autoplaced yes)
-		(property "Reference" "#PWR03"
-			(at 25.4 115.57 0)
-			(effects
-				(font
-					(size 1.27 1.27)
-				)
-				(hide yes)
-			)
-		)
-		(property "Value" "+3.3VA"
-			(at 25.4 124.46 0)
-			(effects
-				(font
-					(size 1.27 1.27)
-				)
-			)
-		)
-		(property "Footprint" ""
-			(at 25.4 119.38 0)
-			(effects
-				(font
-					(size 1.27 1.27)
-				)
-				(hide yes)
-			)
-		)
-		(property "Datasheet" ""
-			(at 25.4 119.38 0)
-			(effects
-				(font
-					(size 1.27 1.27)
-				)
-				(hide yes)
-			)
-		)
-		(property "Description" "Power symbol creates a global label with name \"+3.3VA\""
-			(at 25.4 119.38 0)
-			(effects
-				(font
-					(size 1.27 1.27)
-				)
-				(hide yes)
-			)
-		)
-		(pin "1"
-		)
-		(instances
-			(project "ENIAC"
-				(path "/028e33f3-2d21-4744-a260-423608f4c0b7/cea77956-cbc5-4ddc-8ead-a341e8686604"
-					(reference "#PWR03")
-					(unit 1)
-				)
