File: KiCad/ENIAC/ANT_switch.kicad_sch (KiCad schematic)
At the start: 13 parts, among them J4 Conn_Coaxial, U8 4259-63

Commit message: john d tickle
Parts:
- renumbered AE1 to AE2, C26 to C40, C27 to C41, C28 to C42, C29 to C43, C30 to C44, C31 to C45, D1 to D2, FL1 to FL2, J4 to J5, L6 to L8, L7 to L9, U8 to U1
Other:
- moved on the sheet: AE2, C40, C41, C42, C43, C44, C45, D2, FL2, J5, L8, L9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

Commit message: funny commit message
Parts:
- removed AE2: MLPF-WB55-01E3, MLPF-WB55-01E3_STM, symbol 2025-11-10_00-22-04:MLPF-WB55-01E3
- removed FL2: 2450LP14B0100001T, 3550LP_JOT, symbol 2025-11-10_17-30-01:3550LP14A0300001T
- added FL2: AFII-SW-0059, SMD5_SAW-B7520_QUA, symbol 2026-03-09_02-05-18:B39242B7520P810
- added FL5: LFCN-1325, Filter:Filter_Mini-Circuits_FV1206, symbol RF_Filter:LFCN-1325
Connections:
- net ANT_TX: now also U1.3 (RF2)
- net GND: now also FL2.2 (GROUND), FL2.3 (GROUND), FL2.5 (GROUND), FL5.2 (GND), FL5.4 (GND); no longer U1.2 (GND)
- net ANT_BPF: now reaches C41.2, L9.1
- net ANT_BPF: now also FL2.4 (OUTPUT); no longer U1.5 (RFC)
- net at C42.2, L9.2: now also FL5.3 (OUT)
- net at C43.2, C44.1: now also FL5.1 (IN)
- new net ANT_RF: FL2.1 (INPUT), U1.5 (RFC)
Other:
- moved on the sheet: C40, C41, C42, C43, C44, C45, D2, J5, L8, L9, U1

Commit message: netclasses SUCK
Parts:
- C76: renamed from C40; value ? -> 47pF; footprint (none) -> Capacitor_SMD:C_0603_1608Metric
- C77: renamed from C41; value ? -> NC; footprint (none) -> Capacitor_SMD:C_0603_1608Metric
- C78: renamed from C42; value ? -> NC; footprint (none) -> Capacitor_SMD:C_0603_1608Metric
- C79: renamed from C43; footprint (none) -> Capacitor_SMD:C_0603_1608Metric
- C80: renamed from C44; value ? -> 47pF; footprint (none) -> Capacitor_SMD:C_0603_1608Metric
- C81: renamed from C45; footprint (none) -> Capacitor_SMD:C_0603_1608Metric
- FL4: renamed from FL2; footprint SMD5_SAW-B7520_QUA -> AFS14A04_1575_42_T3:FIL_AFS14A04-1575.42-T3
- J3: renamed from J5; footprint (none) -> Connector_Coaxial:SMA_Molex_73251-1153_EdgeMount_Horizontal
- L12: renamed from L8; value ? -> JP; footprint (none) -> Inductor_SMD:L_0603_1608Metric
- L13: renamed from L9; value ? -> 0; footprint (none) -> Inductor_SMD:L_0603_1608Metric
- U14: renamed from U1; footprint SC-70-6_PSM -> Package_TO_SOT_SMD:SOT-363_SC-70-6_Handsoldering
- renumbered D2 to D1
Connections:
- net lpf in: now reaches C78.2, FL5.3 (OUT), L13.2
- net coax: now reaches C80.2, C81.2, D1.2 (A2), J3.1 (In)
- net lpf out: now reaches C79.2, C80.1, FL5.1 (IN)

Commit message: finally............
Parts:
- added Q2: MMBT3904, Package_TO_SOT_SMD:SOT-23, symbol Transistor_BJT:MMBT3904
- added R18: 10k, Resistor_SMD:R_0603_1608Metric, symbol Device:R
- added R19: 1k, Resistor_SMD:R_0603_1608Metric, symbol Device:R
Connections:
- net ANT_TX: now also U14.1 (RF1); no longer U14.3 (RF2)
- net GND: now also Q2.2 (E)
- net GP1: now also R19.2; no longer U14.4 (CTRL)
- net hatred: now reaches C76.2, L12.1
- net stipd': now reaches L12.2
- net stipd': now also U14.3 (RF2); no longer U14.1 (RF1)
- net +3.3V_RF renamed +3.3VA
- net +3.3VA: now also R18.2
- new net: Q2.1 (B), R19.1
- new net: Q2.3 (C), R18.1, U14.4 (CTRL)
Other:
- moved on the sheet: C76, L12, U14

Commit message: i hate sims
Parts:
- U14: value 4259-63 -> AS215-92
Connections:
- net +3.3VA: no longer U14.6 (*CTRL/VDD)
- net GND: now also U14.6 (*CTRL/VDD)
Changed lines of the file:
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@@
+	)
+	(symbol
+		(lib_id "power:GND")
+		(at 115.57 45.72 180)
+		(unit 1)
+		(exclude_from_sim no)
+		(in_bom yes)
+		(on_board yes)
+		(dnp no)
+		(fields_autoplaced yes)
+		(property "Reference" "#PWR0138"
+			(at 115.57 39.37 0)
+			(effects
+				(font
+					(size 1.27 1.27)
+				)
+				(hide yes)
+			)
+		)
+		(property "Value" "GND"
+			(at 115.57 40.64 0)
+			(effects
+				(font
+					(size 1.27 1.27)
+				)
+			)
+		)
+		(property "Footprint" ""
+			(at 115.57 45.72 0)
+			(effects
+				(font
+					(size 1.27 1.27)
+				)
+				(hide yes)
+			)
+		)
+		(property "Datasheet" ""
+			(at 115.57 45.72 0)
+			(effects
+				(font
+					(size 1.27 1.27)
+				)
+				(hide yes)
+			)
+		)
+		(property "Description" "Power symbol creates a global label with name \"GND\" , ground"
+			(at 115.57 45.72 0)
+			(effects
+				(font
+					(size 1.27 1.27)
+				)
+				(hide yes)
+			)
+		)
+		(pin "1"
+		)
+		(instances
+			(project ""
+				(path "/028e33f3-2d21-4744-a260-423608f4c0b7/cea77956-cbc5-4ddc-8ead-a341e8686604/c3720c13-f22a-4d2b-8cbe-8c286dd367c1"
+					(reference "#PWR0138")
+					(unit 1)
+				)
+			)
+		)
 	)
 	(symbol
@@
 			)
 		)
-		(property "Value" "4259-63"
+		(property "Value" "AS215-92"
 			(at 90.17 41.91 0)
 			(effects
@@
 					(unit 1)
 				)
-			)
-		)
-	)
-	(symbol
-		(lib_id "power:+3.3VA")
-		(at 115.57 45.72 0)
-		(unit 1)
-		(exclude_from_sim no)
-		(in_bom yes)
-		(on_board yes)
-		(dnp no)
-		(fields_autoplaced yes)
-		(property "Reference" "#PWR0138"
-			(at 115.57 49.53 0)
-			(effects
-				(font
-					(size 1.27 1.27)
-				)
-				(hide yes)
-			)
-		)
-		(property "Value" "+3.3VA"
-			(at 115.57 40.64 0)
-			(effects
-				(font
-					(size 1.27 1.27)
-				)
-			)
-		)
-		(property "Footprint" ""
-			(at 115.57 45.72 0)
-			(effects
-				(font
-					(size 1.27 1.27)
-				)
-				(hide yes)
-			)
-		)
-		(property "Datasheet" ""
-			(at 115.57 45.72 0)
-			(effects
-				(font
-					(size 1.27 1.27)
-				)
-				(hide yes)
-			)
-		)
-		(property "Description" "Power symbol creates a global label with name \"+3.3VA\""
-			(at 115.57 45.72 0)
-			(effects
-				(font
-					(size 1.27 1.27)
-				)
-				(hide yes)
-			)
-		)
-		(pin "1"
-		)
-		(instances
-			(project "ENIAC"
-				(path "/028e33f3-2d21-4744-a260-423608f4c0b7/cea77956-cbc5-4ddc-8ead-a341e8686604/c3720c13-f22a-4d2b-8cbe-8c286dd367c1"
-					(reference "#PWR0138")
-					(unit 1)
-				)
