File: KiCad/ENIAC/ENIAC.kicad_pcb (KiCad board)
At the start: 4 copper layers, 105.5 x 63.5 mm, 146 parts, among them J1 B6B-XH-A, J2 Conn_01x07_Pin, J3 Conn_Coaxial, Q1 MMBT3904, U1 4259-63, U10 LT5560, U11 QPL9504, U12 PCA9536DP, U13 QPC6713, U14 4259-63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

Commit message: PEAK PLL ROUTING
Parts:
- moved C11 140.2 mm to (163.7, 27.7)
- moved C12 140.2 mm to (163.7, 30.2)
- moved C15 140.2 mm to (163.7, 37.7)
- moved C8 140.2 mm to (163.7, 20.1)
- moved C9 140.2 mm to (163.7, 22.7)
- moved U3 140.2 mm to (176.8, 28.6)
- moved C1 140.2 mm to (159.6, 22.7)
- moved C10 140.2 mm to (163.7, 25.2)
- moved C13 140.2 mm to (163.7, 32.7)
- moved C14 140.2 mm to (163.7, 35.2)
- moved C16 140.2 mm to (167.7, 20.1)
- moved C17 140.2 mm to (167.7, 22.7)
- moved C18 140.2 mm to (167.7, 25.2)
- moved C19 140.2 mm to (167.7, 27.7)
- moved C20 140.2 mm to (167.7, 30.2)
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Connections:
- net /1_2GHz_Frontend/RX_path/OUT+ renamed /1_2GHz_Frontend/RX_path/OUT_p
- net /1_2GHz_Frontend/RX_path/OUT- renamed /1_2GHz_Frontend/RX_path/OUT_n
- net /1_2GHz_Frontend/RX_path/bal_out+ renamed /1_2GHz_Frontend/RX_path/bal_out_p
- net /1_2GHz_Frontend/RX_path/bal_out- renamed /1_2GHz_Frontend/RX_path/bal_out_n
- C35 pad 2: 3.3VD -> +3.3VD
- C39 pad 2: +3.3VA -> /1_2GHz_Frontend/RX_path/3.6GHz LO/VCCBYPASS
- FB6 pad 2: 3.3VD -> +3.3VD
- U4 pad 30: /1_2GHz_Frontend/RX_path/3.6GHz LO/BYPASS -> /1_2GHz_Frontend/RX_path/3.6GHz LO/VCCBYPASS
Routing:
- net /1_2GHz_Frontend/RX_path/3.6GHz LO/VccPLL1: track 0.00 -> 24.3 mm
- net /1_2GHz_Frontend/RX_path/3.6GHz LO/VccDig: track 0.00 -> 23.9 mm, vias 0 -> 2
- net /1_2GHz_Frontend/RX_path/3.6GHz LO/VccCP1: track 0.00 -> 21.8 mm
- net /1_2GHz_Frontend/RX_path/3.6GHz LO/VccOSCin: track 0.00 -> 21.4 mm, vias 0 -> 2
- net /1_2GHz_Frontend/RX_path/3.6GHz LO/VccCP2: track 0.00 -> 20.9 mm
- net /1_2GHz_Frontend/RX_path/3.6GHz LO/VccPLL2: track 0.00 -> 20.6 mm
- net Net-(U4-VCCFRAC): track 0.00 -> 6.60 mm
- net +3.3VA: track 11.4 -> 17.5 mm, vias 3 -> 9
- net Net-(U4-VREGFRAC): track 0.00 -> 5.21 mm
- net Net-(U4-VREFVCO): track 0.00 -> 5.19 mm
- net /1_2GHz_Frontend/RX_path/3.6GHz LO/CPOUT: track 0.00 -> 5.00 mm
- net Net-(U4-*OSCIN): track 0.00 -> 4.97 mm
- net Net-(U4-VREGRFOUT): track 0.00 -> 3.69 mm
- net Net-(Y1-OUTPUT): track 0.00 -> 3.63 mm
- net Net-(U4-VREGVCO): track 0.00 -> 3.35 mm
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
Commit message: finally............
Parts:
- added Q2: MMBT3904, Package_TO_SOT_SMD:SOT-23, F.Cu at (177.6, 89.9)
- added R18: 10k, Resistor_SMD:R_0603_1608Metric, F.Cu at (176.5, 94.4)
- added R19: 1k, Resistor_SMD:R_0603_1608Metric, F.Cu at (179.0, 94.4)
- moved L12 74.6 mm to (181.6, 80.3), turned to -90 degrees
- moved C79 68.0 mm to (192.2, 94.2), turned to 180 degrees
- moved C81 67.9 mm to (192.2, 99.4), turned to 180 degrees
- moved C80 67.3 mm to (191.4, 96.8), turned to -90 degrees
- moved L13 66.8 mm to (182.8, 94.4)
- moved C76 66.5 mm to (181.6, 76.1), turned to -90 degrees
- moved C16 66.5 mm to (197.0, 79.8), turned to 90 degrees
- moved C17 65.2 mm to (199.2, 79.8), turned to 90 degrees
- moved C24 62.9 mm to (190.0, 75.2), turned to -90 degrees
- moved L2 59.1 mm to (197.0, 76.0), turned to 90 degrees
- moved C9 58.8 mm to (185.6, 77.2), turned to -90 degrees
- moved C78 58.1 mm to (183.8, 97.0), turned to 90 degrees
- moved C10 55.8 mm to (183.9, 77.2), turned to -90 degrees
- moved C1 55.5 mm to (155.2, 78.0), turned to 135 degrees
- moved C77 55.2 mm to (182.0, 97.0), turned to 90 degrees
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Connections:
- net /1_2GHz_Frontend/RX_path/IN+ renamed /1_2GHz_Frontend/RX_path/IN_p
- net /1_2GHz_Frontend/RX_path/IN- renamed /1_2GHz_Frontend/RX_path/IN_n
- net /1_2GHz_Frontend/RX_path/in_bal+ renamed /1_2GHz_Frontend/RX_path/in_bal_p
- net /1_2GHz_Frontend/RX_path/in_bal- renamed /1_2GHz_Frontend/RX_path/in_bal_n
- net Net-(C76-Pad2) renamed /1_2GHz_Frontend/ANT_switch/hatred
- C73 pad 1: 3.3VD -> +3.3VD
- C75 pad 1: 3.3VD -> +3.3VD
- J1 pad 4: /SX_SCK -> /1_2GHz_Frontend/SX_SCK
- J1 pad 5: /SX_MOSI -> /1_2GHz_Frontend/SX_MOSI
- L12 pad 2: Net-(U14-RF1) -> /1_2GHz_Frontend/ANT_switch/stipd'
- U1 pad 6: +3.3V_RF -> +3.3VA
- U11 pad 5: +3.3VA -> Net-(Q1-C)
- U12 pad 8: 3.3VD -> +3.3VD
- U13 pad 1: 3.3VD -> +3.3VD
- U13 pad 15: 3.3VD -> +3.3VD
- U13 pad 16: 3.3VD -> +3.3VD
- U13 pad 2: 3.3VD -> +3.3VD
- U14 pad 1: Net-(U14-RF1) -> /1_2GHz_Frontend/TX_ANT
- U14 pad 3: /1_2GHz_Frontend/TX_ANT -> /1_2GHz_Frontend/ANT_switch/stipd'
- U14 pad 4: /GP1 -> Net-(Q2-C)
- U14 pad 6: +3.3V_RF -> +3.3VA
- U9 pad 17: /SX_MOSI -> /1_2GHz_Frontend/SX_MOSI
- U9 pad 18: /SX_SCK -> /1_2GHz_Frontend/SX_SCK
Routing:
- net +3.3VD: track 0.00 -> 209.6 mm, vias 4 -> 6
- net /GP1: track 0.00 -> 72.7 mm, vias 0 -> 4
- net +3.3VA: track 17.5 -> 75.2 mm, vias 9 -> 19
- net /1_2GHz_Frontend/RX_path/LE: track 0.00 -> 50.6 mm, vias 0 -> 2
- net /1_2GHz_Frontend/SX_SCK: track 0.00 -> 47.8 mm, vias 0 -> 1
- net /1_2GHz_Frontend/RX_path/CLK: track 0.00 -> 46.2 mm, vias 0 -> 2
- net /1_2GHz_Frontend/RX_path/SI: track 0.00 -> 43.7 mm, vias 0 -> 2
- net /1_2GHz_Frontend/SX_MOSI: track 0.00 -> 41.4 mm, vias 0 -> 2
- net /1_2GHz_Frontend/1.2TX_BPF: track 0.00 -> 23.8 mm
- net /1_2GHz_Frontend/RX_path/3.6GHz LO/CE: track 0.00 -> 18.5 mm, vias 0 -> 1
- net /1_2GHz_Frontend/RX_path/3.6GHz LO/LE: track 0.00 -> 16.5 mm, vias 0 -> 1
- net Net-(Q2-C): track 0.00 -> 14.7 mm
- net GND: track 0.00 -> 14.4 mm, vias 64 -> 627
- net /1_2GHz_Frontend/ANT_switch/ANT_RX: track 0.00 -> 12.4 mm
- net /SX_SCK: track 12.4 -> 0.00 mm
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- added copper zone on In2.Cu, net +3.3VA
- added copper zone on In2.Cu, net +5VA
- added copper zone on F.Cu, net /1_2GHz_Frontend/MOMG
- added copper zone on F.Cu, net /1_2GHz_Frontend/OUT_BIAS

Commit message: via hole
Connections:
- U9 pad 25: unconnected-(U9-EXP-Pad25) -> GND
Routing:
- net GND: track 14.4 -> 40.9 mm, vias 627 -> 626
- net +3.3VA: track 75.2 -> 96.2 mm
- net /1_2GHz_Frontend/OUT_BIAS: track 7.34 -> 9.36 mm
- net /1_2GHz_Frontend/RX_path/LE: track 50.6 -> 48.8 mm
- net Net-(U11-GND-Pad4): track 0.00 -> 1.29 mm
- net /1_2GHz_Frontend/RX_path/CLK: track 46.2 -> 45.3 mm
- net /1_2GHz_Frontend/RX_path/3.6GHz LO/CPOUT: track 5.00 -> 5.71 mm
- net /1_2GHz_Frontend/RX_path/3.6GHz LO/VccPLL1: track 24.3 -> 24.1 mm, vias 0 -> 2
- net /1_2GHz_Frontend/RX_path/3.6GHz LO/VccCP2: vias 0 -> 2
- net /1_2GHz_Frontend/RX_path/3.6GHz LO/VccPLL2: vias 0 -> 2
- net /1_2GHz_Frontend/RX_path/3.6GHz LO/VccCP1: vias 0 -> 2
Other:
- board text added: "ENIAC - TRX PARSA NOVIN"

Commit message: i hate sims
Parts:
- U1, U14: value 4259-63 -> AS215-92
Connections:
- U1 pad 6: +3.3VA -> GND
- U14 pad 6: +3.3VA -> GND
Routing:
- net +3.3VA: track 96.2 -> 76.6 mm, vias 19 -> 18
